File: hardware/Eagle/ION-70/ION-70.brd (EAGLE design)
At the start: 300 x 100 mm, 70 parts

Commit message: More work on ortholinear PCB
Parts:
- added U$1: ATMEGA32U4TQFP-44, SparkFun-DigitalIC:TQFP44
- S1, S15, S16, S56: device Jordi:CHERRY-MX-LED-1X1 -> Jordi:CHERRY-MX-LED-1X1.5
- S17: device Jordi:CHERRY-MX-LED-1X1.25 -> Jordi:CHERRY-MX-LED-1X1
- S31: device Jordi:CHERRY-MX-LED-1X1.25 -> Jordi:CHERRY-MX-LED-1X1.5
- S32: device Jordi:CHERRY-MX-LED-1X1.5 -> Jordi:CHERRY-MX-LED-1X1
- S43: device Jordi:CHERRY-MX-LED-1X1 -> Jordi:CHERRY-MX-LED-1X2
- S44: device Jordi:CHERRY-MX-LED-1X2 -> Jordi:CHERRY-MX-LED-1X1.5
- S46, S57: device Jordi:CHERRY-MX-LED-1X2 -> Jordi:CHERRY-MX-LED-1X1
- moved S16 281.6 mm to (11.9, 69.1)
- moved S31 279.3 mm to (11.9, 50.0)
- moved S45 276.9 mm to (11.9, 30.9)
- moved S44 33.3 mm to (288.1, 50.0)
- moved S43 28.6 mm to (254.8, 50.0)
- moved S17 26.2 mm to (35.7, 69.0)
- moved S32 23.8 mm to (35.7, 50.0)
- moved S18 23.8 mm to (54.8, 69.0)
- moved S19 23.8 mm to (73.8, 69.0)
- moved S20 23.8 mm to (92.8, 69.0)
- moved S21 23.8 mm to (111.9, 69.0)
- moved S23 23.8 mm to (150.0, 69.0)
- moved S24 23.8 mm to (169.1, 69.0)
- moved S25 23.8 mm to (188.1, 69.0)
- moved S26 23.8 mm to (207.2, 69.0)
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