File: hardware/Eagle/ION-70/ION-70.sch (EAGLE design)
At the start: 70 parts

Commit message: More work on ortholinear PCB
Parts:
- added U$1: ATMEGA32U4TQFP-44, SparkFun-DigitalIC:ATMEGA32U4TQFP-44
- S1, S15, S16, S56: device Jordi:CHERRY-MX-LED1X1 -> Jordi:CHERRY-MX-LED1X1.5
- S17: device Jordi:CHERRY-MX-LED1X1.25 -> Jordi:CHERRY-MX-LED1X1
- S31: device Jordi:CHERRY-MX-LED1X1.25 -> Jordi:CHERRY-MX-LED1X1.5
- S32: device Jordi:CHERRY-MX-LED1X1.5 -> Jordi:CHERRY-MX-LED1X1
- S43: device Jordi:CHERRY-MX-LED1X1 -> Jordi:CHERRY-MX-LED1X2
- S44: device Jordi:CHERRY-MX-LED1X2 -> Jordi:CHERRY-MX-LED1X1.5
- S46, S57: device Jordi:CHERRY-MX-LED1X2 -> Jordi:CHERRY-MX-LED1X1
Other:
- moved on the sheet: S1, S10, S11, S12, S13, S14, S15, S16, S17, S18, S19, S2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
