File: hardware/ION-60/Eagle/ION-60/ION-60.brd (EAGLE design)
At the start: 300 x 100 mm, 71 parts

Commit message: Edit PCB
Parts:
- S1, S15, S16, S30, S31, S44, S45, S56: device Jordi:CHERRY-MX-LED-1X1.5 -> Jordi:CHERRY-MX-LED-1X1
- S43: device Jordi:CHERRY-MX-LED-1X2 -> Jordi:CHERRY-MX-LED-1X1
- S60: device Jordi:CHERRY-MX-LED-1X1.25 -> Jordi:CHERRY-MX-LED-1X1
- S61, S62, S65, S66, S67: device Jordi:CHERRY-MX-LED-1X1.25 -> Jordi:CHERRY-MX-LED-1X1.5
- S63, S64: device Jordi:CHERRY-MX-LED-1X2.75 -> Jordi:CHERRY-MX-LED-1X1.5
- S68, S69, S70: device Jordi:CHERRY-MX-LED-1X1 -> Jordi:CHERRY-MX-LED-1X1.5
- moved S60 274.5 mm to (283.4, 30.9)
- moved S45 272.1 mm to (283.4, 50.0)
- moved U$1 129.6 mm to (150.0, 11.9)
- moved S65 50.0 mm to (135.7, 11.9)
- moved S66 45.2 mm to (164.3, 11.9)
- moved S64 40.5 mm to (107.1, 11.9)
- moved S67 40.5 mm to (192.9, 11.9)
- moved S68 33.3 mm to (221.4, 11.9)
- moved S57 28.6 mm to (226.2, 30.9)
- moved S58 28.6 mm to (245.2, 30.9)
- moved S59 28.6 mm to (264.3, 30.9)
- moved S44 23.8 mm to (264.3, 50.0)
- moved S56 23.8 mm to (207.2, 30.9)
- moved S69 23.8 mm to (250.0, 11.9)
- moved S50 19.1 mm to (92.8, 30.9)
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Other:
- board size 300 x 100 mm -> 280 x 90 mm
Changed lines of the file:
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@@
 <board>
 <plain>
-<wire x1="0" y1="0" x2="300" y2="0" width="0" layer="20"/>
-<wire x1="300" y1="0" x2="300" y2="100" width="0" layer="20"/>
-<wire x1="300" y1="100" x2="0" y2="100" width="0" layer="20"/>
-<wire x1="0" y1="100" x2="0" y2="0" width="0" layer="20"/>
-<hole x="23.79375" y="78.575" drill="3"/>
-<hole x="276.20625" y="78.575" drill="3"/>
-<hole x="276.20625" y="21.425" drill="3"/>
-<hole x="23.79375" y="21.425" drill="3"/>
-<hole x="102.375" y="78.575" drill="3"/>
-<hole x="102.375" y="21.425" drill="3"/>
-<hole x="197.64375" y="78.58125" drill="3"/>
-<hole x="197.64375" y="21.43125" drill="3"/>
+<wire x1="10" y1="5" x2="290" y2="5" width="0" layer="20"/>
+<wire x1="290" y1="5" x2="290" y2="95" width="0" layer="20"/>
+<wire x1="290" y1="95" x2="12.5" y2="95" width="0" layer="20"/>
+<wire x1="12.5" y1="95" x2="10" y2="92.5" width="0" layer="20" curve="90"/>
+<wire x1="10" y1="92.5" x2="10" y2="5" width="0" layer="20"/>
 </plain>
 <attributes>
@@
 </autorouter>
 <elements>
-<element name="S1" library="Jordi" package="CHERRY-MX-LED-1X1.5" value="" x="11.8875" y="88.1"/>
+<element name="S1" library="Jordi" package="CHERRY-MX-LED-1X1" value="" x="16.65" y="88.1"/>
 <element name="S2" library="Jordi" package="CHERRY-MX-LED-1X1" value="" x="35.7" y="88.1"/>
 <element name="S3" library="Jordi" package="CHERRY-MX-LED-1X1" value="" x="54.75" y="88.1"/>
@@
 <element name="S13" library="Jordi" package="CHERRY-MX-LED-1X1" value="" x="245.25" y="88.1"/>
 <element name="S14" library="Jordi" package="CHERRY-MX-LED-1X1" value="" x="264.3" y="88.1"/>
-<element name="S15" library="Jordi" package="CHERRY-MX-LED-1X1.5" value="" x="288.1125" y="88.1"/>
-<element name="S16" library="Jordi" package="CHERRY-MX-LED-1X1.5" value="" x="11.90625" y="69.05625"/>
+<element name="S15" library="Jordi" package="CHERRY-MX-LED-1X1" value="" x="283.35" y="88.1"/>
+<element name="S16" library="Jordi" package="CHERRY-MX-LED-1X1" value="" x="16.66875" y="69.05625"/>
 <element name="S17" library="Jordi" package="CHERRY-MX-LED-1X1" value="" x="35.7" y="69.05"/>
 <element name="S18" library="Jordi" package="CHERRY-MX-LED-1X1" value="" x="54.75" y="69.05"/>
@@
 <element name="S28" library="Jordi" package="CHERRY-MX-LED-1X1" value="" x="245.25" y="69.05"/>
 <element name="S29" library="Jordi" package="CHERRY-MX-LED-1X1" value="" x="264.3" y="69.05"/>
-<element name="S30" library="Jordi" package="CHERRY-MX-LED-1X1.5" value="" x="288.1125" y="69.05"/>
-<element name="S31" library="Jordi" package="CHERRY-MX-LED-1X1.5" value="" x="11.8875" y="50"/>
+<element name="S30" library="Jordi" package="CHERRY-MX-LED-1X1" value="" x="283.35" y="69.05"/>
+<element name="S31" library="Jordi" package="CHERRY-MX-LED-1X1" value="" x="16.65" y="50"/>
 <element name="S32" library="Jordi" package="CHERRY-MX-LED-1X1" value="" x="35.7" y="50"/>
 <element name="S33" library="Jordi" package="CHERRY-MX-LED-1X1" value="" x="54.75" y="50"/>
@@
 <element name="S41" library="Jordi" package="CHERRY-MX-LED-1X1" value="" x="207.15" y="50"/>
 <element name="S42" library="Jordi" package="CHERRY-MX-LED-1X1" value="" x="226.2" y="50"/>
-<element name="S43" library="Jordi" package="CHERRY-MX-LED-1X2" value="" x="254.775" y="50"/>
-<element name="S44" library="Jordi" package="CHERRY-MX-LED-1X1.5" value="" x="288.1125" y="50"/>
-<element name="S45" library="Jordi" package="CHERRY-MX-LED-1X1.5" value="" x="11.8875" y="30.95"/>
-<element name="S46" library="Jordi" package="CHERRY-MX-LED-1X1" value="" x="35.7" y="30.95"/>
-<element name="S47" library="Jordi" package="CHERRY-MX-LED-1X1" value="" x="54.75" y="30.95"/>
-<element name="S48" library="Jordi" package="CHERRY-MX-LED-1X1" value="" x="73.8" y="30.95"/>
-<element name="S49" library="Jordi" package="CHERRY-MX-LED-1X1" value="" x="92.85" y="30.95"/>
-<element name="S50" library="Jordi" package="CHERRY-MX-LED-1X1" value="" x="111.9" y="30.95"/>
-<element name="S51" library="Jordi" package="CHERRY-MX-LED-1X1" value="" x="130.95" y="30.95"/>
-<element name="S52" library="Jordi" package="CHERRY-MX-LED-1X1" value="" x="150" y="30.95"/>
-<element name="S53" library="Jordi" package="CHERRY-MX-LED-1X1" value="" x="169.05" y="30.95"/>
-<element name="S54" library="Jordi" package="CHERRY-MX-LED-1X1" value="" x="188.1" y="30.95"/>
-<element name="S55" library="Jordi" package="CHERRY-MX-LED-1X1" value="" x="207.15" y="30.95"/>
-<element name="S56" library="Jordi" package="CHERRY-MX-LED-1X1.5" value="" x="230.9625" y="30.95"/>
-<element name="S57" library="Jordi" package="CHERRY-MX-LED-1X1" value="" x="254.775" y="30.95"/>
-<element name="S58" library="Jordi" package="CHERRY-MX-LED-1X1" value="" x="273.825" y="30.95"/>
-<element name="S59" library="Jordi" package="CHERRY-MX-LED-1X1" value="" x="292.875" y="30.95"/>
-<element name="S60" library="Jordi" package="CHERRY-MX-LED-1X1.25" value="" x="9.50625" y="11.9"/>
-<element name="S61" library="Jordi" package="CHERRY-MX-LED-1X1.25" value="" x="33.31875" y="11.9"/>
-<element name="S62" library="Jordi" package="CHERRY-MX-LED-1X1.25" value="" x="57.13125" y="11.9"/>
-<element name="S63" library="Jordi" package="CHERRY-MX-LED-1X2.75" value="" x="95.23125" y="11.9"/>
-<element name="S64" library="Jordi" package="CHERRY-MX-LED-1X2.75" value="" x="147.61875" y="11.9"/>
-<element name="S65" library="Jordi" package="CHERRY-MX-LED-1X1.25" value="" x="185.71875" y="11.9"/>
-<element name="S66" library="Jordi" package="CHERRY-MX-LED-1X1.25" value="" x="209.53125" y="11.9"/>
-<element name="S67" library="Jordi" package="CHERRY-MX-LED-1X1.25" value="" x="233.34375" y="11.9"/>
-<element name="S68" library="Jordi" package="CHERRY-MX-LED-1X1" value="" x="254.775" y="11.9"/>
-<element name="S69" library="Jordi" package="CHERRY-MX-LED-1X1" value="" x="273.825" y="11.9"/>
-<element name="S70" library="Jordi" package="CHERRY-MX-LED-1X1" value="" x="292.875" y="11.9"/>
-<element name="U$1" library="SparkFun-DigitalIC" package="TQFP44" value="ATMEGA32U4TQFP-44" x="273.84375" y="50.00625" rot="MR0"/>
+<element name="S43" library="Jordi" package="CHERRY-MX-LED-1X1" value="" x="245.25" y="50"/>
+<element name="S44" library="Jordi" package="CHERRY-MX-LED-1X1" value="" x="264.3" y="50"/>
+<element name="S45" library="Jordi" package="CHERRY-MX-LED-1X1" value="" x="283.35" y="50"/>
+<element name="S46" library="Jordi" package="CHERRY-MX-LED-1X1" value="" x="16.65" y="30.95"/>
+<element name="S47" library="Jordi" package="CHERRY-MX-LED-1X1" value="" x="35.7" y="30.95"/>
+<element name="S48" library="Jordi" package="CHERRY-MX-LED-1X1" value="" x="54.75" y="30.95"/>
+<element name="S49" library="Jordi" package="CHERRY-MX-LED-1X1" value="" x="73.8" y="30.95"/>
+<element name="S50" library="Jordi" package="CHERRY-MX-LED-1X1" value="" x="92.85" y="30.95"/>
+<element name="S51" library="Jordi" package="CHERRY-MX-LED-1X1" value="" x="111.9" y="30.95"/>
+<element name="S52" library="Jordi" package="CHERRY-MX-LED-1X1" value="" x="130.95" y="30.95"/>
+<element name="S53" library="Jordi" package="CHERRY-MX-LED-1X1" value="" x="150" y="30.95"/>
+<element name="S54" library="Jordi" package="CHERRY-MX-LED-1X1" value="" x="169.05" y="30.95"/>
+<element name="S55" library="Jordi" package="CHERRY-MX-LED-1X1" value="" x="188.1" y="30.95"/>
+<element name="S56" library="Jordi" package="CHERRY-MX-LED-1X1" value="" x="207.15" y="30.95"/>
+<element name="S57" library="Jordi" package="CHERRY-MX-LED-1X1" value="" x="226.2" y="30.95"/>
+<element name="S58" library="Jordi" package="CHERRY-MX-LED-1X1" value="" x="245.25" y="30.95"/>
+<element name="S59" library="Jordi" package="CHERRY-MX-LED-1X1" value="" x="264.3" y="30.95"/>
+<element name="S60" library="Jordi" package="CHERRY-MX-LED-1X1" value="" x="283.35" y="30.95"/>
+<element name="S61" library="Jordi" package="CHERRY-MX-LED-1X1.5" value="" x="21.4125" y="11.9"/>
+<element name="S62" library="Jordi" package="CHERRY-MX-LED-1X1.5" value="" x="49.9875" y="11.9"/>
+<element name="S63" library="Jordi" package="CHERRY-MX-LED-1X1.5" value="" x="78.5625" y="11.9"/>
+<element name="S64" library="Jordi" package="CHERRY-MX-LED-1X1.5" value="" x="107.1375" y="11.9"/>
+<element name="S65" library="Jordi" package="CHERRY-MX-LED-1X1.5" value="" x="135.7125" y="11.9"/>
+<element name="S66" library="Jordi" package="CHERRY-MX-LED-1X1.5" value="" x="164.2875" y="11.9"/>
+<element name="S67" library="Jordi" package="CHERRY-MX-LED-1X1.5" value="" x="192.8625" y="11.9"/>
+<element name="S68" library="Jordi" package="CHERRY-MX-LED-1X1.5" value="" x="221.4375" y="11.9"/>
+<element name="S69" library="Jordi" package="CHERRY-MX-LED-1X1.5" value="" x="250.0125" y="11.9"/>
+<element name="S70" library="Jordi" package="CHERRY-MX-LED-1X1.5" value="" x="278.5875" y="11.9"/>
+<element name="U$1" library="SparkFun-DigitalIC" package="TQFP44" value="ATMEGA32U4TQFP-44" x="150.01875" y="11.90625" rot="MR0"/>
 </elements>
 <signals>

Commit message: Further additions to PCB
Parts:
- added D46: (no value), SparkFun-DiscreteSemi:SOD-123
- added IC1: TLC5947DAP, Jordi:HTSSOP-32
- added Y1: (no value), Jordi:CRYSTAL-SMD-3.2X2.5
Connections:
- new net GND: IC1.1
- new net N$10: U$1.16, Y1.3
- new net N$11: S1.LED1, S10.LED1, S11.LED1, S12.LED1, S13.LED1, S14.LED1, S15.LED1, S2.LED1, S3.LED1, S4.LED1, S5.LED1, S6.LED1, S7.LED1, S8.LED1, S9.LED1
- new net N$12: S1.LED2, S16.LED2, S31.LED2, S46.LED2, S61.LED2
- new net N$13: S17.LED2, S2.LED2, S32.LED2, S47.LED2
- new net N$14: S18.LED2, S3.LED2, S33.LED2, S48.LED2, S62.LED2
- new net N$15: D46.A, S46.SW2, S46.SW4
- new net N$9: U$1.17, Y1.1
- new net PAD: IC1.PAD
- new net VCC: IC1.32
Other:
- outline, holes or cut-outs redrawn
Changed lines of the file:
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@@
 <?xml version="1.0" encoding="utf-8"?>
 <!DOCTYPE eagle SYSTEM "eagle.dtd">
-<eagle version="6.5.0">
+<eagle version="7.2.0">
 <drawing>
 <settings>
@@
 <layer number="59" name="tCarbon" color="7" fill="1" visible="no" active="no"/>
 <layer number="60" name="bCarbon" color="7" fill="1" visible="no" active="no"/>
-<layer number="90" name="Modules" color="5" fill="1" visible="yes" active="yes"/>
+<layer number="90" name="Modules" color="5" fill="1" visible="no" active="no"/>
 <layer number="91" name="Nets" color="2" fill="1" visible="no" active="no"/>
 <layer number="92" name="Busses" color="1" fill="1" visible="no" active="no"/>
@@
 <board>
 <plain>
-<wire x1="10" y1="5" x2="290" y2="5" width="0" layer="20"/>
-<wire x1="290" y1="5" x2="290" y2="95" width="0" layer="20"/>
-<wire x1="290" y1="95" x2="12.5" y2="95" width="0" layer="20"/>
+<wire x1="10" y1="92.5" x2="10" y2="7.5" width="0" layer="20"/>
+<wire x1="10" y1="7.5" x2="12.5" y2="5" width="0" layer="20" curve="90"/>
+<wire x1="12.5" y1="5" x2="287.5" y2="5" width="0" layer="20"/>
+<wire x1="287.5" y1="5" x2="290" y2="7.5" width="0" layer="20" curve="90"/>
+<wire x1="290" y1="7.5" x2="290" y2="92.5" width="0" layer="20"/>
+<wire x1="290" y1="92.5" x2="287.5" y2="95" width="0" layer="20" curve="90"/>
+<wire x1="287.5" y1="95" x2="12.5" y2="95" width="0" layer="20"/>
 <wire x1="12.5" y1="95" x2="10" y2="92.5" width="0" layer="20" curve="90"/>
-<wire x1="10" y1="92.5" x2="10" y2="5" width="0" layer="20"/>
 </plain>
 <attributes>
@@
 <pass name="Default">
 <param name="RoutingGrid" value="50mil"/>
+<param name="AutoGrid" value="1"/>
+<param name="Efforts" value="0"/>
+<param name="TopRouterVariant" value="1"/>
 <param name="tpViaShape" value="round"/>
 <param name="PrefDir.1" value="|"/>
@@
 <element name="S70" library="Jordi" package="CHERRY-MX-LED-1X1.5" value="" x="278.5875" y="11.9"/>
 <element name="U$1" library="SparkFun-DigitalIC" package="TQFP44" value="ATMEGA32U4TQFP-44" x="150.01875" y="11.90625" rot="MR0"/>
+<element name="Y1" library="Jordi" package="CRYSTAL-SMD-3.2X2.5" value="" x="66.675" y="11.90625" rot="MR0"/>
+<element name="D46" library="SparkFun-DiscreteSemi" package="SOD-123" value="" x="21.43125" y="33.3375" rot="MR0"/>
+<element name="IC1" library="Jordi" package="HTSSOP-32" value="TLC5947DAP" x="92.86875" y="11.90625" rot="MR270"/>
 </elements>
 <signals>
+<signal name="N$1">
+<via x="64.29375" y="78.58125" extent="1-16" drill="3" diameter="5"/>
+</signal>
+<signal name="N$2">
+<via x="121.44375" y="78.58125" extent="1-16" drill="3" diameter="5"/>
+</signal>
+<signal name="N$3">
+<via x="178.59375" y="78.58125" extent="1-16" drill="3" diameter="5"/>
+</signal>
+<signal name="N$4">
+<via x="235.74375" y="78.58125" extent="1-16" drill="3" diameter="5"/>
+</signal>
+<signal name="N$5">
+<via x="64.29375" y="21.43125" extent="1-16" drill="3" diameter="5"/>
+</signal>
+<signal name="N$6">
+<via x="121.44375" y="21.43125" extent="1-16" drill="3" diameter="5"/>
+</signal>
+<signal name="N$7">
+<via x="178.59375" y="21.43125" extent="1-16" drill="3" diameter="5"/>
+</signal>
+<signal name="N$8">
+<via x="235.74375" y="21.43125" extent="1-16" drill="3" diameter="5"/>
+</signal>
+<signal name="N$9">
+<contactref element="U$1" pad="17"/>
+<contactref element="Y1" pad="1"/>
+<wire x1="67.775" y1="11.10625" x2="150.01875" y2="6.10625" width="0" layer="19" extent="1-16"/>
+</signal>
+<signal name="N$10">
+<contactref element="U$1" pad="16"/>
+<contactref element="Y1" pad="3"/>
+<wire x1="65.575" y1="12.70625" x2="150.81875" y2="6.10625" width="0" layer="19" extent="1-16"/>
+</signal>
+<signal name="N$11">
+<contactref element="S1" pad="LED1"/>
+<contactref element="S2" pad="LED1"/>
+<contactref element="S3" pad="LED1"/>
+<contactref element="S4" pad="LED1"/>
+<contactref element="S5" pad="LED1"/>
+<contactref element="S6" pad="LED1"/>
+<contactref element="S7" pad="LED1"/>
+<contactref element="S8" pad="LED1"/>
+<contactref element="S9" pad="LED1"/>
+<contactref element="S10" pad="LED1"/>
+<contactref element="S11" pad="LED1"/>
+<contactref element="S12" pad="LED1"/>
+<contactref element="S13" pad="LED1"/>
+<contactref element="S14" pad="LED1"/>
+<contactref element="S15" pad="LED1"/>
+<wire x1="148.73" y1="84.29" x2="167.78" y2="84.29" width="0" layer="19" extent="1-1"/>
+<wire x1="129.68" y1="84.29" x2="148.73" y2="84.29" width="0" layer="19" extent="1-1"/>
+<wire x1="110.63" y1="84.29" x2="129.68" y2="84.29" width="0" layer="19" extent="1-1"/>
+<wire x1="91.58" y1="84.29" x2="110.63" y2="84.29" width="0" layer="19" extent="1-1"/>
+<wire x1="72.53" y1="84.29" x2="91.58" y2="84.29" width="0" layer="19" extent="1-1"/>
+<wire x1="53.48" y1="84.29" x2="72.53" y2="84.29" width="0" layer="19" extent="1-1"/>
+<wire x1="34.43" y1="84.29" x2="53.48" y2="84.29" width="0" layer="19" extent="1-1"/>
+<wire x1="15.38" y1="84.29" x2="34.43" y2="84.29" width="0" layer="19" extent="1-1"/>
+<wire x1="186.83" y1="84.29" x2="167.78" y2="84.29" width="0" layer="19" extent="1-1"/>
+<wire x1="205.88" y1="84.29" x2="186.83" y2="84.29" width="0" layer="19" extent="1-1"/>
+<wire x1="224.93" y1="84.29" x2="205.88" y2="84.29" width="0" layer="19" extent="1-1"/>
+<wire x1="243.98" y1="84.29" x2="224.93" y2="84.29" width="0" layer="19" extent="1-1"/>
+<wire x1="263.03" y1="84.29" x2="243.98" y2="84.29" width="0" layer="19" extent="1-1"/>
+<wire x1="282.08" y1="84.29" x2="263.03" y2="84.29" width="0" layer="19" extent="1-1"/>
+</signal>
+<signal name="N$12">
+<contactref element="S1" pad="LED2"/>
+<contactref element="S16" pad="LED2"/>
+<contactref element="S31" pad="LED2"/>
+<contactref element="S46" pad="LED2"/>
+<contactref element="S61" pad="LED2"/>
+<wire x1="17.93875" y1="65.24625" x2="17.92" y2="84.29" width="0" layer="19" extent="1-1"/>
+<wire x1="17.92" y1="46.19" x2="17.93875" y2="65.24625" width="0" layer="19" extent="1-1"/>
+<wire x1="17.92" y1="27.14" x2="17.92" y2="46.19" width="0" layer="19" extent="1-1"/>
+<wire x1="22.6825" y1="8.09" x2="17.92" y2="27.14" width="0" layer="19" extent="1-1"/>
+</signal>
+<signal name="N$13">
+<contactref element="S2" pad="LED2"/>
+<contactref element="S17" pad="LED2"/>
+<contactref element="S32" pad="LED2"/>
+<contactref element="S47" pad="LED2"/>
+<wire x1="36.97" y1="65.24" x2="36.97" y2="84.29" width="0" layer="19" extent="1-1"/>
+<wire x1="36.97" y1="46.19" x2="36.97" y2="65.24" width="0" layer="19" extent="1-1"/>
+<wire x1="36.97" y1="27.14" x2="36.97" y2="46.19" width="0" layer="19" extent="1-1"/>
+</signal>
+<signal name="N$14">
+<contactref element="S3" pad="LED2"/>
+<contactref element="S18" pad="LED2"/>
+<contactref element="S33" pad="LED2"/>
+<contactref element="S48" pad="LED2"/>
+<contactref element="S62" pad="LED2"/>
+<wire x1="56.02" y1="65.24" x2="56.02" y2="84.29" width="0" layer="19" extent="1-1"/>
+<wire x1="56.02" y1="46.19" x2="56.02" y2="65.24" width="0" layer="19" extent="1-1"/>
+<wire x1="56.02" y1="27.14" x2="56.02" y2="46.19" width="0" layer="19" extent="1-1"/>
+<wire x1="51.2575" y1="8.09" x2="56.02" y2="27.14" width="0" layer="19" extent="1-1"/>
+</signal>
+<signal name="N$15">
+<contactref element="S46" pad="SW2"/>
+<contactref element="S46" pad="SW4"/>
+<contactref element="D46" pad="A"/>
+<wire x1="19.15" y1="35.45" x2="19.19" y2="36.03" width="0" layer="19" extent="1-1"/>
+<wire x1="19.85625" y1="33.3375" x2="19.15" y2="35.45" width="0" layer="19" extent="16-16"/>
+</signal>
+<signal name="GND">
+<contactref element="IC1" pad="1"/>
+</signal>
+<signal name="VCC">
+<contactref element="IC1" pad="32"/>
+</signal>
+<signal name="PAD">
+<contactref element="IC1" pad="PAD"/>
+</signal>
 </signals>
 </board>
