File: hardware/ION-60/Eagle/ION-60/ION-60.brd (EAGLE design)
At the start: 280 x 90 mm, 74 parts, among them IC1 TLC5947DAP

Commit message: More work on PCB
Parts:
- added D1, D10, D11, D12, D13, D14, D15, D16, D17, D18, D19, D2, D20, D21, D22, D23, D24, D25, D26, D27, D28, D29, D3, D30, D31, D32, D33, D34, D35, D36, D37, D38, D39, D4, D40, D41, D42, D43, D44, D45, D47, D48, D49, D5, D50, D51, D52, D53, D54, D55, D56, D57, D58, D59, D6, D60, D61, D62, D63, D64, D65, D66, D67, D68, D69, D7, D70, D8, D9: (no value), SparkFun-DiscreteSemi:SOD-123
- added IC2: 74LS137D, 74xx-us:SO16
- added IC3, IC4: TLC5947DAP, Jordi:HTSSOP-32
- IC1: value TLC5947DAP -> 74LS137D; device Jordi:HTSSOP-32 -> 74xx-us:SO16
- Y1: value (none) -> 16MHz
- moved Y1 90.7 mm to (157.2, 5.95), turned to 180 degrees
- moved IC1 28.6 mm to (121.4, 11.9), turned to 0 degrees
- moved D46 5.32 mm to (16.7, 35.7), turned to 270 degrees
- turned U$1 to 45 degrees
Connections:
- net N$11 renamed LED-A0
- removed net PAD: IC1.PAD
- new net +3V3: IC3.32, IC4.32, U$1.14, U$1.24, U$1.34, U$1.44
- new net A0: IC1.1, IC2.1, U$1.39
- new net A1: IC1.2, IC2.2, U$1.38
- new net A2: IC1.3, IC2.3, U$1.37
- new net A3: IC1.6, IC2.5, U$1.36
- new net AL: IC1.4, IC2.4
- new net C0: IC1.7, S1.SW1, S1.SW3, S16.SW1, S16.SW3, S31.SW1, S31.SW3, S46.SW1, S46.SW3, S61.SW1, S61.SW3
- new net C1: IC1.9, S17.SW1, S17.SW3, S2.SW1, S2.SW3, S32.SW1, S32.SW3, S47.SW1, S47.SW3
- new net C10: IC2.10, S11.SW1, S11.SW3, S26.SW1, S26.SW3, S41.SW1, S41.SW3, S56.SW1, S56.SW3
- new net C11: IC2.11, S12.SW1, S12.SW3, S27.SW1, S27.SW3, S42.SW1, S42.SW3, S57.SW1, S57.SW3, S68.SW1, S68.SW3
- new net C12: IC2.12, S13.SW1, S13.SW3, S28.SW1, S28.SW3, S43.SW1, S43.SW3, S58.SW1, S58.SW3, S69.SW1, S69.SW3
- new net C13: IC2.13, S14.SW1, S14.SW3, S29.SW1, S29.SW3, S44.SW1, S44.SW3, S59.SW1, S59.SW3
- new net C14: IC2.14, S15.SW1, S15.SW3, S30.SW1, S30.SW3, S45.SW1, S45.SW3, S60.SW1, S60.SW3, S70.SW1, S70.SW3
- new net C2: IC1.10, S18.SW1, S18.SW3, S3.SW1, S3.SW3, S33.SW1, S33.SW3, S48.SW1, S48.SW3, S62.SW1, S62.SW3
- new net C3: IC1.11, S19.SW1, S19.SW3, S34.SW1, S34.SW3, S4.SW1, S4.SW3, S49.SW1, S49.SW3, S63.SW1, S63.SW3
- new net C4: IC1.12, S20.SW1, S20.SW3, S35.SW1, S35.SW3, S5.SW1, S5.SW3, S50.SW1, S50.SW3
- new net C5: IC1.13, S21.SW1, S21.SW3, S36.SW1, S36.SW3, S51.SW1, S51.SW3, S6.SW1, S6.SW3, S64.SW1, S64.SW3
- new net C6: IC1.14, S22.SW1, S22.SW3, S37.SW1, S37.SW3, S52.SW1, S52.SW3, S65.SW1, S65.SW3, S7.SW1, S7.SW3
- new net C7: IC1.15, S23.SW1, S23.SW3, S38.SW1, S38.SW3, S53.SW1, S53.SW3, S8.SW1, S8.SW3
- new net C8: IC2.7, S24.SW1, S24.SW3, S39.SW1, S39.SW3, S54.SW1, S54.SW3, S66.SW1, S66.SW3, S9.SW1, S9.SW3
- new net C9: IC2.9, S10.SW1, S10.SW3, S25.SW1, S25.SW3, S40.SW1, S40.SW3, S55.SW1, S55.SW3, S67.SW1, S67.SW3
- new net E0: IC1.5, U$1.41
- new net E1: IC2.6, U$1.40
- new net LED-A1: S16.LED1, S17.LED1, S18.LED1, S19.LED1, S20.LED1, S21.LED1, S22.LED1, S23.LED1, S24.LED1, S25.LED1, S26.LED1, S27.LED1, S28.LED1, S29.LED1, S30.LED1
- new net LED-A2: S31.LED1, S32.LED1, S33.LED1, S34.LED1, S35.LED1, S36.LED1, S37.LED1, S38.LED1, S39.LED1, S40.LED1, S41.LED1, S42.LED1, S43.LED1, S44.LED1, S45.LED1
- new net LED-A3: S46.LED1, S47.LED1, S48.LED1, S49.LED1, S50.LED1, S51.LED1, S52.LED1, S53.LED1, S54.LED1, S55.LED1, S56.LED1, S57.LED1, S58.LED1, S59.LED1, S60.LED1
- new net LED-A4: S61.LED1, S62.LED1, S63.LED1, S64.LED1, S65.LED1, S66.LED1, S67.LED1, S68.LED1, S69.LED1, S70.LED1
- new net LED-B0: IC3.7, S1.D2, S16.D2, S31.D2, S46.D2, S61.D2
- new net LED-B1: IC3.10, S17.D2, S2.D2, S32.D2, S47.D2
- new net LED-B10: S11.D2, S26.D2, S41.D2, S56.D2
- new net LED-B11: S12.D2, S27.D2, S42.D2, S57.D2, S68.D2
- new net LED-B12: S13.D2, S28.D2, S43.D2, S58.D2, S69.D2
- new net LED-B13: S14.D2, S29.D2, S44.D2, S59.D2
- new net LED-B14: S15.D2, S30.D2, S45.D2, S60.D2, S70.D2
- new net LED-B2: IC3.13, S18.D2, S3.D2, S33.D2, S48.D2, S62.D2
- new net LED-B3: IC3.16, S19.D2, S34.D2, S4.D2, S49.D2, S63.D2
- new net LED-B4: IC3.19, S20.D2, S35.D2, S5.D2, S50.D2
- new net LED-B5: IC3.22, S21.D2, S36.D2, S51.D2, S6.D2, S64.D2
- new net LED-B6: IC3.25, S22.D2, S37.D2, S52.D2, S65.D2, S7.D2
- new net LED-B7: IC3.28, S23.D2, S38.D2, S53.D2, S8.D2
- new net LED-B8: S24.D2, S39.D2, S54.D2, S66.D2, S9.D2
- new net LED-B9: S10.D2, S25.D2, S40.D2, S55.D2, S67.D2
- new net LED-G0: IC3.5, S1.D1, S16.D1, S31.D1, S46.D1, S61.D1
- new net LED-G1: IC3.8, S17.D1, S2.D1, S32.D1, S47.D1
- new net LED-G10: S11.D1, S26.D1, S41.D1, S56.D1
- new net LED-G11: S12.D1, S27.D1, S42.D1, S57.D1, S68.D1
- new net LED-G12: S13.D1, S28.D1, S43.D1, S58.D1, S69.D1
- new net LED-G13: S14.D1, S29.D1, S44.D1, S59.D1
- new net LED-G14: S15.D1, S30.D1, S45.D1, S60.D1, S70.D1
- new net LED-G2: IC3.11, S18.D1, S3.D1, S33.D1, S48.D1, S62.D1
- new net LED-G3: IC3.14, S19.D1, S34.D1, S4.D1, S49.D1, S63.D1
- new net LED-G4: IC3.17, S20.D1, S35.D1, S5.D1, S50.D1
- new net LED-G5: IC3.20, S21.D1, S36.D1, S51.D1, S6.D1, S64.D1
- new net LED-G6: IC3.23, S22.D1, S37.D1, S52.D1, S65.D1, S7.D1
- new net LED-G7: IC3.26, S23.D1, S38.D1, S53.D1, S8.D1
- new net LED-G8: S24.D1, S39.D1, S54.D1, S66.D1, S9.D1
- new net LED-G9: S10.D1, S25.D1, S40.D1, S55.D1, S67.D1
- new net LED-R0: IC3.6, S1.LED2, S16.LED2, S31.LED2, S46.LED2, S61.LED2
- new net LED-R1: IC3.9, S17.LED2, S2.LED2, S32.LED2, S47.LED2
- new net LED-R10: S11.LED2, S26.LED2, S41.LED2, S56.LED2
- new net LED-R11: S12.LED2, S27.LED2, S42.LED2, S57.LED2, S68.LED2
- new net LED-R12: S13.LED2, S28.LED2, S43.LED2, S58.LED2, S69.LED2
- new net LED-R13: S14.LED2, S29.LED2, S44.LED2, S59.LED2
- new net LED-R14: S15.LED2, S30.LED2, S45.LED2, S60.LED2, S70.LED2
- new net LED-R2: IC3.12, S18.LED2, S3.LED2, S33.LED2, S48.LED2, S62.LED2
- new net LED-R3: IC3.15, S19.LED2, S34.LED2, S4.LED2, S49.LED2, S63.LED2
- new net LED-R4: IC3.18, S20.LED2, S35.LED2, S5.LED2, S50.LED2
- new net LED-R5: IC3.21, S21.LED2, S36.LED2, S51.LED2, S6.LED2, S64.LED2
- new net LED-R6: IC3.24, S22.LED2, S37.LED2, S52.LED2, S65.LED2, S7.LED2
- new net LED-R7: IC3.27, S23.LED2, S38.LED2, S53.LED2, S8.LED2
- new net LED-R8: S24.LED2, S39.LED2, S54.LED2, S66.LED2, S9.LED2
- new net LED-R9: S10.LED2, S25.LED2, S40.LED2, S55.LED2, S67.LED2
- new net MISO: U$1.11
- new net MOSI: IC3.4, U$1.10
- new net N$100: D29.A, S29.SW2, S29.SW4
- new net N$101: D30.A, S30.SW2, S30.SW4
- new net N$102: D45.A, S45.SW2, S45.SW4
- new net N$103: D60.A, S60.SW2, S60.SW4
- new net N$104: D70.A, S70.SW2, S70.SW4
- new net N$11: D2.A, S2.SW2, S2.SW4
- new net N$15: D53.A, S53.SW2, S53.SW4
- new net N$16: D3.A, S3.SW2, S3.SW4
- new net N$17: D4.A, S4.SW2, S4.SW4
- new net N$18: D5.A, S5.SW2, S5.SW4
- new net N$19: D6.A, S6.SW2, S6.SW4
- new net N$20: D7.A, S7.SW2, S7.SW4
- new net N$21: D8.A, S8.SW2, S8.SW4
- new net N$22: D9.A, S9.SW2, S9.SW4
- new net N$23: D10.A, S10.SW2, S10.SW4
- new net N$24: D11.A, S11.SW2, S11.SW4
- new net N$25: D12.A, S12.SW2, S12.SW4
- new net N$26: D13.A, S13.SW2, S13.SW4
- new net N$27: D14.A, S14.SW2, S14.SW4
- new net N$28: D15.A, S15.SW2, S15.SW4
- new net N$29: D1.A, S1.SW2, S1.SW4
- new net N$30: D54.A, S54.SW2, S54.SW4
- new net N$31: D66.A, S66.SW2, S66.SW4
- new net N$32: D67.A, S67.SW2, S67.SW4
- new net N$37: D55.A, S55.SW2, S55.SW4
- new net N$38: D16.A, S16.SW2, S16.SW4
- new net N$39: D17.A, S17.SW2, S17.SW4
- new net N$40: D18.A, S18.SW2, S18.SW4
- new net N$41: D19.A, S19.SW2, S19.SW4
- new net N$42: D40.A, S40.SW2, S40.SW4
- new net N$43: D25.A, S25.SW2, S25.SW4
- new net N$45: D26.A, S26.SW2, S26.SW4
- new net N$48: D41.A, S41.SW2, S41.SW4
- new net N$49: D56.A, S56.SW2, S56.SW4
- new net N$52: D68.A, S68.SW2, S68.SW4
- new net N$53: D61.A, S61.SW2, S61.SW4
- new net N$54: D57.A, S57.SW2, S57.SW4
- new net N$56: D63.A, S63.SW2, S63.SW4
- new net N$57: D62.A, S62.SW2, S62.SW4
- new net N$58: D52.A, S52.SW2, S52.SW4
- new net N$59: D51.A, S51.SW2, S51.SW4
- new net N$60: D50.A, S50.SW2, S50.SW4
- new net N$62: D42.A, S42.SW2, S42.SW4
- new net N$64: D33.A, S33.SW2, S33.SW4
- new net N$65: D34.A, S34.SW2, S34.SW4
- new net N$66: D49.A, S49.SW2, S49.SW4
- new net N$67: D32.A, S32.SW2, S32.SW4
- new net N$68: D31.A, S31.SW2, S31.SW4
- new net N$71: D20.A, S20.SW2, S20.SW4
- new net N$72: D35.A, S35.SW2, S35.SW4
- new net N$73: D48.A, S48.SW2, S48.SW4
- new net N$76: D21.A, S21.SW2, S21.SW4
- new net N$77: D36.A, S36.SW2, S36.SW4
- new net N$79: D64.A, S64.SW2, S64.SW4
- new net N$80: D47.A, S47.SW2, S47.SW4
- new net N$81: D27.A, S27.SW2, S27.SW4
- new net N$84: D22.A, S22.SW2, S22.SW4
- new net N$85: D37.A, S37.SW2, S37.SW4
- new net N$88: D65.A, S65.SW2, S65.SW4
- new net N$89: D28.A, S28.SW2, S28.SW4
- new net N$91: D23.A, S23.SW2, S23.SW4
- new net N$92: D38.A, S38.SW2, S38.SW4
- new net N$93: D43.A, S43.SW2, S43.SW4
- new net N$96: D58.A, S58.SW2, S58.SW4
- new net N$97: D69.A, S69.SW2, S69.SW4
- new net N$98: D59.A, S59.SW2, S59.SW4
- new net N$99: D44.A, S44.SW2, S44.SW4
- new net R0: D1.C, D10.C, D11.C, D12.C, D13.C, D14.C, D15.C, D2.C, D3.C, D4.C, D5.C, D6.C, D7.C, D8.C, D9.C, U$1.18
- new net R1: D16.C, D17.C, D18.C, D19.C, D20.C, D21.C, D22.C, D23.C, D24.C, D25.C, D26.C, D27.C, D28.C, D29.C, D30.C, U$1.19
- new net R2: D31.C, D32.C, D33.C, D34.C, D35.C, D36.C, D37.C, D38.C, D39.C, D40.C, D41.C, D42.C, D43.C, D44.C, D45.C, U$1.20
- new net R3: D46.C, D47.C, D48.C, D49.C, D50.C, D51.C, D52.C, D53.C, D54.C, D55.C, D56.C, D57.C, D58.C, D59.C, D60.C, U$1.21
- new net R4: D61.C, D62.C, D63.C, D64.C, D65.C, D66.C, D67.C, D68.C, D69.C, D70.C, U$1.22
- new net SCK: IC3.3, IC4.3, U$1.9
- new net SS: IC3.30, IC4.30, U$1.8
- net GND: now also IC1.8, IC2.8, IC3.1, IC3.PAD, IC4.1, IC4.PAD, U$1.15, U$1.23, U$1.35, U$1.43, U$1.5; no longer IC1.1
- net N$12: now also IC3.29, IC4.4; no longer S1.LED2, S16.LED2, S31.LED2, S46.LED2, S61.LED2
- net N$13: now also D24.A, S24.SW2, S24.SW4; no longer S17.LED2, S2.LED2, S32.LED2, S47.LED2
- net N$14: now also D39.A, S39.SW2, S39.SW4; no longer S18.LED2, S3.LED2, S33.LED2, S48.LED2, S62.LED2
- net VCC: now also IC1.16, IC2.16; no longer IC1.32
Routing:
- net LED-A0: track 0.00 -> 298.8 mm
- net LED-A3: track 0.00 -> 298.8 mm
- net LED-A2: track 0.00 -> 298.8 mm
- net LED-A1: track 0.00 -> 298.7 mm
- net LED-A4: track 0.00 -> 283.3 mm
- net R1: track 0.00 -> 282.7 mm
- net R0: track 0.00 -> 278.8 mm
- net R3: track 0.00 -> 278.8 mm
- net R2: track 0.00 -> 278.8 mm
- net R4: track 0.00 -> 271.6 mm
- net C0: track 0.00 -> 107.6 mm
- net C2: track 0.00 -> 98.2 mm
- net LED-G0: track 0.00 -> 90.8 mm
- net LED-R0: track 0.00 -> 89.8 mm
- net LED-B0: track 0.00 -> 89.3 mm
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Other:
- board size 280 x 90 mm -> 285 x 95 mm

Commit message: Lots more work on main PCB
Parts:
- removed IC1, IC2: 74LS137D, 74xx-us:SO16
- added C1, C2: (no value), Jordi:C0603
- added C3, C4: 1uF, Jordi:C0603
- added C5, C6, C7, C8: 0.1uF, Jordi:C0603
- added D71, D72, D73, D74, D75: MOSFET-PSUPERSOT, Jordi:SUPERSOT-3
- added D76, D77, D78, D79, D80: (no value), Jordi:SOT23
- added J1: (no value), Jordi:M-1X04-0.1-PTH
- added J2: (no value), Jordi:M-1X06-0.05-PTH
- added R1: 1K, Jordi:R0603
- added R10, R16, R17, R18, R19, R20, R6, R7, R8, R9: 4.7k, Jordi:R0603
- added R11, R12, R13, R14, R15, R21, R22, R23, R24, R25: 100, Jordi:R0603
- added R2, R3: 22, Jordi:R0603
- added R4, R5: (no value), Jordi:R0603
- added S71: (no value), Jordi:SWITCH-TACTILE-SMD
- added U$2, U$3: 74LVC138AD, SparkFun-DigitalIC:SO016
- moved Y1 1.19 mm to (158.4, 5.95)
Connections:
- net MOSI renamed SIN
- removed net AL: IC1.4, IC2.4
- removed net E0: IC1.5, U$1.41
- removed net E1: IC2.6, U$1.40
- removed net MISO: U$1.11
- removed net SS: IC3.30, IC4.30, U$1.8
- removed net VCC: IC1.16, IC2.16
- new net !E1: U$1.1, U$2.4, U$3.4
- new net BLANK: IC3.2, IC4.2, U$1.8
- new net D+: R2.2, U$1.4
- new net D-: R3.2, U$1.3
- new net N$105: D76.1, R16.2, R21.2
- new net N$106: D78.1, R18.2, R23.2
- new net N$107: D79.1, R19.2, R24.2
- new net N$108: D80.1, R20.2, R25.2
- new net N$33: R1.2, U$1.33
- new net N$34: C3.2, U$1.6
- new net N$35: C5.2, U$1.42
- new net N$36: J1.2, R3.1
- new net N$44: J1.3, R2.1
- new net N$46: IC3.31, R4.1
- new net N$47: IC4.31, R5.1
- new net N$50: D71.1, R11.2, R6.1
- new net N$51: D71.3, S1.LED1, S10.LED1, S11.LED1, S12.LED1, S13.LED1, S14.LED1, S15.LED1, S2.LED1, S3.LED1, S4.LED1, S5.LED1, S6.LED1, S7.LED1, S8.LED1, S9.LED1
- new net N$55: D72.3, S16.LED1, S17.LED1, S18.LED1, S19.LED1, S20.LED1, S21.LED1, S22.LED1, S23.LED1, S24.LED1, S25.LED1, S26.LED1, S27.LED1, S28.LED1, S29.LED1, S30.LED1
- new net N$61: D73.3, S31.LED1, S32.LED1, S33.LED1, S34.LED1, S35.LED1, S36.LED1, S37.LED1, S38.LED1, S39.LED1, S40.LED1, S41.LED1, S42.LED1, S43.LED1, S44.LED1, S45.LED1
- new net N$63: D74.3, S46.LED1, S47.LED1, S48.LED1, S49.LED1, S50.LED1, S51.LED1, S52.LED1, S53.LED1, S54.LED1, S55.LED1, S56.LED1, S57.LED1, S58.LED1, S59.LED1, S60.LED1
- new net N$69: D75.1, R10.1, R15.2
- new net N$70: D74.1, R14.2, R9.1
- new net N$74: D73.1, R13.2, R8.1
- new net N$75: D72.1, R12.2, R7.1
- new net N$78: D75.3, S61.LED1, S62.LED1, S63.LED1, S64.LED1, S65.LED1, S66.LED1, S67.LED1, S68.LED1, S69.LED1, S70.LED1
- new net N$82: D76.2, R11.1
- new net N$83: D77.1, R17.2, R22.2
- new net N$87: D79.2, R14.1
- new net N$90: D78.2, R13.1
- new net N$94: D77.2, R12.1
- new net N$95: D80.2, R15.1
- new net RST: S71.3, S71.4, U$1.13
- new net RX: J2.4, U$1.20
- new net TX: J2.3, U$1.21
- new net UVCC: C4.2, U$1.2, U$1.7
- new net VIN: D71.2, D72.2, D73.2, D74.2, D75.2, J1.4, J2.5, R10.2, R6.2, R7.2, R8.2, R9.2
- new net XLAT: IC3.30, IC4.30, U$1.11
- net +3V3: now also C6.2, C7.2, C8.2, J2.6, U$2.16, U$2.6, U$3.16
- net A0: now also U$1.28, U$2.1, U$3.1; no longer IC1.1, IC2.1, U$1.39
- net A1: now also U$1.29, U$2.2, U$3.2; no longer IC1.2, IC2.2, U$1.38
- net A2: now also U$1.30, U$2.3, U$3.3; no longer IC1.3, IC2.3, U$1.37
- net A3: now also U$1.12, U$2.5, U$3.6; no longer IC1.6, IC2.5, U$1.36
- net C0: now also U$2.7; no longer IC1.7
- net C1: now also U$2.9; no longer IC1.9
- net C10: now also U$3.10; no longer IC2.10
- net C11: now also U$3.11; no longer IC2.11
- net C12: now also U$3.12; no longer IC2.12
- net C13: now also U$3.13; no longer IC2.13
- net C14: now also U$3.14; no longer IC2.14
- net C2: now also U$2.10; no longer IC1.10
- net C3: now also U$2.11; no longer IC1.11
- net C4: now also U$2.12; no longer IC1.12
- net C5: now also U$2.13; no longer IC1.13
- net C6: now also U$2.14; no longer IC1.14
- net C7: now also U$2.15; no longer IC1.15
- net C8: now also U$3.7; no longer IC2.7
- net C9: now also U$3.9; no longer IC2.9
- net GND: now also C1.1, C2.1, C3.1, C4.1, C5.1, C6.1, C7.1, C8.1, D76.3, D77.3, D78.3, D79.3, D80.3, J1.1, J2.1, R1.1, R16.1, R17.1, R18.1, R19.1, R20.1, R4.2, R5.2, S71.1, S71.2, U$2.8, U$3.5, U$3.8, Y1.2, Y1.4; no longer IC1.8, IC2.8
- net LED-A0: now also R21.1; no longer S1.LED1, S10.LED1, S11.LED1, S12.LED1, S13.LED1, S14.LED1, S15.LED1, S2.LED1, S3.LED1, S4.LED1, S5.LED1, S6.LED1, S7.LED1, S8.LED1, S9.LED1
- net LED-A1: now also R22.1; no longer S16.LED1, S17.LED1, S18.LED1, S19.LED1, S20.LED1, S21.LED1, S22.LED1, S23.LED1, S24.LED1, S25.LED1, S26.LED1, S27.LED1, S28.LED1, S29.LED1, S30.LED1
- net LED-A2: now also R23.1; no longer S31.LED1, S32.LED1, S33.LED1, S34.LED1, S35.LED1, S36.LED1, S37.LED1, S38.LED1, S39.LED1, S40.LED1, S41.LED1, S42.LED1, S43.LED1, S44.LED1, S45.LED1
- net LED-A3: now also R24.1; no longer S46.LED1, S47.LED1, S48.LED1, S49.LED1, S50.LED1, S51.LED1, S52.LED1, S53.LED1, S54.LED1, S55.LED1, S56.LED1, S57.LED1, S58.LED1, S59.LED1, S60.LED1
- net LED-A4: now also R25.1; no longer S61.LED1, S62.LED1, S63.LED1, S64.LED1, S65.LED1, S66.LED1, S67.LED1, S68.LED1, S69.LED1, S70.LED1
- net LED-B10: now also IC4.16
- net LED-B11: now also IC4.19
- net LED-B12: now also IC4.22
- net LED-B13: now also IC4.25
- net LED-B14: now also IC4.28
- net LED-B8: now also IC4.10
- net LED-B9: now also IC4.13
- net LED-G10: now also IC4.14
- net LED-G11: now also IC4.17
- net LED-G12: now also IC4.20
- net LED-G13: now also IC4.23
- net LED-G14: now also IC4.26
- net LED-G8: now also IC4.8
- net LED-G9: now also IC4.11
- net LED-R10: now also IC4.15
- net LED-R11: now also IC4.18
- net LED-R12: now also IC4.21
- net LED-R13: now also IC4.24
- net LED-R14: now also IC4.27
- net LED-R8: now also IC4.9
- net LED-R9: now also IC4.12
- net N$10: now also C2.2
- net N$9: now also C1.2
- net R0: no longer U$1.18
- net R1: no longer U$1.19
- net R2: no longer U$1.20
- net R3: no longer U$1.21
- net R4: no longer U$1.22
Routing:
- net N$51: track 0.00 -> 298.8 mm
- net LED-A0: track 298.8 -> 0.00 mm
- net N$63: track 0.00 -> 298.8 mm
- net N$61: track 0.00 -> 298.8 mm
- net LED-A3: track 298.8 -> 0.00 mm
- net LED-A2: track 298.8 -> 0.00 mm
- net N$55: track 0.00 -> 298.7 mm
- net LED-A1: track 298.7 -> 0.00 mm
- net N$78: track 0.00 -> 283.3 mm
- net LED-A4: track 283.3 -> 0.00 mm
- net C9: track 0.00 -> 109.5 mm
- net C12: track 0.00 -> 109.5 mm
- net C3: track 0.00 -> 109.5 mm
- net C6: track 0.00 -> 109.5 mm
- net C14: track 0.00 -> 98.2 mm
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
Commit message: Hardware debouncing and 5V VCC
Parts:
- added C10, C11, C12, C13, C14, C15, C16, C17, C18, C19, C20, C21, C22, C23, C24, C25, C26, C27, C28, C29, C30, C31, C32, C33, C34, C35, C36, C37, C38, C39, C40, C41, C42, C43, C44, C45, C46, C47, C48, C49, C50, C51, C52, C53, C54, C55, C56, C57, C58, C59, C60, C61, C62, C63, C64, C65, C66, C67, C68, C69, C70, C71, C72, C73, C74, C75, C76, C77, C78, C9: 1uF, Jordi:C0603
- added F1: 500mA, Jordi:FUSE-1812
- added IC1, IC10, IC11, IC12, IC13, IC14, IC15, IC16, IC17, IC18, IC19, IC2, IC20, IC21, IC22, IC23, IC24, IC25, IC26, IC27, IC28, IC29, IC30, IC31, IC32, IC33, IC34, IC35, IC36, IC37, IC38, IC39, IC40, IC41, IC42, IC43, IC44, IC45, IC46, IC47, IC48, IC49, IC5, IC50, IC51, IC52, IC53, IC54, IC55, IC56, IC57, IC58, IC59, IC6, IC60, IC61, IC62, IC63, IC64, IC65, IC66, IC67, IC68, IC69, IC7, IC70, IC71, IC72, IC8, IC9: 74LVC1G14DCK, 74xx-little-us:SC70-5
- added JP1, JP2, JP3, JP4: USB-MICROBSMD, Jordi:USB-MICRO-B-SMD
- added R100, R102, R104, R106, R108, R110, R112, R114, R116, R118, R120, R122, R124, R126, R128, R130, R132, R134, R136, R138, R140, R142, R144, R146, R148, R150, R152, R154, R156, R158, R160, R162, R164, R27, R28, R30, R32, R34, R36, R38, R40, R42, R44, R46, R48, R50, R52, R54, R56, R58, R60, R62, R64, R66, R68, R70, R72, R74, R76, R78, R80, R82, R84, R86, R88, R90, R92, R94, R96, R98: 4.7k?, Jordi:R0603
- added R101, R103, R105, R107, R109, R111, R113, R115, R117, R119, R121, R123, R125, R127, R129, R131, R133, R135, R137, R139, R141, R143, R145, R147, R149, R151, R153, R155, R157, R159, R161, R163, R165, R26, R29, R31, R33, R35, R37, R39, R41, R43, R45, R47, R49, R51, R53, R55, R57, R59, R61, R63, R65, R67, R69, R71, R73, R75, R77, R79, R81, R83, R85, R87, R89, R91, R93, R95, R97, R99: 22k?, Jordi:R0603
- J1: device Jordi:M-1X04-0.1-PTH -> Jordi:M-2X03-0.1-PTH-SHROUDED
- J2, S71: value (none) -> change
- R4, R5: value (none) -> 2.4k/3k
- moved R21 274.0 mm to (140.5, 83.9), flipped to the bottom
- moved R22 262.9 mm to (140.5, 64.9), flipped to the bottom
- moved R16 257.0 mm to (140.5, 85.7), flipped to the bottom
- moved R23 252.1 mm to (140.5, 45.8), flipped to the bottom
- moved R17 246.4 mm to (140.5, 66.7), flipped to the bottom
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Connections:
- removed net +3V3: C6.2, C7.2, C8.2, IC3.32, IC4.32, J2.6, U$1.14, U$1.24, U$1.34, U$1.44, U$2.16, U$2.6, U$3.16
- removed net C0: S1.SW1, S1.SW3, S16.SW1, S16.SW3, S31.SW1, S31.SW3, S46.SW1, S46.SW3, S61.SW1, S61.SW3, U$2.7
- removed net N$100: D29.A, S29.SW2, S29.SW4
- removed net N$101: D30.A, S30.SW2, S30.SW4
- removed net N$102: D45.A, S45.SW2, S45.SW4
- removed net N$103: D60.A, S60.SW2, S60.SW4
- removed net N$13: D24.A, S24.SW2, S24.SW4
- removed net N$14: D39.A, S39.SW2, S39.SW4
- removed net N$15: D53.A, S53.SW2, S53.SW4
- removed net N$16: D3.A, S3.SW2, S3.SW4
- removed net N$21: D8.A, S8.SW2, S8.SW4
- removed net N$30: D54.A, S54.SW2, S54.SW4
- removed net N$31: D66.A, S66.SW2, S66.SW4
- removed net N$32: D67.A, S67.SW2, S67.SW4
- removed net N$37: D55.A, S55.SW2, S55.SW4
- removed net N$38: D16.A, S16.SW2, S16.SW4
- removed net N$39: D17.A, S17.SW2, S17.SW4
- removed net N$40: D18.A, S18.SW2, S18.SW4
- removed net N$41: D19.A, S19.SW2, S19.SW4
- removed net N$42: D40.A, S40.SW2, S40.SW4
- removed net N$43: D25.A, S25.SW2, S25.SW4
- removed net N$45: D26.A, S26.SW2, S26.SW4
- removed net N$48: D41.A, S41.SW2, S41.SW4
- removed net N$49: D56.A, S56.SW2, S56.SW4
- removed net N$52: D68.A, S68.SW2, S68.SW4
- removed net N$53: D61.A, S61.SW2, S61.SW4
- removed net N$54: D57.A, S57.SW2, S57.SW4
- removed net N$56: D63.A, S63.SW2, S63.SW4
- removed net N$57: D62.A, S62.SW2, S62.SW4
- removed net N$58: D52.A, S52.SW2, S52.SW4
- removed net N$59: D51.A, S51.SW2, S51.SW4
- removed net N$60: D50.A, S50.SW2, S50.SW4
- removed net N$62: D42.A, S42.SW2, S42.SW4
- removed net N$64: D33.A, S33.SW2, S33.SW4
- removed net N$65: D34.A, S34.SW2, S34.SW4
- removed net N$66: D49.A, S49.SW2, S49.SW4
- removed net N$67: D32.A, S32.SW2, S32.SW4
- removed net N$68: D31.A, S31.SW2, S31.SW4
- removed net N$71: D20.A, S20.SW2, S20.SW4
- removed net N$72: D35.A, S35.SW2, S35.SW4
- removed net N$73: D48.A, S48.SW2, S48.SW4
- removed net N$76: D21.A, S21.SW2, S21.SW4
- removed net N$77: D36.A, S36.SW2, S36.SW4
- removed net N$79: D64.A, S64.SW2, S64.SW4
- removed net N$80: D47.A, S47.SW2, S47.SW4
- removed net N$81: D27.A, S27.SW2, S27.SW4
- removed net N$84: D22.A, S22.SW2, S22.SW4
- removed net N$85: D37.A, S37.SW2, S37.SW4
- removed net N$86: D46.A, S46.SW2, S46.SW4
- removed net N$88: D65.A, S65.SW2, S65.SW4
- removed net N$89: D28.A, S28.SW2, S28.SW4
- removed net N$91: D23.A, S23.SW2, S23.SW4
- removed net N$92: D38.A, S38.SW2, S38.SW4
- removed net N$93: D43.A, S43.SW2, S43.SW4
- removed net N$96: D58.A, S58.SW2, S58.SW4
- removed net N$97: D69.A, S69.SW2, S69.SW4
- removed net N$98: D59.A, S59.SW2, S59.SW4
- removed net N$99: D44.A, S44.SW2, S44.SW4
- removed net SIN: IC3.4, U$1.10
- removed net VIN: D71.2, D72.2, D73.2, D74.2, D75.2, J1.4, J2.5, R10.2, R6.2, R7.2, R8.2, R9.2
- new net !C0: C24.1, C39.1, C54.1, C69.1, C9.1, S1.SW1, S1.SW3, S16.SW1, S16.SW3, S31.SW1, S31.SW3, S46.SW1, S46.SW3, S61.SW1, S61.SW3, U$2.7
- new net !C1: C10.1, C25.1, C40.1, C55.1, S17.SW1, S17.SW3, S2.SW1, S2.SW3, S32.SW1, S32.SW3, S47.SW1, S47.SW3
- new net !C10: C19.1, C34.1, C49.1, C64.1, S11.SW1, S11.SW3, S26.SW1, S26.SW3, S41.SW1, S41.SW3, S56.SW1, S56.SW3
- new net !C11: C20.1, C35.1, C50.1, C65.1, S12.SW1, S12.SW3, S27.SW1, S27.SW3, S42.SW1, S42.SW3, S57.SW1, S57.SW3, S68.SW1, S68.SW3
- new net !C12: C21.1, C36.1, C51.1, C66.1, C77.1, S13.SW1, S13.SW3, S28.SW1, S28.SW3, S43.SW1, S43.SW3, S58.SW1, S58.SW3, S69.SW1, S69.SW3
- new net !C13: C22.1, C37.1, C52.1, C67.1, S14.SW1, S14.SW3, S29.SW1, S29.SW3, S44.SW1, S44.SW3, S59.SW1, S59.SW3
- new net !C14: C23.1, C38.1, C53.1, C68.1, S15.SW1, S15.SW3, S30.SW1, S30.SW3, S45.SW1, S45.SW3, S60.SW1, S60.SW3, S70.SW1, S70.SW3
- new net !C2: C11.1, C26.1, C41.1, C56.1, S18.SW1, S18.SW3, S3.SW1, S3.SW3, S33.SW1, S33.SW3, S48.SW1, S48.SW3, S62.SW1, S62.SW3
- new net !C3: C12.1, C27.1, C42.1, C57.1, C71.1, S19.SW1, S19.SW3, S34.SW1, S34.SW3, S4.SW1, S4.SW3, S49.SW1, S49.SW3, S63.SW1, S63.SW3
- new net !C4: C13.1, C28.1, C43.1, C58.1, S20.SW1, S20.SW3, S35.SW1, S35.SW3, S5.SW1, S5.SW3, S50.SW1, S50.SW3
- new net !C5: C14.1, C29.1, C44.1, C59.1, S21.SW1, S21.SW3, S36.SW1, S36.SW3, S51.SW1, S51.SW3, S6.SW1, S6.SW3, S64.SW1, S64.SW3
- new net !C6: C15.1, C30.1, C45.1, C60.1, C73.1, S22.SW1, S22.SW3, S37.SW1, S37.SW3, S52.SW1, S52.SW3, S65.SW1, S65.SW3, S7.SW1, S7.SW3
- new net !C7: C16.1, C31.1, C46.1, C61.1, S23.SW1, S23.SW3, S38.SW1, S38.SW3, S53.SW1, S53.SW3, S8.SW1, S8.SW3
- new net !C8: C17.1, C32.1, C47.1, C62.1, S24.SW1, S24.SW3, S39.SW1, S39.SW3, S54.SW1, S54.SW3, S66.SW1, S66.SW3, S9.SW1, S9.SW3
- new net !C9: C18.1, C33.1, C48.1, C63.1, C75.1, S10.SW1, S10.SW3, S25.SW1, S25.SW3, S40.SW1, S40.SW3, S55.SW1, S55.SW3, S67.SW1, S67.SW3
- new net !COL: C9.2, IC1.2, R26.1
- new net !COL1: C10.2, IC2.2, R29.1
- new net !COL10: C19.2, IC13.2, R47.1
- new net !COL11: C20.2, IC14.2, R49.1
- new net !COL12: C21.2, IC15.2, R51.1
- new net !COL13: C22.2, IC16.2, R53.1
- new net !COL14: C23.2, IC17.2, R55.1
- new net !COL15: C24.2, IC18.2, R57.1
- new net !COL16: C25.2, IC19.2, R59.1
- new net !COL17: C26.2, IC20.2, R61.1
- new net !COL18: C27.2, IC21.2, R63.1
- new net !COL19: C28.2, IC22.2, R65.1
- new net !COL2: C11.2, IC5.2, R31.1
- new net !COL20: C29.2, IC23.2, R67.1
- new net !COL21: C30.2, IC24.2, R69.1
- new net !COL22: C31.2, IC25.2, R71.1
- new net !COL23: C32.2, IC26.2, R73.1
- new net !COL24: C33.2, IC27.2, R75.1
- new net !COL25: C34.2, IC28.2, R77.1
- new net !COL26: C35.2, IC29.2, R79.1
- new net !COL27: C36.2, IC30.2, R81.1
- new net !COL28: C37.2, IC31.2, R83.1
- new net !COL29: C38.2, IC32.2, R85.1
- new net !COL3: C12.2, IC6.2, R33.1
- new net !COL30: C39.2, IC33.2, R87.1
- new net !COL31: C40.2, IC34.2, R89.1
- new net !COL32: C41.2, IC35.2, R91.1
- new net !COL33: C42.2, IC36.2, R93.1
- new net !COL34: C43.2, IC37.2, R95.1
- new net !COL35: C44.2, IC38.2, R97.1
- new net !COL36: C45.2, IC39.2, R99.1
- new net !COL37: C46.2, IC40.2, R101.1
- new net !COL38: C47.2, IC41.2, R103.1
- new net !COL39: C48.2, IC42.2, R105.1
- new net !COL4: C13.2, IC7.2, R35.1
- new net !COL40: C49.2, IC43.2, R107.1
- new net !COL41: C50.2, IC44.2, R109.1
- new net !COL42: C51.2, IC45.2, R111.1
- new net !COL43: C52.2, IC46.2, R113.1
- new net !COL44: C53.2, IC47.2, R115.1
- new net !COL45: C54.2, IC48.2, R117.1
- new net !COL46: C55.2, IC49.2, R119.1
- new net !COL47: C56.2, IC50.2, R121.1
- new net !COL48: C57.2, IC51.2, R123.1
- new net !COL49: C58.2, IC52.2, R125.1
- new net !COL5: C14.2, IC8.2, R37.1
- new net !COL50: C59.2, IC53.2, R127.1
- new net !COL51: C60.2, IC54.2, R129.1
- new net !COL52: C61.2, IC55.2, R131.1
- new net !COL53: C62.2, IC56.2, R133.1
- new net !COL54: C63.2, IC57.2, R135.1
- new net !COL55: C64.2, IC58.2, R137.1
- new net !COL56: C65.2, IC59.2, R139.1
- new net !COL57: C66.2, IC60.2, R141.1
- new net !COL58: C67.2, IC61.2, R143.1
- new net !COL59: C68.2, IC62.2, R145.1
- new net !COL6: C15.2, IC9.2, R39.1
- new net !COL60: C69.2, IC63.2, R147.1
- new net !COL61: C70.2, IC64.2, R149.1
- new net !COL62: C71.2, IC65.2, R151.1
- new net !COL63: C72.2, IC66.2, R153.1
- new net !COL64: C73.2, IC67.2, R155.1
- new net !COL65: C74.2, IC68.2, R157.1
- new net !COL66: C75.2, IC69.2, R159.1
- new net !COL67: C76.2, IC70.2, R161.1
- new net !COL68: C77.2, IC71.2, R163.1
- new net !COL69: C78.2, IC72.2, R165.1
- new net !COL7: C16.2, IC10.2, R41.1
- new net !COL8: C17.2, IC11.2, R43.1
- new net !COL9: C18.2, IC12.2, R45.1
- new net +5V: C6.2, C7.2, C8.2, D71.2, D72.2, D73.2, D74.2, D75.2, F1.2, IC1.5, IC10.5, IC11.5, IC12.5, IC13.5, IC14.5, IC15.5, IC16.5, IC17.5, IC18.5, IC19.5, IC2.5, IC20.5, IC21.5, IC22.5, IC23.5, IC24.5, IC25.5, IC26.5, IC27.5, IC28.5, IC29.5, IC3.32, IC30.5, IC31.5, IC32.5, IC33.5, IC34.5, IC35.5, IC36.5, IC37.5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
- new net MISO: J1.1, U$1.11
- new net MOSI: IC3.4, J1.4, U$1.10
- new net N$109: IC16.4
- new net N$110: IC17.4
- new net N$112: IC18.4
- new net N$113: IC19.4
- new net N$114: IC20.4
- new net N$115: IC21.4
- new net N$116: IC22.4
- new net N$117: IC23.4
- new net N$118: IC24.4
- new net N$119: IC25.4
- new net N$120: IC26.4
- new net N$121: IC27.4
- new net N$122: IC28.4
- new net N$123: IC29.4
- new net N$124: IC30.4
- new net N$125: IC31.4
- new net N$126: IC32.4
- new net N$130: IC33.4
- new net N$131: IC34.4
- new net N$132: IC35.4
- new net N$133: IC36.4
- new net N$134: IC37.4
- new net N$135: IC38.4
- new net N$136: IC39.4
- new net N$137: IC40.4
- new net N$138: IC41.4
- new net N$139: IC42.4
- new net N$140: IC43.4
- new net N$141: IC44.4
- new net N$142: IC45.4
- new net N$143: IC46.4
- new net N$144: IC47.4
- new net N$148: IC48.4
- new net N$149: IC49.4
- new net N$150: IC50.4
- new net N$151: IC51.4
- new net N$152: IC52.4
- new net N$153: IC53.4
- new net N$154: IC54.4
- new net N$155: IC55.4
- new net N$156: IC56.4
- new net N$157: IC57.4
- new net N$158: IC58.4
- new net N$159: IC59.4
- new net N$160: IC60.4
- new net N$161: IC61.4
- new net N$162: IC62.4
- new net N$166: IC63.4
- new net N$167: IC64.4
- new net N$168: IC65.4
- new net N$169: IC66.4
- new net N$170: IC67.4
- new net N$171: IC68.4
- new net N$172: IC69.4
- new net N$173: IC70.4
- new net N$174: IC71.4
- new net N$175: IC72.4
- new net SW1: D1.A, R26.2, R27.1, S1.SW2, S1.SW4
- new net SW10: D10.A, R44.1, R45.2, S10.SW2, S10.SW4
- new net SW11: D11.A, R46.1, R47.2, S11.SW2, S11.SW4
- new net SW12: D12.A, R48.1, R49.2, S12.SW2, S12.SW4
- new net SW13: D13.A, R50.1, R51.2, S13.SW2, S13.SW4
- new net SW14: D14.A, R52.1, R53.2, S14.SW2, S14.SW4
- new net SW15: D15.A, R54.1, R55.2, S15.SW2, S15.SW4
- new net SW16: D16.A, R56.1, R57.2, S16.SW2, S16.SW4
- new net SW17: D17.A, R58.1, R59.2, S17.SW2, S17.SW4
- new net SW18: D18.A, R60.1, R61.2, S18.SW2, S18.SW4
- new net SW19: D19.A, R62.1, R63.2, S19.SW2, S19.SW4
- new net SW2: D2.A, R28.1, R29.2, S2.SW2, S2.SW4
- new net SW20: D20.A, R64.1, R65.2, S20.SW2, S20.SW4
- new net SW21: D21.A, R66.1, R67.2, S21.SW2, S21.SW4
- new net SW22: D22.A, R68.1, R69.2, S22.SW2, S22.SW4
- new net SW23: D23.A, R70.1, R71.2, S23.SW2, S23.SW4
- new net SW24: D24.A, R72.1, R73.2, S24.SW2, S24.SW4
- new net SW25: D25.A, R74.1, R75.2, S25.SW2, S25.SW4
- new net SW26: D26.A, R76.1, R77.2, S26.SW2, S26.SW4
- new net SW27: D27.A, R78.1, R79.2, S27.SW2, S27.SW4
- new net SW28: D28.A, R80.1, R81.2, S28.SW2, S28.SW4
- new net SW29: D29.A, R82.1, R83.2, S29.SW2, S29.SW4
- new net SW3: D3.A, R30.1, R31.2, S3.SW2, S3.SW4
- new net SW30: D30.A, R84.1, R85.2, S30.SW2, S30.SW4
- new net SW31: D31.A, R86.1, R87.2, S31.SW2, S31.SW4
- new net SW32: D32.A, R88.1, R89.2, S32.SW2, S32.SW4
- new net SW33: D33.A, R90.1, R91.2, S33.SW2, S33.SW4
- new net SW34: D34.A, R92.1, R93.2, S34.SW2, S34.SW4
- new net SW35: D35.A, R94.1, R95.2, S35.SW2, S35.SW4
- new net SW36: D36.A, R96.1, R97.2, S36.SW2, S36.SW4
- new net SW37: D37.A, R98.1, R99.2, S37.SW2, S37.SW4
- new net SW38: D38.A, R100.1, R101.2, S38.SW2, S38.SW4
- new net SW39: D39.A, R102.1, R103.2, S39.SW2, S39.SW4
- new net SW4: D4.A, R32.1, R33.2, S4.SW2, S4.SW4
- new net SW40: D40.A, R104.1, R105.2, S40.SW2, S40.SW4
- new net SW41: D41.A, R106.1, R107.2, S41.SW2, S41.SW4
- new net SW42: D42.A, R108.1, R109.2, S42.SW2, S42.SW4
- new net SW43: D43.A, R110.1, R111.2, S43.SW2, S43.SW4
- new net SW44: D44.A, R112.1, R113.2, S44.SW2, S44.SW4
- new net SW45: D45.A, R114.1, R115.2, S45.SW2, S45.SW4
- new net SW46: D46.A, R116.1, R117.2, S46.SW2, S46.SW4
- new net SW47: D47.A, R118.1, R119.2, S47.SW2, S47.SW4
- new net SW48: D48.A, R120.1, R121.2, S48.SW2, S48.SW4
- new net SW49: D49.A, R122.1, R123.2, S49.SW2, S49.SW4
- new net SW5: D5.A, R34.1, R35.2, S5.SW2, S5.SW4
- new net SW50: D50.A, R124.1, R125.2, S50.SW2, S50.SW4
- new net SW51: D51.A, R126.1, R127.2, S51.SW2, S51.SW4
- new net SW52: D52.A, R128.1, R129.2, S52.SW2, S52.SW4
- new net SW53: D53.A, R130.1, R131.2, S53.SW2, S53.SW4
- new net SW54: D54.A, R132.1, R133.2, S54.SW2, S54.SW4
- new net SW55: D55.A, R134.1, R135.2, S55.SW2, S55.SW4
- new net SW56: D56.A, R136.1, R137.2, S56.SW2, S56.SW4
- new net SW57: D57.A, R138.1, R139.2, S57.SW2, S57.SW4
- new net SW58: D58.A, R140.1, R141.2, S58.SW2, S58.SW4
- new net SW59: D59.A, R142.1, R143.2, S59.SW2, S59.SW4
- new net SW6: D6.A, R36.1, R37.2, S6.SW2, S6.SW4
- new net SW60: D60.A, R144.1, R145.2, S60.SW2, S60.SW4
- new net SW61: D61.A, R146.1, R147.2, S61.SW2, S61.SW4
- new net SW62: D62.A, R148.1, R149.2, S62.SW2, S62.SW4
- new net SW63: D63.A, R150.1, R151.2, S63.SW2, S63.SW4
- new net SW64: D64.A, R152.1, R153.2, S64.SW2, S64.SW4
- new net SW65: D65.A, R154.1, R155.2, S65.SW2, S65.SW4
- new net SW66: D66.A, R156.1, R157.2, S66.SW2, S66.SW4
- new net SW67: D67.A, R158.1, R159.2, S67.SW2, S67.SW4
- new net SW68: D68.A, R160.1, R161.2, S68.SW2, S68.SW4
- new net SW69: D69.A, R162.1, R163.2, S69.SW2, S69.SW4
- new net SW7: D7.A, R38.1, R39.2, S7.SW2, S7.SW4
- new net SW70: D70.A, R164.1, R165.2, S70.SW2, S70.SW4
- new net SW8: D8.A, R40.1, R41.2, S8.SW2, S8.SW4
- new net SW9: D9.A, R42.1, R43.2, S9.SW2, S9.SW4
- net C1: no longer S17.SW1, S17.SW3, S2.SW1, S2.SW3, S32.SW1, S32.SW3, S47.SW1, S47.SW3
- net C10: no longer S11.SW1, S11.SW3, S26.SW1, S26.SW3, S41.SW1, S41.SW3, S56.SW1, S56.SW3
- net C11: no longer S12.SW1, S12.SW3, S27.SW1, S27.SW3, S42.SW1, S42.SW3, S57.SW1, S57.SW3, S68.SW1, S68.SW3
- net C12: no longer S13.SW1, S13.SW3, S28.SW1, S28.SW3, S43.SW1, S43.SW3, S58.SW1, S58.SW3, S69.SW1, S69.SW3
- net C13: no longer S14.SW1, S14.SW3, S29.SW1, S29.SW3, S44.SW1, S44.SW3, S59.SW1, S59.SW3
- net C14: no longer S15.SW1, S15.SW3, S30.SW1, S30.SW3, S45.SW1, S45.SW3, S60.SW1, S60.SW3, S70.SW1, S70.SW3
- net C2: no longer S18.SW1, S18.SW3, S3.SW1, S3.SW3, S33.SW1, S33.SW3, S48.SW1, S48.SW3, S62.SW1, S62.SW3
- net C3: no longer S19.SW1, S19.SW3, S34.SW1, S34.SW3, S4.SW1, S4.SW3, S49.SW1, S49.SW3, S63.SW1, S63.SW3
- net C4: no longer S20.SW1, S20.SW3, S35.SW1, S35.SW3, S5.SW1, S5.SW3, S50.SW1, S50.SW3
- net C5: no longer S21.SW1, S21.SW3, S36.SW1, S36.SW3, S51.SW1, S51.SW3, S6.SW1, S6.SW3, S64.SW1, S64.SW3
- net C6: no longer S22.SW1, S22.SW3, S37.SW1, S37.SW3, S52.SW1, S52.SW3, S65.SW1, S65.SW3, S7.SW1, S7.SW3
- net C7: no longer S23.SW1, S23.SW3, S38.SW1, S38.SW3, S53.SW1, S53.SW3, S8.SW1, S8.SW3
- net C8: no longer S24.SW1, S24.SW3, S39.SW1, S39.SW3, S54.SW1, S54.SW3, S66.SW1, S66.SW3, S9.SW1, S9.SW3
- net C9: no longer S10.SW1, S10.SW3, S25.SW1, S25.SW3, S40.SW1, S40.SW3, S55.SW1, S55.SW3, S67.SW1, S67.SW3
- net D+: now also JP1.D+, JP2.D+, JP3.D+, JP4.D+, R2.1; no longer R2.2, U$1.4
- net D-: now also JP1.D-, JP2.D-, JP3.D-, JP4.D-, R3.1; no longer R3.2, U$1.3
- net GND: now also IC1.3, IC10.3, IC11.3, IC12.3, IC13.3, IC14.3, IC15.3, IC16.3, IC17.3, IC18.3, IC19.3, IC2.3, IC20.3, IC21.3, IC22.3, IC23.3, IC24.3, IC25.3, IC26.3, IC27.3, IC28.3, IC29.3, IC30.3, IC31.3, IC32.3, IC33.3, IC34.3, IC35.3, IC36.3, IC37.3, IC38.3, IC39.3, IC40.3, IC41.3, IC42.3, IC43.3, IC44.3, IC45.3, IC46.3, IC47.3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; no longer J1.1
- net LED-G11: now also C76.1
- net LED-G14: now also C78.1
- net LED-G2: now also C70.1
- net LED-G5: now also C72.1
- net LED-G8: now also C74.1
- net N$104: now also IC15.4; no longer D70.A, S70.SW2, S70.SW4
- net N$11: now also F1.1, JP1.VBUS, JP2.VBUS, JP3.VBUS, JP4.VBUS; no longer D2.A, S2.SW2, S2.SW4
- net N$17: now also IC1.4; no longer D4.A, S4.SW2, S4.SW4
- net N$18: now also IC2.4; no longer D5.A, S5.SW2, S5.SW4
- net N$19: now also IC5.4; no longer D6.A, S6.SW2, S6.SW4
- net N$20: now also IC6.4; no longer D7.A, S7.SW2, S7.SW4
- net N$22: now also IC7.4; no longer D9.A, S9.SW2, S9.SW4
- net N$23: now also IC8.4; no longer D10.A, S10.SW2, S10.SW4
- net N$24: now also IC9.4; no longer D11.A, S11.SW2, S11.SW4
- net N$25: now also IC10.4; no longer D12.A, S12.SW2, S12.SW4
- net N$26: now also IC11.4; no longer D13.A, S13.SW2, S13.SW4
- net N$27: now also IC12.4; no longer D14.A, S14.SW2, S14.SW4
- net N$28: now also IC13.4; no longer D15.A, S15.SW2, S15.SW4
- net N$29: now also IC14.4; no longer D1.A, S1.SW2, S1.SW4
- net N$36: now also R2.2, U$1.4; no longer J1.2, R3.1
- net N$44: now also R3.2, U$1.3; no longer J1.3, R2.1
- net RST: now also J1.5
- net SCK: now also J1.3
- net XLAT: no longer U$1.11
Routing:
- net !C0: track 0.00 -> 118.1 mm
- net C9: track 109.5 -> 0.00 mm
- net !C9: track 0.00 -> 109.5 mm
- net C12: track 109.5 -> 0.00 mm
- net !C12: track 0.00 -> 109.5 mm
- net C3: track 109.5 -> 0.00 mm
- net !C3: track 0.00 -> 109.5 mm
- net C6: track 109.5 -> 0.00 mm
- net !C6: track 0.00 -> 109.5 mm
- net C0: track 107.6 -> 0.00 mm
- net C14: track 98.2 -> 0.00 mm
- net !C14: track 0.00 -> 98.2 mm
- net C8: track 98.2 -> 0.00 mm
- net !C8: track 0.00 -> 98.2 mm
- net C5: track 98.2 -> 0.00 mm
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
Commit message: Back to 3V3 because LiPo
Parts:
- added C81: 470pF, Jordi:C0603
- added C82: 1uF, Jordi:C0603
- added D81: BAT20J, SparkFun-DiscreteSemi:SOD-323
- added IC73: VREG-5SOT23, Jordi:SOT23-5
- added J3: (no value), Jordi:M-1X06-0.1-PTH
- added Q1: MOSFET-PSUPERSOT, Jordi:SUPERSOT-3
- added R168: 100K, Jordi:R0603
- added USB: (no value), Jordi:M-1X04-0.1-PTH
- R4, R5: value 2.4k/3k -> 4.7k/5.1k
- moved F1 153.4 mm to (156.6, 20.2), flipped to the bottom, turned to 270 degrees
- moved C8 35.3 mm to (182.8, 5.36), turned to 270 degrees
- moved C7 33.0 mm to (181.0, 5.36), turned to 270 degrees
- moved C6 30.7 mm to (179.2, 5.36), turned to 270 degrees
- moved C4 28.5 mm to (177.4, 5.36), turned to 270 degrees
- moved C5 26.3 mm to (175.6, 5.36), turned to 270 degrees
- moved C3 24.2 mm to (173.8, 5.36), turned to 270 degrees
- moved R155 4.65 mm to (138.7, 13.1), turned to 90 degrees
- moved R154 2.98 mm to (141.1, 17.3), turned to 180 degrees
- moved J1 2.38 mm to (178.6, 11.9)
- moved R4 1.79 mm to (92.9, 5.36)
- moved R5 1.79 mm to (207.2, 5.36)
Connections:
- removed net +5V: C6.2, C7.2, C8.2, D71.2, D72.2, D73.2, D74.2, D75.2, F1.2, IC1.5, IC10.5, IC11.5, IC12.5, IC13.5, IC14.5, IC15.5, IC16.5, IC17.5, IC18.5, IC19.5, IC2.5, IC20.5, IC21.5, IC22.5, IC23.5, IC24.5, IC25.5, IC26.5, IC27.5, IC28.5, IC29.5, IC3.32, IC30.5, IC31.5, IC32.5, IC33.5, IC34.5, IC35.5, IC36.5, IC37.5, IC38.5, IC39.5, IC4.32, IC40.5, IC41.5, IC42.5, IC43.5, IC44.5, IC45.5, IC46.5, IC47.5, IC48.5, IC49.5, IC5.5, IC50.5, IC51.5, IC52.5, IC53.5, IC54.5, IC55.5, IC56.5, IC57.5, IC58.5, IC59.5, IC6.5, IC60.5, IC61.5, IC62.5, IC63.5, IC64.5, IC65.5, IC66.5, IC67.5, IC68.5, IC69.5, IC7.5, IC70.5, IC71.5, IC72.5, IC8.5, IC9.5, J1.2, J2.6, R10.2, R100.2, R102.2, R104.2, R106.2, R108.2, R110.2, R112.2, R114.2, R116.2, R118.2, R120.2, R122.2, R124.2, R126.2, R128.2, R130.2, R132.2, R134.2, R136.2, R138.2, R140.2, R142.2, R144.2, R146.2, R148.2, R150.2, R152.2, R154.2, R156.2, R158.2, R160.2, R162.2, R164.2, R27.2, R28.2, R30.2, R32.2, R34.2, R36.2, R38.2, R40.2, R42.2, R44.2, R46.2, R48.2, R50.2, R52.2, R54.2, R56.2, R58.2, R6.2, R60.2, R62.2, R64.2, R66.2, R68.2, R7.2, R70.2, R72.2, R74.2, R76.2, R78.2, R8.2, R80.2, R82.2, R84.2, R86.2, R88.2, R9.2, R90.2, R92.2, R94.2, R96.2, R98.2, U$1.14, U$1.24, U$1.34, U$1.44, U$2.16, U$2.6, U$3.16
- new net +3V3: C6.2, C7.2, C8.2, IC1.5, IC10.5, IC11.5, IC12.5, IC13.5, IC14.5, IC15.5, IC16.5, IC17.5, IC18.5, IC19.5, IC2.5, IC20.5, IC21.5, IC22.5, IC23.5, IC24.5, IC25.5, IC26.5, IC27.5, IC28.5, IC29.5, IC3.32, IC30.5, IC31.5, IC32.5, IC33.5, IC34.5, IC35.5, IC36.5, IC37.5, IC38.5, IC39.5, IC4.32, IC40.5, IC41.5, IC42.5, IC43.5, IC44.5, IC45.5, IC46.5, IC47.5, IC48.5, IC49.5, IC5.5, IC50.5, IC51.5, IC52.5, IC53.5, IC54.5, IC55.5, IC56.5, IC57.5, IC58.5, IC59.5, IC6.5, IC60.5, IC61.5, IC62.5, IC63.5, IC64.5, IC65.5, IC66.5, IC67.5, IC68.5, IC69.5, IC7.5, IC70.5, IC71.5, IC72.5, IC73.4, IC8.5, IC9.5, J1.2, J2.6, R100.2, R102.2, R104.2, R106.2, R108.2, R110.2, R112.2, R114.2, R116.2, R118.2, R120.2, R122.2, R124.2, R126.2, R128.2, R130.2, R132.2, R134.2, R136.2, R138.2, R140.2, R142.2, R144.2, R146.2, R148.2, R150.2, R152.2, R154.2, R156.2, R158.2, R160.2, R162.2, R164.2, R27.2, R28.2, R30.2, R32.2, R34.2, R36.2, R38.2, R40.2, R42.2, R44.2, R46.2, R48.2, R50.2, R52.2, R54.2, R56.2, R58.2, R60.2, R62.2, R64.2, R66.2, R68.2, R70.2, R72.2, R74.2, R76.2, R78.2, R80.2, R82.2, R84.2, R86.2, R88.2, R90.2, R92.2, R94.2, R96.2, R98.2, U$1.14, U$1.24, U$1.34, U$1.44, U$2.16, U$2.6, U$3.16
- new net N$14: C81.1, IC73.3
- new net SOUT: IC4.29, J3.6
- new net VBAT: J2.2, Q1.3
- new net VCC: C82.2, D81.C, IC73.1, IC73.5, Q1.2
- new net VIN: D71.2, D72.2, D73.2, D74.2, D75.2, D81.A, F1.2, J2.5, Q1.1, R10.2, R168.2, R6.2, R7.2, R8.2, R9.2, USB.4
- net D+: now also USB.3
- net D-: now also USB.2
- net GND: now also C81.2, C82.1, IC73.2, R168.1, USB.1
- net LED-A0: now also J3.1
- net LED-A1: now also J3.2
- net LED-A2: now also J3.3
- net LED-A3: now also J3.4
- net LED-A4: now also J3.5
Routing:
- net N$78: track 283.3 -> 297.6 mm
- net +5V: track 1.14 -> 0.00 mm
- net +3V3: track 0.00 -> 1.14 mm

Commit message: More work, maybe removing RGB LEDs after this
Connections:
- removed net C1: U$2.9
- removed net C10: U$3.10
- removed net C11: U$3.11
- removed net C12: U$3.12
- removed net C13: U$3.13
- removed net C14: U$3.14
- removed net C2: U$2.10
- removed net C3: U$2.11
- removed net C4: U$2.12
- removed net C5: U$2.13
- removed net C6: U$2.14
- removed net C7: U$2.15
- removed net C8: U$3.7
- removed net C9: U$3.9
- net !C1: now also U$2.9
- net !C10: now also U$3.10
- net !C11: now also U$3.11
- net !C12: now also U$3.12
- net !C13: now also U$3.13
- net !C14: now also U$3.14
- net !C2: now also U$2.10
- net !C3: now also U$2.11
- net !C4: now also U$2.12
- net !C5: now also U$2.13
- net !C6: now also U$2.14
- net !C7: now also U$2.15
- net !C8: now also U$3.7
- net !C9: now also U$3.9
