File: hardware/ION-60/Eagle/ION-60/ION-60.brd (EAGLE design)
At the start: 285 x 95 mm, 485 parts, among them IC1 74LVC1G14DCK, IC10 74LVC1G14DCK, IC11 74LVC1G14DCK, IC12 74LVC1G14DCK, IC13 74LVC1G14DCK, IC14 74LVC1G14DCK, IC15 74LVC1G14DCK, IC16 74LVC1G14DCK, IC17 74LVC1G14DCK, IC18 74LVC1G14DCK, IC19 74LVC1G14DCK, IC2 74LVC1G14DCK, IC20 74LVC1G14DCK, IC21 74LVC1G14DCK, IC22 74LVC1G14DCK, IC23 74LVC1G14DCK, IC24 74LVC1G14DCK, IC25 74LVC1G14DCK, IC26 74LVC1G14DCK, IC27 74LVC1G14DCK, IC28 74LVC1G14DCK, IC29 74LVC1G14DCK, IC3 TLC5947DAP, IC30 74LVC1G14DCK, IC31 74LVC1G14DCK, IC32 74LVC1G14DCK, IC33 74LVC1G14DCK, IC34 74LVC1G14DCK, IC35 74LVC1G14DCK, IC36 74LVC1G14DCK, IC37 74LVC1G14DCK, IC38 74LVC1G14DCK, IC39 74LVC1G14DCK, IC4 TLC5947DAP, IC40 74LVC1G14DCK, IC41 74LVC1G14DCK, IC42 74LVC1G14DCK, IC43 74LVC1G14DCK, IC44 74LVC1G14DCK, IC45 74LVC1G14DCK, IC46 74LVC1G14DCK, IC47 74LVC1G14DCK, IC48 74LVC1G14DCK, IC49 74LVC1G14DCK, IC5 74LVC1G14DCK, IC50 74LVC1G14DCK, IC51 74LVC1G14DCK, IC52 74LVC1G14DCK, IC53 74LVC1G14DCK, IC54 74LVC1G14DCK, IC55 74LVC1G14DCK, IC56 74LVC1G14DCK, IC57 74LVC1G14DCK, IC58 74LVC1G14DCK, IC59 74LVC1G14DCK, IC6 74LVC1G14DCK, IC60 74LVC1G14DCK, IC61 74LVC1G14DCK, IC62 74LVC1G14DCK, IC63 74LVC1G14DCK, IC64 74LVC1G14DCK, IC65 74LVC1G14DCK, IC66 74LVC1G14DCK, IC67 74LVC1G14DCK, IC68 74LVC1G14DCK, IC69 74LVC1G14DCK, IC7 74LVC1G14DCK, IC70 74LVC1G14DCK, IC71 74LVC1G14DCK, IC72 74LVC1G14DCK, IC73 VREG-5SOT23, IC8 74LVC1G14DCK, IC9 74LVC1G14DCK, J2 change, Q1 MOSFET-PSUPERSOT, Y1 16MHz

Commit message: Remove RGB LEDs, change reset switch
Parts:
- removed D74, D75: MOSFET-PSUPERSOT, Jordi:SUPERSOT-3
- removed D79, D80: (no value), Jordi:SOT23
- removed IC4: TLC5947DAP, Jordi:HTSSOP-32
- removed R10, R19, R20, R9: 4.7k, Jordi:R0603
- removed R14, R15, R24, R25: 100, Jordi:R0603
- removed R5: 4.7k/5.1k, Jordi:R0603
- added SJ1, SJ10, SJ11, SJ12, SJ13, SJ14, SJ15, SJ2, SJ3, SJ4, SJ5, SJ6, SJ7, SJ8, SJ9: JUMPER-PAD-3-2OF3_NC_BY_TRACE_SMALL, SparkFun-Passives:PAD-JUMPER-3-2OF3_NC_BY_TRACE_YES_SILK_FULL_BOX
- S71: value change -> RESET; device Jordi:SWITCH-TACTILE-SMD -> Jordi:SWITCH-TACTILE-SMD-RA
- moved S71 4.17 mm to (159.5, 97.0), turned to 180 degrees
- moved C9 3.77 mm to (23.8, 85.1), turned to 90 degrees
- moved C22 3.77 mm to (271.5, 85.1), turned to 90 degrees
- moved C12 3.62 mm to (81.0, 86.9), turned to 90 degrees
- moved C13 3.62 mm to (100.0, 86.9), turned to 90 degrees
- moved C14 3.62 mm to (119.1, 86.9), turned to 90 degrees
- moved C15 3.62 mm to (138.1, 86.9), turned to 90 degrees
- moved C16 3.62 mm to (157.2, 86.9), turned to 90 degrees
- moved C17 3.62 mm to (176.2, 86.9), turned to 90 degrees
- moved C19 3.62 mm to (214.3, 86.9), turned to 90 degrees
- moved C20 3.62 mm to (233.4, 86.9), turned to 90 degrees
- moved C21 3.62 mm to (252.4, 86.9), turned to 90 degrees
- moved R33 3.62 mm to (81.0, 89.9), turned to 90 degrees
- moved R35 3.62 mm to (100.0, 89.9), turned to 90 degrees
- moved R37 3.62 mm to (119.1, 89.9), turned to 90 degrees
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Connections:
- net !C0 renamed C0
- net !C1 renamed C1
- net !C10 renamed C10
- net !C12 renamed C12
- net !C13 renamed C13
- net !C3 renamed C3
- net !C4 renamed C4
- net !C6 renamed C6
- net !C7 renamed C7
- net !C9 renamed C9
- removed net !C11: C20.1, C35.1, C50.1, C65.1, S12.SW1, S12.SW3, S27.SW1, S27.SW3, S42.SW1, S42.SW3, S57.SW1, S57.SW3, S68.SW1, S68.SW3, U$3.11
- removed net !C14: C23.1, C38.1, C53.1, C68.1, S15.SW1, S15.SW3, S30.SW1, S30.SW3, S45.SW1, S45.SW3, S60.SW1, S60.SW3, S70.SW1, S70.SW3, U$3.14
- removed net !C2: C11.1, C26.1, C41.1, C56.1, S18.SW1, S18.SW3, S3.SW1, S3.SW3, S33.SW1, S33.SW3, S48.SW1, S48.SW3, S62.SW1, S62.SW3, U$2.10
- removed net !C5: C14.1, C29.1, C44.1, C59.1, S21.SW1, S21.SW3, S36.SW1, S36.SW3, S51.SW1, S51.SW3, S6.SW1, S6.SW3, S64.SW1, S64.SW3, U$2.13
- removed net !C8: C17.1, C32.1, C47.1, C62.1, S24.SW1, S24.SW3, S39.SW1, S39.SW3, S54.SW1, S54.SW3, S66.SW1, S66.SW3, S9.SW1, S9.SW3, U$3.7
- removed net LED-B0: IC3.7, S1.D2, S16.D2, S31.D2, S46.D2, S61.D2
- removed net LED-B1: IC3.10, S17.D2, S2.D2, S32.D2, S47.D2
- removed net LED-B10: IC4.16, S11.D2, S26.D2, S41.D2, S56.D2
- removed net LED-B11: IC4.19, S12.D2, S27.D2, S42.D2, S57.D2, S68.D2
- removed net LED-B12: IC4.22, S13.D2, S28.D2, S43.D2, S58.D2, S69.D2
- removed net LED-B13: IC4.25, S14.D2, S29.D2, S44.D2, S59.D2
- removed net LED-B14: IC4.28, S15.D2, S30.D2, S45.D2, S60.D2, S70.D2
- removed net LED-B2: IC3.13, S18.D2, S3.D2, S33.D2, S48.D2, S62.D2
- removed net LED-B3: IC3.16, S19.D2, S34.D2, S4.D2, S49.D2, S63.D2
- removed net LED-B4: IC3.19, S20.D2, S35.D2, S5.D2, S50.D2
- removed net LED-B5: IC3.22, S21.D2, S36.D2, S51.D2, S6.D2, S64.D2
- removed net LED-B6: IC3.25, S22.D2, S37.D2, S52.D2, S65.D2, S7.D2
- removed net LED-B7: IC3.28, S23.D2, S38.D2, S53.D2, S8.D2
- removed net LED-B8: IC4.10, S24.D2, S39.D2, S54.D2, S66.D2, S9.D2
- removed net LED-B9: IC4.13, S10.D2, S25.D2, S40.D2, S55.D2, S67.D2
- removed net LED-G0: IC3.5, S1.D1, S16.D1, S31.D1, S46.D1, S61.D1
- removed net LED-G1: IC3.8, S17.D1, S2.D1, S32.D1, S47.D1
- removed net LED-G10: IC4.14, S11.D1, S26.D1, S41.D1, S56.D1
- removed net LED-G11: C76.1, IC4.17, S12.D1, S27.D1, S42.D1, S57.D1, S68.D1
- removed net LED-G12: IC4.20, S13.D1, S28.D1, S43.D1, S58.D1, S69.D1
- removed net LED-G13: IC4.23, S14.D1, S29.D1, S44.D1, S59.D1
- removed net LED-G14: C78.1, IC4.26, S15.D1, S30.D1, S45.D1, S60.D1, S70.D1
- removed net LED-G2: C70.1, IC3.11, S18.D1, S3.D1, S33.D1, S48.D1, S62.D1
- removed net LED-G3: IC3.14, S19.D1, S34.D1, S4.D1, S49.D1, S63.D1
- removed net LED-G4: IC3.17, S20.D1, S35.D1, S5.D1, S50.D1
- removed net LED-G5: C72.1, IC3.20, S21.D1, S36.D1, S51.D1, S6.D1, S64.D1
- removed net LED-G6: IC3.23, S22.D1, S37.D1, S52.D1, S65.D1, S7.D1
- removed net LED-G7: IC3.26, S23.D1, S38.D1, S53.D1, S8.D1
- removed net LED-G8: C74.1, IC4.8, S24.D1, S39.D1, S54.D1, S66.D1, S9.D1
- removed net LED-G9: IC4.11, S10.D1, S25.D1, S40.D1, S55.D1, S67.D1
- removed net LED-R0: IC3.6, S1.LED2, S16.LED2, S31.LED2, S46.LED2, S61.LED2
- removed net LED-R1: IC3.9, S17.LED2, S2.LED2, S32.LED2, S47.LED2
- removed net LED-R10: IC4.15, S11.LED2, S26.LED2, S41.LED2, S56.LED2
- removed net LED-R11: IC4.18, S12.LED2, S27.LED2, S42.LED2, S57.LED2, S68.LED2
- removed net LED-R12: IC4.21, S13.LED2, S28.LED2, S43.LED2, S58.LED2, S69.LED2
- removed net LED-R13: IC4.24, S14.LED2, S29.LED2, S44.LED2, S59.LED2
- removed net LED-R14: IC4.27, S15.LED2, S30.LED2, S45.LED2, S60.LED2, S70.LED2
- removed net LED-R2: IC3.12, S18.LED2, S3.LED2, S33.LED2, S48.LED2, S62.LED2
- removed net LED-R3: IC3.15, S19.LED2, S34.LED2, S4.LED2, S49.LED2, S63.LED2
- removed net LED-R4: IC3.18, S20.LED2, S35.LED2, S5.LED2, S50.LED2
- removed net LED-R5: IC3.21, S21.LED2, S36.LED2, S51.LED2, S6.LED2, S64.LED2
- removed net LED-R6: IC3.24, S22.LED2, S37.LED2, S52.LED2, S65.LED2, S7.LED2
- removed net LED-R7: IC3.27, S23.LED2, S38.LED2, S53.LED2, S8.LED2
- removed net LED-R8: IC4.9, S24.LED2, S39.LED2, S54.LED2, S66.LED2, S9.LED2
- removed net LED-R9: IC4.12, S10.LED2, S25.LED2, S40.LED2, S55.LED2, S67.LED2
- removed net N$104: IC15.4
- removed net N$107: D79.1, R19.2, R24.2
- removed net N$108: D80.1, R20.2, R25.2
- removed net N$109: IC16.4
- removed net N$110: IC17.4
- removed net N$69: D75.1, R10.1, R15.2
- removed net N$70: D74.1, R14.2, R9.1
- removed net N$87: D79.2, R14.1
- removed net N$95: D80.2, R15.1
- new net C11: C20.1, C35.1, C50.1, C65.1, C76.1, S12.SW1, S12.SW3, S27.SW1, S27.SW3, S42.SW1, S42.SW3, S57.SW1, S57.SW3, S68.SW1, S68.SW3, U$3.11
- new net C14: C23.1, C38.1, C53.1, C68.1, C78.1, S15.SW1, S15.SW3, S30.SW1, S30.SW3, S45.SW1, S45.SW3, S60.SW1, S60.SW3, S70.SW1, S70.SW3, U$3.14
- new net C2: C11.1, C26.1, C41.1, C56.1, C70.1, S18.SW1, S18.SW3, S3.SW1, S3.SW3, S33.SW1, S33.SW3, S48.SW1, S48.SW3, S62.SW1, S62.SW3, U$2.10
- new net C5: C14.1, C29.1, C44.1, C59.1, C72.1, S21.SW1, S21.SW3, S36.SW1, S36.SW3, S51.SW1, S51.SW3, S6.SW1, S6.SW3, S64.SW1, S64.SW3, U$2.13
- new net C8: C17.1, C32.1, C47.1, C62.1, C74.1, S24.SW1, S24.SW3, S39.SW1, S39.SW3, S54.SW1, S54.SW3, S66.SW1, S66.SW3, S9.SW1, S9.SW3, U$3.7
- new net LED0: IC3.5
- new net LED1: IC3.6
- new net LED10: IC3.15
- new net LED11: IC3.16
- new net LED12: IC3.17
- new net LED13: IC3.18
- new net LED14: IC3.19
- new net LED15: IC3.20
- new net LED16: IC3.21
- new net LED17: IC3.22
- new net LED18: IC3.23
- new net LED19: IC3.24
- new net LED2: IC3.7
- new net LED20: IC3.25
- new net LED21: IC3.26
- new net LED22: IC3.27
- new net LED23: IC3.28
- new net LED3: IC3.8
- new net LED4: IC3.9
- new net LED5: IC3.10
- new net LED6: IC3.11
- new net LED7: IC3.12
- new net LED8: IC3.13
- new net LED9: IC3.14
- new net N$13: S16.LED1, S17.LED1, S18.LED1, S19.LED1, S20.LED1
- new net N$15: S31.LED1, S32.LED1, S33.LED1, S34.LED1, S35.LED1
- new net N$16: S46.LED1, S47.LED1, S48.LED1, S49.LED1, S50.LED1
- new net N$21: S61.LED1, S62.LED1, S63.LED1
- new net N$30: S68.LED1, S69.LED1, S70.LED1
- new net N$31: S56.LED1, S57.LED1, S58.LED1, S59.LED1, S60.LED1
- new net N$32: S41.LED1, S42.LED1, S43.LED1, S44.LED1, S45.LED1
- new net N$37: S26.LED1, S27.LED1, S28.LED1, S29.LED1, S30.LED1
- new net N$38: S11.LED1, S12.LED1, S13.LED1, S14.LED1, S15.LED1
- new net N$39: IC1.4, SJ1.3
- new net N$40: D2.C, SJ2.1
- new net N$41: D73.3
- new net N$42: D72.3
- new net N$43: D71.3
- new net N$45: D76.3, D77.3, D78.3, R16.1, R17.1, R18.1
- new net N$48: D4.C, SJ4.1
- new net N$49: D5.C, SJ5.1
- new net N$52: D6.C, SJ6.1
- new net N$53: D7.C, SJ7.1
- new net N$54: IC5.4, SJ3.3
- new net N$56: IC6.4, SJ4.3
- new net N$57: IC7.4, SJ5.3
- new net N$58: D8.C, SJ8.1
- new net N$59: D9.C, SJ9.1
- new net N$60: D10.C, SJ10.1
- new net N$62: D11.C, SJ11.1
- new net N$64: D12.C, SJ12.1
- new net N$65: D13.C, SJ13.1
- new net N$66: D14.C, SJ14.1
- new net N$67: D15.C, SJ15.1
- net +3V3: no longer IC4.32
- net BLANK: no longer IC4.2
- net GND: now also S71.3; no longer D76.3, D77.3, D78.3, D79.3, D80.3, IC4.1, IC4.PAD, R16.1, R17.1, R18.1, R19.1, R20.1, R5.2, S71.2
- net LED-A3: no longer R24.1
- net LED-A4: no longer R25.1
- net N$12: now also S1.LED1, S2.LED1, S3.LED1, S4.LED1, S5.LED1; no longer IC3.29, IC4.4
- net N$17: now also D1.C, SJ1.1; no longer IC1.4
- net N$18: now also IC8.4, SJ6.3; no longer IC2.4
- net N$19: now also IC9.4, SJ7.3; no longer IC5.4
- net N$20: now also IC10.4, SJ8.3; no longer IC6.4
- net N$22: now also IC2.4, SJ2.3; no longer IC7.4
- net N$23: now also IC11.4, SJ9.3; no longer IC8.4
- net N$24: now also IC12.4, SJ10.3; no longer IC9.4
- net N$25: now also IC13.4, SJ11.3; no longer IC10.4
- net N$26: now also IC14.4, SJ12.3; no longer IC11.4
- net N$27: now also IC15.4, SJ13.3; no longer IC12.4
- net N$28: now also IC16.4, SJ14.3; no longer IC13.4
- net N$29: now also IC17.4, SJ15.3; no longer IC14.4
- net N$47: now also D3.C, SJ3.1; no longer IC4.31, R5.1
- net N$51: no longer D71.3, S1.LED1, S11.LED1, S12.LED1, S13.LED1, S14.LED1, S15.LED1, S2.LED1, S3.LED1, S4.LED1, S5.LED1
- net N$55: no longer D72.3, S16.LED1, S17.LED1, S18.LED1, S19.LED1, S20.LED1, S26.LED1, S27.LED1, S28.LED1, S29.LED1, S30.LED1
- net N$61: no longer D73.3, S31.LED1, S32.LED1, S33.LED1, S34.LED1, S35.LED1, S41.LED1, S42.LED1, S43.LED1, S44.LED1, S45.LED1
- net N$63: no longer D74.3, S46.LED1, S47.LED1, S48.LED1, S49.LED1, S50.LED1, S56.LED1, S57.LED1, S58.LED1, S59.LED1, S60.LED1
- net N$78: no longer D75.3, S61.LED1, S62.LED1, S63.LED1, S68.LED1, S69.LED1, S70.LED1
- net R0: now also SJ1.2, SJ10.2, SJ11.2, SJ12.2, SJ13.2, SJ14.2, SJ15.2, SJ2.2, SJ3.2, SJ4.2, SJ5.2, SJ6.2, SJ7.2, SJ8.2, SJ9.2, U$1.40; no longer D1.C, D10.C, D11.C, D12.C, D13.C, D14.C, D15.C, D2.C, D3.C, D4.C, D5.C, D6.C, D7.C, D8.C, D9.C
- net R1: now also U$1.39
- net R2: now also U$1.38
- net R3: now also U$1.37
- net R4: now also U$1.36
- net RST: now also S71.2; no longer S71.3, S71.4
- net SCK: no longer IC4.3
- net SOUT: now also IC3.29; no longer IC4.29
- net VIN: no longer D74.2, D75.2, R10.2, R9.2
- net XLAT: no longer IC4.30
Routing:
- net N$51: track 298.8 -> 86.9 mm
- net N$61: track 298.8 -> 86.9 mm
- net N$63: track 298.8 -> 86.9 mm
- net N$55: track 298.7 -> 86.9 mm
- net N$78: track 297.6 -> 103.8 mm
- net C2: track 0.00 -> 113.0 mm
- net C14: track 0.00 -> 98.2 mm
- net !C14: track 98.2 -> 0.00 mm
- net C8: track 0.00 -> 98.2 mm
- net !C8: track 98.2 -> 0.00 mm
- net C5: track 0.00 -> 98.2 mm
- net C11: track 0.00 -> 98.2 mm
- net !C5: track 98.2 -> 0.00 mm
- net !C2: track 98.2 -> 0.00 mm
- net !C11: track 98.2 -> 0.00 mm
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