File: hardware/ION-60/Eagle/ION-60/ION-60.brd (EAGLE design)
At the start: 285 x 95 mm, 486 parts, among them IC1 74LVC1G14DCK, IC10 74LVC1G14DCK, IC11 74LVC1G14DCK, IC12 74LVC1G14DCK, IC13 74LVC1G14DCK, IC14 74LVC1G14DCK, IC15 74LVC1G14DCK, IC16 74LVC1G14DCK, IC17 74LVC1G14DCK, IC18 74LVC1G14DCK, IC19 74LVC1G14DCK, IC2 74LVC1G14DCK, IC20 74LVC1G14DCK, IC21 74LVC1G14DCK, IC22 74LVC1G14DCK, IC23 74LVC1G14DCK, IC24 74LVC1G14DCK, IC25 74LVC1G14DCK, IC26 74LVC1G14DCK, IC27 74LVC1G14DCK, IC28 74LVC1G14DCK, IC29 74LVC1G14DCK, IC3 TLC5947DAP, IC30 74LVC1G14DCK, IC31 74LVC1G14DCK, IC32 74LVC1G14DCK, IC33 74LVC1G14DCK, IC34 74LVC1G14DCK, IC35 74LVC1G14DCK, IC36 74LVC1G14DCK, IC37 74LVC1G14DCK, IC38 74LVC1G14DCK, IC39 74LVC1G14DCK, IC40 74LVC1G14DCK, IC41 74LVC1G14DCK, IC42 74LVC1G14DCK, IC43 74LVC1G14DCK, IC44 74LVC1G14DCK, IC45 74LVC1G14DCK, IC46 74LVC1G14DCK, IC47 74LVC1G14DCK, IC48 74LVC1G14DCK, IC49 74LVC1G14DCK, IC5 74LVC1G14DCK, IC50 74LVC1G14DCK, IC51 74LVC1G14DCK, IC52 74LVC1G14DCK, IC53 74LVC1G14DCK, IC54 74LVC1G14DCK, IC55 74LVC1G14DCK, IC56 74LVC1G14DCK, IC57 74LVC1G14DCK, IC58 74LVC1G14DCK, IC59 74LVC1G14DCK, IC6 74LVC1G14DCK, IC60 74LVC1G14DCK, IC61 74LVC1G14DCK, IC62 74LVC1G14DCK, IC63 74LVC1G14DCK, IC64 74LVC1G14DCK, IC65 74LVC1G14DCK, IC66 74LVC1G14DCK, IC67 74LVC1G14DCK, IC68 74LVC1G14DCK, IC69 74LVC1G14DCK, IC7 74LVC1G14DCK, IC70 74LVC1G14DCK, IC71 74LVC1G14DCK, IC72 74LVC1G14DCK, IC73 VREG-5SOT23, IC8 74LVC1G14DCK, IC9 74LVC1G14DCK, J2 change, Q1 MOSFET-PSUPERSOT, Y1 16MHz

Commit message: Lots more work
Parts:
- removed J1: (no value), Jordi:M-2X03-0.1-PTH-SHROUDED
- removed J2: change, Jordi:M-1X06-0.05-PTH
- removed J3: (no value), Jordi:M-1X06-0.1-PTH
- removed JP1, JP2, JP3, JP4: USB-MICROBSMD, Jordi:USB-MICRO-B-SMD
- removed U$2, U$3: 74LVC138AD, SparkFun-DigitalIC:SO016
- added C79, C80, C83, C84: 1uF, Jordi:C0603
- added COL-EXP, LED-EXP: (no value), Jordi:M-1X06-0.05-PTH
- added D74, D75, D79, D80: (no value), SparkFun-DiscreteSemi:SOD-123
- added EXP: check, Jordi:M-1X06-0.05-PTH
- added IC4, IC74, IC75, IC76: 74LVC1G14DCK, 74xx-little-us:SC70-5
- added IC77, IC78: 74LS595D, SparkFun-DigitalIC:SO16
- added ICSP: (no value), Jordi:M-2X03-0.1-PTH-SHROUDED
- added R10, R15, R20, R5: 4.7k?, Jordi:R0603
- added R14, R19, R24, R9: 22k?, Jordi:R0603
- added R166, R167, R169, R170, R25: 10K, Jordi:R0603
- added ROW-EXP: (no value), Jordi:M-1X06-0.1-PTH
- added RST: (no value), Jordi:SWITCH-TACTILE-SMD-RA
- added S72, S73, S74, S75, S76, S77, S78, S79, S80, S81, S82: (no value), Jordi:CHERRY-MX-LED-1X1
- added SJ16, SJ17, SJ18, SJ19, SJ20, SJ21, SJ22, SJ23, SJ24, SJ25, SJ26, SJ27, SJ28, SJ29, SJ30, SJ31, SJ32, SJ33, SJ34, SJ35, SJ36, SJ37, SJ38, SJ39, SJ40, SJ41, SJ42, SJ43, SJ44, SJ45, SJ46, SJ47, SJ48, SJ49, SJ50, SJ51, SJ52, SJ53, SJ54, SJ55, SJ56, SJ57, SJ58, SJ59, SJ60, SJ61, SJ62, SJ63, SJ64, SJ65, SJ66, SJ67, SJ68, SJ69, SJ70, SJ71, SJ72, SJ73, SJ74: JUMPER-PAD-3-2OF3_NC_BY_TRACE_SMALL, SparkFun-Passives:PAD-JUMPER-3-2OF3_NC_BY_TRACE_YES_SILK_FULL_BOX
- added USB1, USB2: USB-MICROBSMD, Jordi:USB-MICRO-B-SMD
- S71: value RESET -> (none); device Jordi:SWITCH-TACTILE-SMD-RA -> Jordi:CHERRY-MX-LED-1X1
- moved S71 173.7 mm to (9.53, 9.53), flipped to the top, turned to 0 degrees
- moved R6 125.7 mm to (71.4, -8.93)
- moved D76 125.5 mm to (67.9, -10.1), turned to 270 degrees
- moved R11 125.2 mm to (71.4, -10.7)
- moved R16 118.4 mm to (67.9, -7.74), turned to 180 degrees
- moved D71 117.2 mm to (71.4, -6.55), turned to 0 degrees
- moved R21 115.6 mm to (67.9, -5.95), turned to 180 degrees
- moved R8 104.4 mm to (214.9, -14.9)
- moved R13 104.0 mm to (214.9, -16.7)
- moved D78 99.3 mm to (211.3, -16.1), turned to 270 degrees
- moved D73 97.2 mm to (214.9, -12.5), turned to 0 degrees
- moved R7 95.1 mm to (149.4, -17.3)
- moved R12 94.5 mm to (149.4, -19.1)
- moved R18 93.7 mm to (211.3, -13.7), turned to 180 degrees
- moved R23 91.4 mm to (211.3, -11.9), turned to 180 degrees
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Connections:
- net SW31 renamed N$12
- net SW32 renamed N$13
- net SW33 renamed N$15
- net SW34 renamed N$16
- net SW35 renamed N$30
- net SW36 renamed N$31
- net SW37 renamed N$32
- net SW38 renamed N$37
- net SW39 renamed N$38
- net SW40 renamed N$41
- net SW41 renamed N$42
- net SW42 renamed N$43
- net SW43 renamed N$51
- net SW44 renamed N$55
- net SW45 renamed N$61
- removed net !E1: U$1.1, U$2.4, U$3.4
- removed net A0: U$1.28, U$2.1, U$3.1
- removed net A1: U$1.29, U$2.2, U$3.2
- removed net A2: U$1.30, U$2.3, U$3.3
- removed net A3: U$1.12, U$2.5, U$3.6
- removed net BLANK: IC3.2, U$1.8
- removed net LED-A0: J3.1, R21.1
- removed net LED-A1: J3.2, R22.1
- removed net LED-A2: J3.3, R23.1
- removed net LED-A3: J3.4
- removed net LED-A4: J3.5
- removed net N$12 (its old number): S1.LED1, S2.LED1, S3.LED1, S4.LED1, S5.LED1
- removed net N$13 (its old number): S16.LED1, S17.LED1, S18.LED1, S19.LED1, S20.LED1
- removed net N$15 (its old number): S31.LED1, S32.LED1, S33.LED1, S34.LED1, S35.LED1
- removed net N$16 (its old number): S46.LED1, S47.LED1, S48.LED1, S49.LED1, S50.LED1
- removed net N$30 (its old number): S68.LED1, S69.LED1, S70.LED1
- removed net N$31 (its old number): S56.LED1, S57.LED1, S58.LED1, S59.LED1, S60.LED1
- removed net N$32 (its old number): S41.LED1, S42.LED1, S43.LED1, S44.LED1, S45.LED1
- removed net N$37 (its old number): S26.LED1, S27.LED1, S28.LED1, S29.LED1, S30.LED1
- removed net N$38 (its old number): S11.LED1, S12.LED1, S13.LED1, S14.LED1, S15.LED1
- removed net N$41 (its old number): D73.3
- removed net N$42 (its old number): D72.3
- removed net N$43 (its old number): D71.3
- removed net N$51 (its old number): S10.LED1, S6.LED1, S7.LED1, S8.LED1, S9.LED1
- removed net N$55 (its old number): S21.LED1, S22.LED1, S23.LED1, S24.LED1, S25.LED1
- removed net N$61 (its old number): S36.LED1, S37.LED1, S38.LED1, S39.LED1, S40.LED1
- removed net SOUT: IC3.29, J3.6
- removed net XLAT: IC3.30
- new net !COL70: C79.2, IC4.2, R9.1
- new net !COL71: C80.2, IC74.2, R14.1
- new net !COL72: C83.2, IC75.2, R19.1
- new net !COL73: C84.2, IC76.2, R24.1
- new net C-!OE: COL-EXP.3, IC77.13, IC78.13, U$1.27
- new net C-CLK: COL-EXP.5, IC77.11, IC78.11, U$1.22
- new net C-LAT: COL-EXP.4, IC77.12, IC78.12, U$1.26
- new net C-SIN: IC77.14, U$1.25
- new net C-SOUT: COL-EXP.6, IC78.9
- new net C15: IC78.7, ROW-EXP.6
- new net G0: D71.3, S1.LED1, S16.LED1, S17.LED1, S18.LED1, S19.LED1, S2.LED1, S20.LED1, S21.LED1, S3.LED1, S31.LED1, S32.LED1, S33.LED1, S34.LED1, S35.LED1, S36.LED1, S4.LED1, S46.LED1, S47.LED1, S48.LED1, S49.LED1, S5.LED1, S50.LED1, S51.LED1, S6.LED1
- new net G1: D72.3, S22.LED1, S23.LED1, S24.LED1, S37.LED1, S38.LED1, S39.LED1, S52.LED1, S53.LED1, S54.LED1, S61.LED1, S62.LED1, S63.LED1, S64.LED1, S67.LED1, S68.LED1, S69.LED1, S7.LED1, S70.LED1, S71.LED1, S72.LED1, S73.LED1, S74.LED1, S75.LED1, S76.LED1, S77.LED1, S78.LED1, S79.LED1, S8.LED1, S80.LED1, S81.LED1, S82.LED1, S9.LED1
- new net G2: D73.3, S10.LED1, S11.LED1, S12.LED1, S13.LED1, S14.LED1, S15.LED1, S25.LED1, S26.LED1, S27.LED1, S28.LED1, S29.LED1, S30.LED1, S40.LED1, S41.LED1, S42.LED1, S43.LED1, S44.LED1, S45.LED1, S55.LED1, S56.LED1, S57.LED1, S58.LED1, S59.LED1, S60.LED1
- new net LED-BLANK: IC3.2, LED-EXP.3, U$1.8
- new net LED-G0: R21.1, U$1.29
- new net LED-G1: R22.1, U$1.30
- new net LED-G2: R23.1, U$1.12
- new net LED-SOUT: IC3.29, LED-EXP.6
- new net LED-XLAT: IC3.30, LED-EXP.4, U$1.28
- new net N$100: IC21.4, SJ19.1
- new net N$101: D20.C, SJ20.3
- new net N$102: IC22.4, SJ20.1
- new net N$103: D32.C, SJ32.3
- new net N$104: D31.C, SJ31.3
- new net N$107: D61.A, R146.1, R147.2, S61.SW1, S61.SW3, S71.SW2, S71.SW4
- new net N$108: IC68.4, SJ66.1
- new net N$109: D65.C, SJ65.3
- new net N$110: IC67.4, SJ65.1
- new net N$111: D64.C, SJ64.3
- new net N$127: IC56.4, SJ54.3
- new net N$128: IC57.4, SJ55.3
- new net N$129: IC58.4, SJ56.3
- new net N$145: IC59.4, SJ57.3
- new net N$146: IC60.4, SJ58.3
- new net N$147: IC61.4, SJ59.3
- new net N$163: D80.C, SJ74.3
- new net N$164: IC76.4, SJ74.1
- new net N$165: D80.A, R20.1, R24.2, S70.SW2, S70.SW4, S82.SW1, S82.SW3
- new net N$176: IC49.4, SJ47.1
- new net N$177: D48.C, SJ48.3
- new net N$178: IC50.4, SJ48.1
- new net N$179: D49.C, SJ49.3
- new net N$180: IC48.4, SJ46.1
- new net N$181: IC51.4, SJ49.1
- new net N$182: D50.C, SJ50.3
- new net N$183: IC52.4, SJ50.1
- new net N$184: D36.C, SJ36.1
- new net N$185: D37.C, SJ37.1
- new net N$186: D38.C, SJ38.1
- new net N$187: D39.C, SJ39.1
- new net N$188: D40.C, SJ40.1
- new net N$189: D41.C, SJ41.1
- new net N$190: D42.C, SJ42.1
- new net N$191: D43.C, SJ43.1
- new net N$192: D44.C, SJ44.1
- new net N$193: D45.C, SJ45.1
- new net N$194: IC77.9, IC78.14
- new net N$68: IC18.4, SJ16.1
- new net N$69: D17.C, SJ17.3
- new net N$70: IC19.4, SJ17.1
- new net N$71: D18.C, SJ18.3
- new net N$72: IC20.4, SJ18.1
- new net N$73: IC23.4, SJ21.3
- new net N$76: IC24.4, SJ22.3
- new net N$77: IC25.4, SJ23.3
- new net N$79: IC26.4, SJ24.3
- new net N$80: IC27.4, SJ25.3
- new net N$81: IC28.4, SJ26.3
- new net N$84: IC29.4, SJ27.3
- new net N$85: IC30.4, SJ28.3
- new net N$86: IC31.4, SJ29.3
- new net N$87: IC32.4, SJ30.3
- new net N$88: D30.C, SJ30.1
- new net N$89: D29.C, SJ29.1
- new net N$91: D28.C, SJ28.1
- new net N$92: D27.C, SJ27.1
- new net N$93: D26.C, SJ26.1
- new net N$95: D25.C, SJ25.1
- new net N$96: D24.C, SJ24.1
- new net N$97: D23.C, SJ23.1
- new net N$98: D22.C, SJ22.1
- new net N$99: D21.C, SJ21.1
- new net SW71: D75.A, R10.1, R14.2, S69.SW1, S69.SW3, S80.SW2, S80.SW4
- new net SW72: D79.A, R15.1, R19.2, S81.SW2, S81.SW4
- net +3V3: now also COL-EXP.2, EXP.6, IC4.5, IC74.5, IC75.5, IC76.5, IC77.10, IC77.16, IC78.10, IC78.16, ICSP.2, LED-EXP.2, R10.2, R15.2, R20.2, R5.2; no longer J1.2, J2.6, U$2.16, U$2.6, U$3.16
- net C0: now also IC77.15, S61.SW2, S61.SW4, S71.SW1, S71.SW3; no longer S61.SW1, S61.SW3, U$2.7
- net C1: now also C70.1, IC77.1, S72.SW1, S72.SW3; no longer U$2.9
- net C10: now also C78.1, IC78.2, S78.SW1, S78.SW3; no longer U$3.10
- net C11: now also C79.1, IC78.3, S79.SW2, S79.SW4; no longer C76.1, U$3.11
- net C12: now also C80.1, IC78.4, S69.SW2, S69.SW4, S80.SW1, S80.SW3; no longer C77.1, S69.SW1, S69.SW3, U$3.12
- net C13: now also C83.1, IC78.5, S81.SW1, S81.SW3; no longer U$3.13
- net C14: now also C84.1, IC78.6, S82.SW2, S82.SW4; no longer C78.1, U$3.14
- net C2: now also C71.1, IC77.2, S73.SW2, S73.SW4; no longer C70.1, U$2.10
- net C3: now also C72.1, IC77.3, S63.SW2, S63.SW4, S74.SW1, S74.SW3; no longer C71.1, S63.SW1, S63.SW3, U$2.11
- net C4: now also C73.1, IC77.4, S75.SW1, S75.SW3; no longer U$2.12
- net C5: now also C74.1, IC77.5, S76.SW2, S76.SW4; no longer C72.1, U$2.13
- net C6: now also C75.1, IC77.6; no longer C73.1, U$2.14
- net C7: now also IC77.7; no longer U$2.15
- net C8: now also C76.1, IC78.15; no longer C74.1, U$3.7
- net C9: now also C77.1, IC78.1, S67.SW2, S67.SW4, S77.SW1, S77.SW3; no longer C75.1, S67.SW1, S67.SW3, U$3.9
- net D+: now also USB1.D+, USB2.D+; no longer JP1.D+, JP2.D+, JP3.D+, JP4.D+
- net D-: now also USB1.D-, USB2.D-; no longer JP1.D-, JP2.D-, JP3.D-, JP4.D-
- net GND: now also COL-EXP.1, EXP.1, IC4.3, IC74.3, IC75.3, IC76.3, IC77.8, IC78.8, ICSP.6, LED-EXP.1, R166.1, R167.1, R169.1, R170.1, R25.1, RST.1, RST.3, USB1.GND, USB2.GND; no longer J1.6, J2.1, JP1.GND, JP2.GND, JP3.GND, JP4.GND, S71.1, S71.3, U$2.8, U$3.5, U$3.8
- net LED0: now also S46.LED2, S60.LED2, S72.LED2, S75.LED2
- net LED1: now also S31.LED2, S45.LED2, S61.LED2, S71.LED2
- net LED10: now also S18.LED2, S28.LED2, S70.LED2, S82.LED2
- net LED11: now also S13.LED2, S3.LED2, S78.LED2, S81.LED2
- net LED12: now also S49.LED2, S52.LED2, S57.LED2
- net LED13: now also S34.LED2, S37.LED2, S42.LED2
- net LED14: now also S19.LED2, S22.LED2, S27.LED2
- net LED15: now also S12.LED2, S4.LED2, S7.LED2
- net LED16: now also S50.LED2, S53.LED2, S56.LED2
- net LED17: now also S35.LED2, S38.LED2, S41.LED2
- net LED18: now also S20.LED2, S23.LED2, S26.LED2
- net LED19: now also S11.LED2, S5.LED2, S8.LED2
- net LED2: now also S16.LED2, S30.LED2, S62.LED2, S73.LED2
- net LED20: now also S51.LED2, S54.LED2, S55.LED2
- net LED21: now also S36.LED2, S39.LED2, S40.LED2
- net LED22: now also S21.LED2, S24.LED2, S25.LED2
- net LED23: now also S10.LED2, S6.LED2, S9.LED2
- net LED3: now also S1.LED2, S15.LED2, S63.LED2, S74.LED2
- net LED4: now also S47.LED2, S59.LED2, S64.LED2, S76.LED2
- net LED5: now also S32.LED2, S44.LED2, S65.LED2
- net LED6: now also S17.LED2, S29.LED2, S66.LED2
- net LED7: now also S14.LED2, S2.LED2, S67.LED2, S77.LED2
- net LED8: now also S48.LED2, S58.LED2, S68.LED2, S79.LED2
- net LED9: now also S33.LED2, S43.LED2, S69.LED2, S80.LED2
- net MISO: now also ICSP.1; no longer J1.1
- net MOSI: now also ICSP.4; no longer J1.4
- net N$11: now also USB1.VBUS, USB2.VBUS; no longer JP1.VBUS, JP2.VBUS, JP3.VBUS, JP4.VBUS
- net N$112: now also IC66.4, SJ64.1; no longer IC18.4
- net N$113: now also D63.C, SJ63.3; no longer IC19.4
- net N$114: now also IC65.4, SJ63.1; no longer IC20.4
- net N$115: now also D62.C, SJ62.3; no longer IC21.4
- net N$116: now also IC64.4, SJ62.1; no longer IC22.4
- net N$117: now also D61.C, SJ61.3; no longer IC23.4
- net N$118: now also IC63.4, SJ61.1; no longer IC24.4
- net N$119: now also IC33.4, SJ31.1; no longer IC25.4
- net N$120: now also IC34.4, SJ32.1; no longer IC26.4
- net N$121: now also D33.C, SJ33.3; no longer IC27.4
- net N$122: now also IC35.4, SJ33.1; no longer IC28.4
- net N$123: now also D34.C, SJ34.3; no longer IC29.4
- net N$124: now also IC53.4, SJ51.3; no longer IC30.4
- net N$125: now also IC54.4, SJ52.3; no longer IC31.4
- net N$126: now also IC55.4, SJ53.3; no longer IC32.4
- net N$130: now also IC36.4, SJ34.1; no longer IC33.4
- net N$131: now also D35.C, SJ35.3; no longer IC34.4
- net N$132: now also IC37.4, SJ35.1; no longer IC35.4
- net N$133: now also IC38.4, SJ36.3; no longer IC36.4
- net N$134: now also IC39.4, SJ37.3; no longer IC37.4
- net N$135: now also IC40.4, SJ38.3; no longer IC38.4
- net N$136: now also IC41.4, SJ39.3; no longer IC39.4
- net N$137: now also IC42.4, SJ40.3; no longer IC40.4
- net N$138: now also IC43.4, SJ41.3; no longer IC41.4
- net N$139: now also IC44.4, SJ42.3; no longer IC42.4
- net N$140: now also IC45.4, SJ43.3; no longer IC43.4
- net N$141: now also IC46.4, SJ44.3; no longer IC44.4
- net N$142: now also IC47.4, SJ45.3; no longer IC45.4
- net N$143: now also D46.C, SJ46.3; no longer IC46.4
- net N$144: now also D47.C, SJ47.3; no longer IC47.4
- net N$148: now also IC62.4, SJ60.3; no longer IC48.4
- net N$149: now also D69.C, SJ69.3; no longer IC49.4
- net N$150: now also IC71.4, SJ69.1; no longer IC50.4
- net N$151: now also D70.C, SJ70.3; no longer IC51.4
- net N$152: now also IC72.4, SJ70.1; no longer IC52.4
- net N$153: now also D67.C, SJ67.3; no longer IC53.4
- net N$154: now also IC69.4, SJ67.1; no longer IC54.4
- net N$155: now also D68.C, SJ68.3; no longer IC55.4
- net N$156: now also IC70.4, SJ68.1; no longer IC56.4
- net N$157: now also D74.C, SJ71.3; no longer IC57.4
- net N$158: now also IC4.4, SJ71.1; no longer IC58.4
- net N$159: now also D75.C, SJ72.3; no longer IC59.4
- net N$160: now also IC74.4, SJ72.1; no longer IC60.4
- net N$161: now also D79.C, SJ73.3; no longer IC61.4
- net N$162: now also IC75.4, SJ73.1; no longer IC62.4
- net N$166: now also D60.C, SJ60.1; no longer IC63.4
- net N$167: now also D59.C, SJ59.1; no longer IC64.4
- net N$168: now also D58.C, SJ58.1; no longer IC65.4
- net N$169: now also D57.C, SJ57.1; no longer IC66.4
- net N$17: now also SJ1.3; no longer SJ1.1
- net N$170: now also D56.C, SJ56.1; no longer IC67.4
- net N$171: now also D55.C, SJ55.1; no longer IC68.4
- net N$172: now also D54.C, SJ54.1; no longer IC69.4
- net N$173: now also D53.C, SJ53.1; no longer IC70.4
- net N$174: now also D52.C, SJ52.1; no longer IC71.4
- net N$175: now also D51.C, SJ51.1; no longer IC72.4
- net N$21: now also D66.C, SJ66.3; no longer S61.LED1, S62.LED1, S63.LED1
- net N$22: now also D2.C; no longer IC2.4
- net N$39: now also SJ1.1; no longer SJ1.3
- net N$40: now also IC2.4; no longer D2.C
- net N$47: now also SJ3.3; no longer SJ3.1
- net N$48: now also IC5.4, SJ3.1; no longer D4.C, SJ4.1
- net N$49: now also D4.C, SJ4.3; no longer D5.C, SJ5.1
- net N$54: now also IC6.4, SJ4.1; no longer IC5.4, SJ3.3
- net N$56: now also D5.C, SJ5.3; no longer IC6.4, SJ4.3
- net N$57: now also SJ5.1; no longer SJ5.3
- net N$63: now also D16.C, SJ16.3; no longer S51.LED1, S52.LED1, S53.LED1, S54.LED1, S55.LED1
- net N$78: now also D19.C, SJ19.3; no longer S64.LED1, S65.LED1, S66.LED1, S67.LED1
- net R0: now also R25.2, ROW-EXP.1, U$1.41; no longer U$1.40
- net R1: now also R166.2, ROW-EXP.2, SJ16.2, SJ17.2, SJ18.2, SJ19.2, SJ20.2, SJ21.2, SJ22.2, SJ23.2, SJ24.2, SJ25.2, SJ26.2, SJ27.2, SJ28.2, SJ29.2, SJ30.2; no longer D16.C, D17.C, D18.C, D19.C, D20.C, D21.C, D22.C, D23.C, D24.C, D25.C, D26.C, D27.C, D28.C, D29.C, D30.C
- net R2: now also R167.2, ROW-EXP.3, SJ31.2, SJ32.2, SJ33.2, SJ34.2, SJ35.2, SJ36.2, SJ37.2, SJ38.2, SJ39.2, SJ40.2, SJ41.2, SJ42.2, SJ43.2, SJ44.2, SJ45.2; no longer D31.C, D32.C, D33.C, D34.C, D35.C, D36.C, D37.C, D38.C, D39.C, D40.C, D41.C, D42.C, D43.C, D44.C, D45.C
- net R3: now also R169.2, ROW-EXP.4, SJ46.2, SJ47.2, SJ48.2, SJ49.2, SJ50.2, SJ51.2, SJ52.2, SJ53.2, SJ54.2, SJ55.2, SJ56.2, SJ57.2, SJ58.2, SJ59.2, SJ60.2; no longer D46.C, D47.C, D48.C, D49.C, D50.C, D51.C, D52.C, D53.C, D54.C, D55.C, D56.C, D57.C, D58.C, D59.C, D60.C
- net R4: now also R170.2, ROW-EXP.5, SJ61.2, SJ62.2, SJ63.2, SJ64.2, SJ65.2, SJ66.2, SJ69.2, SJ70.2, SJ71.2, SJ72.2, SJ73.2, SJ74.2; no longer D61.C, D62.C, D63.C, D64.C, D65.C, D66.C, D67.C, D68.C, D69.C, D70.C
- net RST: now also ICSP.5, RST.2; no longer J1.5, S71.2
- net RX: now also EXP.4; no longer J2.4
- net SCK: now also ICSP.3, LED-EXP.5; no longer J1.3
- net SW61: now also D74.A, R5.1, R9.2, S68.SW2, S68.SW4, S79.SW1, S79.SW3; no longer D61.A, R146.1, R147.2, S61.SW2, S61.SW4
- net SW62: now also S72.SW2, S72.SW4; no longer S62.SW2, S62.SW4
- net SW63: now also S62.SW2, S62.SW4, S73.SW1, S73.SW3; no longer S63.SW2, S63.SW4
- net SW64: now also S63.SW1, S63.SW3, S74.SW2, S74.SW4; no longer S64.SW2, S64.SW4
- net SW65: now also S75.SW2, S75.SW4; no longer S65.SW2, S65.SW4
- net SW66: now also S64.SW2, S64.SW4, S76.SW1, S76.SW3; no longer S66.SW2, S66.SW4
- net SW67: now also S65.SW2, S65.SW4; no longer S67.SW2, S67.SW4
- net SW68: now also S66.SW2, S66.SW4; no longer S68.SW2, S68.SW4
- net SW69: now also S67.SW1, S67.SW3, S77.SW2, S77.SW4; no longer S69.SW2, S69.SW4
- net SW70: now also S78.SW2, S78.SW4; no longer S70.SW2, S70.SW4
- net TX: now also EXP.3; no longer J2.3
- net VBAT: now also EXP.2; no longer J2.2
- net VIN: now also EXP.5; no longer J2.5
Routing:
- net G1: track 0.00 -> 612.2 mm, vias 0 -> 26
- net G0: track 0.00 -> 479.1 mm, vias 0 -> 4
- net G2: track 0.00 -> 477.4 mm, vias 0 -> 4
- net LED0: track 0.00 -> 294.9 mm, vias 0 -> 2
- net LED3: track 0.00 -> 292.9 mm, vias 0 -> 2
- net LED1: track 0.00 -> 280.1 mm, vias 0 -> 2
- net LED2: track 0.00 -> 280.1 mm, vias 0 -> 2
- net R3: track 278.8 -> 0.00 mm
- net R2: track 278.8 -> 0.00 mm
- net R4: track 271.6 -> 0.00 mm
- net LED4: track 0.00 -> 253.3 mm, vias 0 -> 2
- net LED7: track 0.00 -> 251.4 mm, vias 0 -> 2
- net LED5: track 0.00 -> 240.7 mm, vias 0 -> 2
- net LED6: track 0.00 -> 240.7 mm, vias 0 -> 2
- net LED8: track 0.00 -> 211.9 mm, vias 0 -> 2
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