File: hardware/ION-60/Eagle/ION-60/ION-60.sch (EAGLE design)
At the start: 71 parts

Commit message: Edit PCB
Parts:
- S1, S15, S16, S30, S31, S44, S45, S56: device Jordi:CHERRY-MX-LED1X1.5 -> Jordi:CHERRY-MX-LED1X1
- S43: device Jordi:CHERRY-MX-LED1X2 -> Jordi:CHERRY-MX-LED1X1
- S60: device Jordi:CHERRY-MX-LED1X1.25 -> Jordi:CHERRY-MX-LED1X1
- S61, S62, S65, S66, S67: device Jordi:CHERRY-MX-LED1X1.25 -> Jordi:CHERRY-MX-LED1X1.5
- S63, S64: device Jordi:CHERRY-MX-LED1X2.75 -> Jordi:CHERRY-MX-LED1X1.5
- S68, S69, S70: device Jordi:CHERRY-MX-LED1X1 -> Jordi:CHERRY-MX-LED1X1.5
Other:
- moved on the sheet: S1, S10, S11, S12, S13, S14, S15, S16, S17, S18, S19, S2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

Commit message: Further additions to PCB
Parts:
- added D46: (no value), SparkFun-DiscreteSemi:DIODESOD123
- added IC1: TLC5947DAP, Jordi:TLC5947DAP
- added Y1: (no value), Jordi:CRYSTAL
Connections:
- new net N$10: U$1.XTAL2, Y1.2
- new net N$11: S1.LED1, S10.LED1, S11.LED1, S12.LED1, S13.LED1, S14.LED1, S15.LED1, S2.LED1, S3.LED1, S4.LED1, S5.LED1, S6.LED1, S7.LED1, S8.LED1, S9.LED1
- new net N$12: S1.LED2, S16.LED2, S31.LED2, S46.LED2, S61.LED2
- new net N$13: S17.LED2, S2.LED2, S32.LED2, S47.LED2
- new net N$14: S18.LED2, S3.LED2, S33.LED2, S48.LED2, S62.LED2
- new net N$15: D46.A, S46.SW2
- new net N$9: U$1.XTAL1, Y1.1
Changed lines of the file:
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@@
 <?xml version="1.0" encoding="utf-8"?>
 <!DOCTYPE eagle SYSTEM "eagle.dtd">
-<eagle version="6.5.0">
+<eagle version="7.2.0">
 <drawing>
 <settings>
@@
 <part name="S70" library="Jordi" deviceset="CHERRY-MX-LED" device="1X1.5"/>
 <part name="U$1" library="SparkFun-DigitalIC" deviceset="ATMEGA32U4" device="TQFP-44"/>
+<part name="Y1" library="Jordi" deviceset="CRYSTAL" device=""/>
+<part name="D46" library="SparkFun-DiscreteSemi" deviceset="DIODE" device="SOD123"/>
+<part name="IC1" library="Jordi" deviceset="TLC5947" device="DAP"/>
 </parts>
 <sheets>
@@
 <instance part="S70" gate="G$1" x="579.12" y="10.16"/>
 <instance part="U$1" gate="G$1" x="48.26" y="160.02"/>
+<instance part="Y1" gate="G$1" x="25.4" y="147.32" rot="R270"/>
+<instance part="D46" gate="G$1" x="33.02" y="38.1"/>
+<instance part="IC1" gate="G$1" x="116.84" y="147.32"/>
 </instances>
 <busses>
 </busses>
 <nets>
+<net name="N$9" class="0">
+<segment>
+<pinref part="U$1" gate="G$1" pin="XTAL1"/>
+<pinref part="Y1" gate="G$1" pin="1"/>
+<wire x1="30.48" y1="149.86" x2="25.4" y2="149.86" width="0.1524" layer="91"/>
+</segment>
+</net>
+<net name="N$10" class="0">
+<segment>
+<pinref part="U$1" gate="G$1" pin="XTAL2"/>
+<pinref part="Y1" gate="G$1" pin="2"/>
+<wire x1="30.48" y1="144.78" x2="25.4" y2="144.78" width="0.1524" layer="91"/>
+</segment>
+</net>
+<net name="N$11" class="0">
+<segment>
+<pinref part="S1" gate="G$1" pin="LED1"/>
+<wire x1="7.62" y1="88.9" x2="5.08" y2="88.9" width="0.1524" layer="91"/>
+<wire x1="5.08" y1="88.9" x2="5.08" y2="83.82" width="0.1524" layer="91"/>
+<wire x1="5.08" y1="83.82" x2="45.72" y2="83.82" width="0.1524" layer="91"/>
+<wire x1="45.72" y1="83.82" x2="45.72" y2="88.9" width="0.1524" layer="91"/>
+<pinref part="S2" gate="G$1" pin="LED1"/>
+<wire x1="45.72" y1="88.9" x2="48.26" y2="88.9" width="0.1524" layer="91"/>
+<wire x1="45.72" y1="83.82" x2="86.36" y2="83.82" width="0.1524" layer="91"/>
+<wire x1="86.36" y1="83.82" x2="86.36" y2="88.9" width="0.1524" layer="91"/>
+<pinref part="S3" gate="G$1" pin="LED1"/>
+<wire x1="86.36" y1="88.9" x2="88.9" y2="88.9" width="0.1524" layer="91"/>
+<wire x1="86.36" y1="83.82" x2="127" y2="83.82" width="0.1524" layer="91"/>
+<wire x1="127" y1="83.82" x2="127" y2="88.9" width="0.1524" layer="91"/>
+<pinref part="S4" gate="G$1" pin="LED1"/>
+<wire x1="127" y1="88.9" x2="129.54" y2="88.9" width="0.1524" layer="91"/>
+<wire x1="127" y1="83.82" x2="167.64" y2="83.82" width="0.1524" layer="91"/>
+<wire x1="167.64" y1="83.82" x2="167.64" y2="88.9" width="0.1524" layer="91"/>
+<pinref part="S5" gate="G$1" pin="LED1"/>
+<wire x1="167.64" y1="88.9" x2="170.18" y2="88.9" width="0.1524" layer="91"/>
+<wire x1="167.64" y1="83.82" x2="208.28" y2="83.82" width="0.1524" layer="91"/>
+<wire x1="208.28" y1="83.82" x2="208.28" y2="88.9" width="0.1524" layer="91"/>
+<pinref part="S6" gate="G$1" pin="LED1"/>
+<wire x1="208.28" y1="88.9" x2="210.82" y2="88.9" width="0.1524" layer="91"/>
+<wire x1="208.28" y1="83.82" x2="248.92" y2="83.82" width="0.1524" layer="91"/>
+<wire x1="248.92" y1="83.82" x2="248.92" y2="88.9" width="0.1524" layer="91"/>
+<pinref part="S7" gate="G$1" pin="LED1"/>
+<wire x1="248.92" y1="88.9" x2="251.46" y2="88.9" width="0.1524" layer="91"/>
+<wire x1="248.92" y1="83.82" x2="289.56" y2="83.82" width="0.1524" layer="91"/>
+<wire x1="289.56" y1="83.82" x2="289.56" y2="88.9" width="0.1524" layer="91"/>
+<pinref part="S8" gate="G$1" pin="LED1"/>
+<wire x1="289.56" y1="88.9" x2="292.1" y2="88.9" width="0.1524" layer="91"/>
+<wire x1="289.56" y1="83.82" x2="330.2" y2="83.82" width="0.1524" layer="91"/>
+<wire x1="330.2" y1="83.82" x2="330.2" y2="88.9" width="0.1524" layer="91"/>
+<pinref part="S9" gate="G$1" pin="LED1"/>
+<wire x1="330.2" y1="88.9" x2="332.74" y2="88.9" width="0.1524" layer="91"/>
+<wire x1="330.2" y1="83.82" x2="370.84" y2="83.82" width="0.1524" layer="91"/>
+<wire x1="370.84" y1="83.82" x2="370.84" y2="88.9" width="0.1524" layer="91"/>
+<pinref part="S10" gate="G$1" pin="LED1"/>
+<wire x1="370.84" y1="88.9" x2="373.38" y2="88.9" width="0.1524" layer="91"/>
+<wire x1="370.84" y1="83.82" x2="411.48" y2="83.82" width="0.1524" layer="91"/>
+<wire x1="411.48" y1="83.82" x2="411.48" y2="88.9" width="0.1524" layer="91"/>
+<pinref part="S11" gate="G$1" pin="LED1"/>
+<wire x1="411.48" y1="88.9" x2="414.02" y2="88.9" width="0.1524" layer="91"/>
+<wire x1="411.48" y1="83.82" x2="452.12" y2="83.82" width="0.1524" layer="91"/>
+<wire x1="452.12" y1="83.82" x2="452.12" y2="88.9" width="0.1524" layer="91"/>
+<pinref part="S12" gate="G$1" pin="LED1"/>
+<wire x1="452.12" y1="88.9" x2="454.66" y2="88.9" width="0.1524" layer="91"/>
+<wire x1="452.12" y1="83.82" x2="492.76" y2="83.82" width="0.1524" layer="91"/>
+<wire x1="492.76" y1="83.82" x2="492.76" y2="88.9" width="0.1524" layer="91"/>
+<pinref part="S13" gate="G$1" pin="LED1"/>
+<wire x1="492.76" y1="88.9" x2="495.3" y2="88.9" width="0.1524" layer="91"/>
+<wire x1="492.76" y1="83.82" x2="533.4" y2="83.82" width="0.1524" layer="91"/>
+<wire x1="533.4" y1="83.82" x2="533.4" y2="88.9" width="0.1524" layer="91"/>
+<pinref part="S14" gate="G$1" pin="LED1"/>
+<wire x1="533.4" y1="88.9" x2="535.94" y2="88.9" width="0.1524" layer="91"/>
+<wire x1="533.4" y1="83.82" x2="574.04" y2="83.82" width="0.1524" layer="91"/>
+<wire x1="574.04" y1="83.82" x2="574.04" y2="88.9" width="0.1524" layer="91"/>
+<pinref part="S15" gate="G$1" pin="LED1"/>
+<wire x1="574.04" y1="88.9" x2="576.58" y2="88.9" width="0.1524" layer="91"/>
+<junction x="45.72" y="83.82"/>
+<junction x="86.36" y="83.82"/>
+<junction x="127" y="83.82"/>
+<junction x="167.64" y="83.82"/>
+<junction x="208.28" y="83.82"/>
+<junction x="248.92" y="83.82"/>
+<junction x="289.56" y="83.82"/>
+<junction x="330.2" y="83.82"/>
+<junction x="370.84" y="83.82"/>
+<junction x="411.48" y="83.82"/>
+<junction x="452.12" y="83.82"/>
+<junction x="492.76" y="83.82"/>
+<junction x="533.4" y="83.82"/>
+</segment>
+</net>
+<net name="N$12" class="0">
+<segment>
+<pinref part="S1" gate="G$1" pin="LED2"/>
+<wire x1="33.02" y1="88.9" x2="38.1" y2="88.9" width="0.1524" layer="91"/>
+<wire x1="38.1" y1="88.9" x2="38.1" y2="68.58" width="0.1524" layer="91"/>
+<pinref part="S16" gate="G$1" pin="LED2"/>
+<wire x1="38.1" y1="68.58" x2="33.02" y2="68.58" width="0.1524" layer="91"/>
+<pinref part="S31" gate="G$1" pin="LED2"/>
+<wire x1="33.02" y1="48.26" x2="38.1" y2="48.26" width="0.1524" layer="91"/>
+<wire x1="38.1" y1="48.26" x2="38.1" y2="68.58" width="0.1524" layer="91"/>
+<pinref part="S46" gate="G$1" pin="LED2"/>
+<wire x1="33.02" y1="27.94" x2="38.1" y2="27.94" width="0.1524" layer="91"/>
+<wire x1="38.1" y1="27.94" x2="38.1" y2="48.26" width="0.1524" layer="91"/>
+<wire x1="38.1" y1="27.94" x2="38.1" y2="17.78" width="0.1524" layer="91"/>
+<wire x1="38.1" y1="17.78" x2="48.26" y2="17.78" width="0.1524" layer="91"/>
+<wire x1="48.26" y1="17.78" x2="48.26" y2="7.62" width="0.1524" layer="91"/>
+<pinref part="S61" gate="G$1" pin="LED2"/>
+<wire x1="48.26" y1="7.62" x2="43.18" y2="7.62" width="0.1524" layer="91"/>
+</segment>
+</net>
+<net name="N$13" class="0">
+<segment>
+<pinref part="S2" gate="G$1" pin="LED2"/>
+<wire x1="73.66" y1="88.9" x2="78.74" y2="88.9" width="0.1524" layer="91"/>
+<pinref part="S17" gate="G$1" pin="LED2"/>
+<wire x1="73.66" y1="68.58" x2="78.74" y2="68.58" width="0.1524" layer="91"/>
+<wire x1="78.74" y1="68.58" x2="78.74" y2="88.9" width="0.1524" layer="91"/>
+<pinref part="S32" gate="G$1" pin="LED2"/>
+<wire x1="73.66" y1="48.26" x2="78.74" y2="48.26" width="0.1524" layer="91"/>
+<wire x1="78.74" y1="48.26" x2="78.74" y2="68.58" width="0.1524" layer="91"/>
+<pinref part="S47" gate="G$1" pin="LED2"/>
+<wire x1="73.66" y1="27.94" x2="78.74" y2="27.94" width="0.1524" layer="91"/>
+<wire x1="78.74" y1="27.94" x2="78.74" y2="48.26" width="0.1524" layer="91"/>
+</segment>
+</net>
+<net name="N$14" class="0">
+<segment>
+<pinref part="S3" gate="G$1" pin="LED2"/>
+<wire x1="114.3" y1="88.9" x2="119.38" y2="88.9" width="0.1524" layer="91"/>
+<pinref part="S18" gate="G$1" pin="LED2"/>
+<wire x1="114.3" y1="68.58" x2="119.38" y2="68.58" width="0.1524" layer="91"/>
+<wire x1="119.38" y1="68.58" x2="119.38" y2="88.9" width="0.1524" layer="91"/>
+<pinref part="S33" gate="G$1" pin="LED2"/>
+<wire x1="114.3" y1="48.26" x2="119.38" y2="48.26" width="0.1524" layer="91"/>
+<wire x1="119.38" y1="48.26" x2="119.38" y2="68.58" width="0.1524" layer="91"/>
+<pinref part="S48" gate="G$1" pin="LED2"/>
+<wire x1="114.3" y1="27.94" x2="119.38" y2="27.94" width="0.1524" layer="91"/>
+<wire x1="119.38" y1="27.94" x2="119.38" y2="48.26" width="0.1524" layer="91"/>
+<pinref part="S62" gate="G$1" pin="LED2"/>
+<wire x1="104.14" y1="7.62" x2="119.38" y2="7.62" width="0.1524" layer="91"/>
+<wire x1="119.38" y1="7.62" x2="119.38" y2="27.94" width="0.1524" layer="91"/>
+</segment>
+</net>
+<net name="N$15" class="0">
+<segment>
+<pinref part="S46" gate="G$1" pin="SW2"/>
+<wire x1="33.02" y1="33.02" x2="35.56" y2="33.02" width="0.1524" layer="91"/>
+<wire x1="35.56" y1="33.02" x2="35.56" y2="35.56" width="0.1524" layer="91"/>
+<pinref part="D46" gate="G$1" pin="A"/>
+<wire x1="35.56" y1="35.56" x2="30.48" y2="35.56" width="0.1524" layer="91"/>
+<wire x1="30.48" y1="35.56" x2="30.48" y2="38.1" width="0.1524" layer="91"/>
+</segment>
+</net>
 </nets>
 </sheet>

Commit message: More work on PCB
Parts:
- added D1, D10, D11, D12, D13, D14, D15, D16, D17, D18, D19, D2, D20, D21, D22, D23, D24, D25, D26, D27, D28, D29, D3, D30, D31, D32, D33, D34, D35, D36, D37, D38, D39, D4, D40, D41, D42, D43, D44, D45, D47, D48, D49, D5, D50, D51, D52, D53, D54, D55, D56, D57, D58, D59, D6, D60, D61, D62, D63, D64, D65, D66, D67, D68, D69, D7, D70, D8, D9: (no value), SparkFun-DiscreteSemi:DIODESOD123
- added IC2: 74LS137D, 74xx-us:74LS137D
- added IC3, IC4: TLC5947DAP, Jordi:TLC5947DAP
- IC1: value TLC5947DAP -> 74LS137D; device Jordi:TLC5947DAP -> 74xx-us:74LS137D
- Y1: value (none) -> 16MHz
Connections:
- net N$11 renamed LED-A0
- new net +3V3: IC3.VCC, IC4.VCC, U$1.AVCC@24, U$1.AVCC@44, U$1.VCC@14, U$1.VCC@34
- new net A0: IC1A.A, IC2A.A, U$1.PF4(ADC4)
- new net A1: IC1A.B, IC2A.B, U$1.PF5(ADC5)
- new net A2: IC1A.C, IC2A.C, U$1.PF6(ADC6)
- new net A3: IC1A.G1, IC2A.G2, U$1.PF7(ADC7)
- new net AL: IC1A.GL, IC2A.GL
- new net C0: IC1A.Y7, S1.SW1, S16.SW1, S31.SW1, S46.SW1, S61.SW1
- new net C1: IC1A.Y6, S17.SW1, S2.SW1, S32.SW1, S47.SW1
- new net C10: IC2A.Y5, S11.SW1, S26.SW1, S41.SW1, S56.SW1
- new net C11: IC2A.Y4, S12.SW1, S27.SW1, S42.SW1, S57.SW1, S68.SW1
- new net C12: IC2A.Y3, S13.SW1, S28.SW1, S43.SW1, S58.SW1, S69.SW1
- new net C13: IC2A.Y2, S14.SW1, S29.SW1, S44.SW1, S59.SW1
- new net C14: IC2A.Y1, S15.SW1, S30.SW1, S45.SW1, S60.SW1, S70.SW1
- new net C2: IC1A.Y5, S18.SW1, S3.SW1, S33.SW1, S48.SW1, S62.SW1
- new net C3: IC1A.Y4, S19.SW1, S34.SW1, S4.SW1, S49.SW1, S63.SW1
- new net C4: IC1A.Y3, S20.SW1, S35.SW1, S5.SW1, S50.SW1
- new net C5: IC1A.Y2, S21.SW1, S36.SW1, S51.SW1, S6.SW1, S64.SW1
- new net C6: IC1A.Y1, S22.SW1, S37.SW1, S52.SW1, S65.SW1, S7.SW1
- new net C7: IC1A.Y0, S23.SW1, S38.SW1, S53.SW1, S8.SW1
- new net C8: IC2A.Y7, S24.SW1, S39.SW1, S54.SW1, S66.SW1, S9.SW1
- new net C9: IC2A.Y6, S10.SW1, S25.SW1, S40.SW1, S55.SW1, S67.SW1
- new net E0: IC1A.G2, U$1.PF0(ADC0)
- new net E1: IC2A.G1, U$1.PF1(ADC1)
- new net GND: IC3.GND, IC3.PAD, IC4.GND, IC4.PAD, U$1.GND@15, U$1.GND@23, U$1.GND@35, U$1.GND@43, U$1.UGND
- new net LED-A1: S16.LED1, S17.LED1, S18.LED1, S19.LED1, S20.LED1, S21.LED1, S22.LED1, S23.LED1, S24.LED1, S25.LED1, S26.LED1, S27.LED1, S28.LED1, S29.LED1, S30.LED1
- new net LED-A2: S31.LED1, S32.LED1, S33.LED1, S34.LED1, S35.LED1, S36.LED1, S37.LED1, S38.LED1, S39.LED1, S40.LED1, S41.LED1, S42.LED1, S43.LED1, S44.LED1, S45.LED1
- new net LED-A3: S46.LED1, S47.LED1, S48.LED1, S49.LED1, S50.LED1, S51.LED1, S52.LED1, S53.LED1, S54.LED1, S55.LED1, S56.LED1, S57.LED1, S58.LED1, S59.LED1, S60.LED1
- new net LED-A4: S61.LED1, S62.LED1, S63.LED1, S64.LED1, S65.LED1, S66.LED1, S67.LED1, S68.LED1, S69.LED1, S70.LED1
- new net LED-B0: IC3.OUT2, S1.D2, S16.D2, S31.D2, S46.D2, S61.D2
- new net LED-B1: IC3.OUT5, S17.D2, S2.D2, S32.D2, S47.D2
- new net LED-B10: S11.D2, S26.D2, S41.D2, S56.D2
- new net LED-B11: S12.D2, S27.D2, S42.D2, S57.D2, S68.D2
- new net LED-B12: S13.D2, S28.D2, S43.D2, S58.D2, S69.D2
- new net LED-B13: S14.D2, S29.D2, S44.D2, S59.D2
- new net LED-B14: S15.D2, S30.D2, S45.D2, S60.D2, S70.D2
- new net LED-B2: IC3.OUT8, S18.D2, S3.D2, S33.D2, S48.D2, S62.D2
- new net LED-B3: IC3.OUT11, S19.D2, S34.D2, S4.D2, S49.D2, S63.D2
- new net LED-B4: IC3.OUT14, S20.D2, S35.D2, S5.D2, S50.D2
- new net LED-B5: IC3.OUT17, S21.D2, S36.D2, S51.D2, S6.D2, S64.D2
- new net LED-B6: IC3.OUT20, S22.D2, S37.D2, S52.D2, S65.D2, S7.D2
- new net LED-B7: IC3.OUT23, S23.D2, S38.D2, S53.D2, S8.D2
- new net LED-B8: S24.D2, S39.D2, S54.D2, S66.D2, S9.D2
- new net LED-B9: S10.D2, S25.D2, S40.D2, S55.D2, S67.D2
- new net LED-G0: IC3.OUT0, S1.D1, S16.D1, S31.D1, S46.D1, S61.D1
- new net LED-G1: IC3.OUT3, S17.D1, S2.D1, S32.D1, S47.D1
- new net LED-G10: S11.D1, S26.D1, S41.D1, S56.D1
- new net LED-G11: S12.D1, S27.D1, S42.D1, S57.D1, S68.D1
- new net LED-G12: S13.D1, S28.D1, S43.D1, S58.D1, S69.D1
- new net LED-G13: S14.D1, S29.D1, S44.D1, S59.D1
- new net LED-G14: S15.D1, S30.D1, S45.D1, S60.D1, S70.D1
- new net LED-G2: IC3.OUT6, S18.D1, S3.D1, S33.D1, S48.D1, S62.D1
- new net LED-G3: IC3.OUT9, S19.D1, S34.D1, S4.D1, S49.D1, S63.D1
- new net LED-G4: IC3.OUT12, S20.D1, S35.D1, S5.D1, S50.D1
- new net LED-G5: IC3.OUT15, S21.D1, S36.D1, S51.D1, S6.D1, S64.D1
- new net LED-G6: IC3.OUT18, S22.D1, S37.D1, S52.D1, S65.D1, S7.D1
- new net LED-G7: IC3.OUT21, S23.D1, S38.D1, S53.D1, S8.D1
- new net LED-G8: S24.D1, S39.D1, S54.D1, S66.D1, S9.D1
- new net LED-G9: S10.D1, S25.D1, S40.D1, S55.D1, S67.D1
- new net LED-R0: IC3.OUT1, S1.LED2, S16.LED2, S31.LED2, S46.LED2, S61.LED2
- new net LED-R1: IC3.OUT4, S17.LED2, S2.LED2, S32.LED2, S47.LED2
- new net LED-R10: S11.LED2, S26.LED2, S41.LED2, S56.LED2
- new net LED-R11: S12.LED2, S27.LED2, S42.LED2, S57.LED2, S68.LED2
- new net LED-R12: S13.LED2, S28.LED2, S43.LED2, S58.LED2, S69.LED2
- new net LED-R13: S14.LED2, S29.LED2, S44.LED2, S59.LED2
- new net LED-R14: S15.LED2, S30.LED2, S45.LED2, S60.LED2, S70.LED2
- new net LED-R2: IC3.OUT7, S18.LED2, S3.LED2, S33.LED2, S48.LED2, S62.LED2
- new net LED-R3: IC3.OUT10, S19.LED2, S34.LED2, S4.LED2, S49.LED2, S63.LED2
- new net LED-R4: IC3.OUT13, S20.LED2, S35.LED2, S5.LED2, S50.LED2
- new net LED-R5: IC3.OUT16, S21.LED2, S36.LED2, S51.LED2, S6.LED2, S64.LED2
- new net LED-R6: IC3.OUT19, S22.LED2, S37.LED2, S52.LED2, S65.LED2, S7.LED2
- new net LED-R7: IC3.OUT22, S23.LED2, S38.LED2, S53.LED2, S8.LED2
- new net LED-R8: S24.LED2, S39.LED2, S54.LED2, S66.LED2, S9.LED2
- new net LED-R9: S10.LED2, S25.LED2, S40.LED2, S55.LED2, S67.LED2
- new net MISO: U$1.PB3(MISO)
- new net MOSI: IC3.SIN, U$1.PB2(MOSI)
- new net N$100: D29.A, S29.SW2
- new net N$101: D30.A, S30.SW2
- new net N$102: D45.A, S45.SW2
- new net N$103: D60.A, S60.SW2
- new net N$104: D70.A, S70.SW2
- new net N$11: D2.A, S2.SW2
- new net N$15: D53.A, S53.SW2
- new net N$16: D3.A, S3.SW2
- new net N$17: D4.A, S4.SW2
- new net N$18: D5.A, S5.SW2
- new net N$19: D6.A, S6.SW2
- new net N$20: D7.A, S7.SW2
- new net N$21: D8.A, S8.SW2
- new net N$22: D9.A, S9.SW2
- new net N$23: D10.A, S10.SW2
- new net N$24: D11.A, S11.SW2
- new net N$25: D12.A, S12.SW2
- new net N$26: D13.A, S13.SW2
- new net N$27: D14.A, S14.SW2
- new net N$28: D15.A, S15.SW2
- new net N$29: D1.A, S1.SW2
- new net N$30: D54.A, S54.SW2
- new net N$31: D66.A, S66.SW2
- new net N$32: D67.A, S67.SW2
- new net N$37: D55.A, S55.SW2
- new net N$38: D16.A, S16.SW2
- new net N$39: D17.A, S17.SW2
- new net N$40: D18.A, S18.SW2
- new net N$41: D19.A, S19.SW2
- new net N$42: D40.A, S40.SW2
- new net N$43: D25.A, S25.SW2
- new net N$45: D26.A, S26.SW2
- new net N$48: D41.A, S41.SW2
- new net N$49: D56.A, S56.SW2
- new net N$52: D68.A, S68.SW2
- new net N$53: D61.A, S61.SW2
- new net N$54: D57.A, S57.SW2
- new net N$56: D63.A, S63.SW2
- new net N$57: D62.A, S62.SW2
- new net N$58: D52.A, S52.SW2
- new net N$59: D51.A, S51.SW2
- new net N$60: D50.A, S50.SW2
- new net N$62: D42.A, S42.SW2
- new net N$64: D33.A, S33.SW2
- new net N$65: D34.A, S34.SW2
- new net N$66: D49.A, S49.SW2
- new net N$67: D32.A, S32.SW2
- new net N$68: D31.A, S31.SW2
- new net N$71: D20.A, S20.SW2
- new net N$72: D35.A, S35.SW2
- new net N$73: D48.A, S48.SW2
- new net N$76: D21.A, S21.SW2
- new net N$77: D36.A, S36.SW2
- new net N$79: D64.A, S64.SW2
- new net N$80: D47.A, S47.SW2
- new net N$81: D27.A, S27.SW2
- new net N$84: D22.A, S22.SW2
- new net N$85: D37.A, S37.SW2
- new net N$88: D65.A, S65.SW2
- new net N$89: D28.A, S28.SW2
- new net N$91: D23.A, S23.SW2
- new net N$92: D38.A, S38.SW2
- new net N$93: D43.A, S43.SW2
- new net N$96: D58.A, S58.SW2
- new net N$97: D69.A, S69.SW2
- new net N$98: D59.A, S59.SW2
- new net N$99: D44.A, S44.SW2
- new net R0: D1.C, D10.C, D11.C, D12.C, D13.C, D14.C, D15.C, D2.C, D3.C, D4.C, D5.C, D6.C, D7.C, D8.C, D9.C, U$1.PD0(SCL)
- new net R1: D16.C, D17.C, D18.C, D19.C, D20.C, D21.C, D22.C, D23.C, D24.C, D25.C, D26.C, D27.C, D28.C, D29.C, D30.C, U$1.PD1(SDA)
- new net R2: D31.C, D32.C, D33.C, D34.C, D35.C, D36.C, D37.C, D38.C, D39.C, D40.C, D41.C, D42.C, D43.C, D44.C, D45.C, U$1.PD2(RX)
- new net R3: D46.C, D47.C, D48.C, D49.C, D50.C, D51.C, D52.C, D53.C, D54.C, D55.C, D56.C, D57.C, D58.C, D59.C, D60.C, U$1.PD3(TX)
- new net R4: D61.C, D62.C, D63.C, D64.C, D65.C, D66.C, D67.C, D68.C, D69.C, D70.C, U$1.PD5
- new net SCK: IC3.SCLK, IC4.SCLK, U$1.PB1(SCK)
- new net SS: IC3.XLAT, IC4.XLAT, U$1.PB0(SS)
- net N$12: now also IC3.SOUT, IC4.SIN; no longer S1.LED2, S16.LED2, S31.LED2, S46.LED2, S61.LED2
- net N$13: now also D24.A, S24.SW2; no longer S17.LED2, S2.LED2, S32.LED2, S47.LED2
- net N$14: now also D39.A, S39.SW2; no longer S18.LED2, S3.LED2, S33.LED2, S48.LED2, S62.LED2
Other:
- moved on the sheet: D46, S1, S10, S11, S12, S13, S14, S15, S16, S17, S18, S19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

Commit message: Lots more work on main PCB
Parts:
- removed IC1, IC2: 74LS137D, 74xx-us:74LS137D
- added C1, C2: (no value), Jordi:CAPACITOR0603
- added C3, C4: 1uF, Jordi:CAPACITOR0603
- added C5, C6, C7, C8: 0.1uF, Jordi:CAPACITOR0603
- added D71, D72, D73, D74, D75: MOSFET-PSUPERSOT, Jordi:MOSFET-PSUPERSOT
- added D76, D77, D78, D79, D80: (no value), Jordi:BSS138SOT23
- added J1: (no value), Jordi:1X04M-0.1-PTH
- added J2: (no value), Jordi:1X06M-0.05-PTH
- added R1: 1K, Jordi:RESISTOR0603
- added R10, R16, R17, R18, R19, R20, R6, R7, R8, R9: 4.7k, Jordi:RESISTOR0603
- added R11, R12, R13, R14, R15, R21, R22, R23, R24, R25: 100, Jordi:RESISTOR0603
- added R2, R3: 22, Jordi:RESISTOR0603
- added R4, R5: (no value), Jordi:RESISTOR0603
- added S71: (no value), Jordi:SWITCH-TACTILESMD
- added U$2, U$3: 74LVC138AD, SparkFun-DigitalIC:74LVC138AD
Connections:
- net MOSI renamed SIN
- removed net AL: IC1A.GL, IC2A.GL
- removed net E0: IC1A.G2, U$1.PF0(ADC0)
- removed net E1: IC2A.G1, U$1.PF1(ADC1)
- removed net MISO: U$1.PB3(MISO)
- removed net SS: IC3.XLAT, IC4.XLAT, U$1.PB0(SS)
- new net !E1: U$1.PE6, U$2./E1, U$3./E1
- new net BLANK: IC3.BLANK, IC4.BLANK, U$1.PB0(SS)
- new net D+: R2.2, U$1.D+
- new net D-: R3.2, U$1.D-
- new net N$105: D76.B, R16.2, R21.2
- new net N$106: D78.B, R18.2, R23.2
- new net N$107: D79.B, R19.2, R24.2
- new net N$108: D80.B, R20.2, R25.2
- new net N$33: R1.2, U$1.PE2/!HWB
- new net N$34: C3.2, U$1.UCAP
- new net N$35: C5.2, U$1.AREF
- new net N$36: J1.2, R3.1
- new net N$44: J1.3, R2.1
- new net N$46: IC3.IREF, R4.1
- new net N$47: IC4.IREF, R5.1
- new net N$50: D71.G, R11.2, R6.1
- new net N$51: D71.D, S1.LED1, S10.LED1, S11.LED1, S12.LED1, S13.LED1, S14.LED1, S15.LED1, S2.LED1, S3.LED1, S4.LED1, S5.LED1, S6.LED1, S7.LED1, S8.LED1, S9.LED1
- new net N$55: D72.D, S16.LED1, S17.LED1, S18.LED1, S19.LED1, S20.LED1, S21.LED1, S22.LED1, S23.LED1, S24.LED1, S25.LED1, S26.LED1, S27.LED1, S28.LED1, S29.LED1, S30.LED1
- new net N$61: D73.D, S31.LED1, S32.LED1, S33.LED1, S34.LED1, S35.LED1, S36.LED1, S37.LED1, S38.LED1, S39.LED1, S40.LED1, S41.LED1, S42.LED1, S43.LED1, S44.LED1, S45.LED1
- new net N$63: D74.D, S46.LED1, S47.LED1, S48.LED1, S49.LED1, S50.LED1, S51.LED1, S52.LED1, S53.LED1, S54.LED1, S55.LED1, S56.LED1, S57.LED1, S58.LED1, S59.LED1, S60.LED1
- new net N$69: D75.G, R10.1, R15.2
- new net N$70: D74.G, R14.2, R9.1
- new net N$74: D73.G, R13.2, R8.1
- new net N$75: D72.G, R12.2, R7.1
- new net N$78: D75.D, S61.LED1, S62.LED1, S63.LED1, S64.LED1, S65.LED1, S66.LED1, S67.LED1, S68.LED1, S69.LED1, S70.LED1
- new net N$82: D76.C, R11.1
- new net N$83: D77.B, R17.2, R22.2
- new net N$87: D79.C, R14.1
- new net N$90: D78.C, R13.1
- new net N$94: D77.C, R12.1
- new net N$95: D80.C, R15.1
- new net RST: S71.3, S71.4, U$1.!RESET
- new net RX: J2.4, U$1.PD2(RX)
- new net TX: J2.3, U$1.PD3(TX)
- new net UVCC: C4.2, U$1.UVCC, U$1.VBUS
- new net VIN: D71.S, D72.S, D73.S, D74.S, D75.S, J1.4, J2.5, R10.2, R6.2, R7.2, R8.2, R9.2
- new net XLAT: IC3.XLAT, IC4.XLAT, U$1.PB3(MISO)
- net +3V3: now also C6.2, C7.2, C8.2, J2.6, U$2.E3, U$2.VCC, U$3.VCC
- net A0: now also U$1.PB4(ADC11), U$2.A0, U$3.A0; no longer IC1A.A, IC2A.A, U$1.PF4(ADC4)
- net A1: now also U$1.PB5(ADC12), U$2.A1, U$3.A1; no longer IC1A.B, IC2A.B, U$1.PF5(ADC5)
- net A2: now also U$1.PB6(ADC13), U$2.A2, U$3.A2; no longer IC1A.C, IC2A.C, U$1.PF6(ADC6)
- net A3: now also U$1.PB7, U$2./E2, U$3.E3; no longer IC1A.G1, IC2A.G2, U$1.PF7(ADC7)
- net C0: now also U$2./Y7; no longer IC1A.Y7
- net C1: now also U$2./Y6; no longer IC1A.Y6
- net C10: now also U$3./Y5; no longer IC2A.Y5
- net C11: now also U$3./Y4; no longer IC2A.Y4
- net C12: now also U$3./Y3; no longer IC2A.Y3
- net C13: now also U$3./Y2; no longer IC2A.Y2
- net C14: now also U$3./Y1; no longer IC2A.Y1
- net C2: now also U$2./Y5; no longer IC1A.Y5
- net C3: now also U$2./Y4; no longer IC1A.Y4
- net C4: now also U$2./Y3; no longer IC1A.Y3
- net C5: now also U$2./Y2; no longer IC1A.Y2
- net C6: now also U$2./Y1; no longer IC1A.Y1
- net C7: now also U$2./Y0; no longer IC1A.Y0
- net C8: now also U$3./Y7; no longer IC2A.Y7
- net C9: now also U$3./Y6; no longer IC2A.Y6
- net GND: now also C1.1, C2.1, C3.1, C4.1, C5.1, C6.1, C7.1, C8.1, D76.E, D77.E, D78.E, D79.E, D80.E, J1.1, J2.1, R1.1, R16.1, R17.1, R18.1, R19.1, R20.1, R4.2, R5.2, S71.1, S71.2, U$2.GND, U$3./E2, U$3.GND, Y1.GND
- net LED-A0: now also R21.1; no longer S1.LED1, S10.LED1, S11.LED1, S12.LED1, S13.LED1, S14.LED1, S15.LED1, S2.LED1, S3.LED1, S4.LED1, S5.LED1, S6.LED1, S7.LED1, S8.LED1, S9.LED1
- net LED-A1: now also R22.1; no longer S16.LED1, S17.LED1, S18.LED1, S19.LED1, S20.LED1, S21.LED1, S22.LED1, S23.LED1, S24.LED1, S25.LED1, S26.LED1, S27.LED1, S28.LED1, S29.LED1, S30.LED1
- net LED-A2: now also R23.1; no longer S31.LED1, S32.LED1, S33.LED1, S34.LED1, S35.LED1, S36.LED1, S37.LED1, S38.LED1, S39.LED1, S40.LED1, S41.LED1, S42.LED1, S43.LED1, S44.LED1, S45.LED1
- net LED-A3: now also R24.1; no longer S46.LED1, S47.LED1, S48.LED1, S49.LED1, S50.LED1, S51.LED1, S52.LED1, S53.LED1, S54.LED1, S55.LED1, S56.LED1, S57.LED1, S58.LED1, S59.LED1, S60.LED1
- net LED-A4: now also R25.1; no longer S61.LED1, S62.LED1, S63.LED1, S64.LED1, S65.LED1, S66.LED1, S67.LED1, S68.LED1, S69.LED1, S70.LED1
- net LED-B10: now also IC4.OUT11
- net LED-B11: now also IC4.OUT14
- net LED-B12: now also IC4.OUT17
- net LED-B13: now also IC4.OUT20
- net LED-B14: now also IC4.OUT23
- net LED-B8: now also IC4.OUT5
- net LED-B9: now also IC4.OUT8
- net LED-G10: now also IC4.OUT9
- net LED-G11: now also IC4.OUT12
- net LED-G12: now also IC4.OUT15
- net LED-G13: now also IC4.OUT18
- net LED-G14: now also IC4.OUT21
- net LED-G8: now also IC4.OUT3
- net LED-G9: now also IC4.OUT6
- net LED-R10: now also IC4.OUT10
- net LED-R11: now also IC4.OUT13
- net LED-R12: now also IC4.OUT16
- net LED-R13: now also IC4.OUT19
- net LED-R14: now also IC4.OUT22
- net LED-R8: now also IC4.OUT4
- net LED-R9: now also IC4.OUT7
- net N$10: now also C2.2
- net N$9: now also C1.2
- net R0: no longer U$1.PD0(SCL)
- net R1: no longer U$1.PD1(SDA)
- net R2: no longer U$1.PD2(RX)
- net R3: no longer U$1.PD3(TX)
- net R4: no longer U$1.PD5
Other:
- moved on the sheet: IC4
