File: hardware/ION-60/Eagle/ION-60/ION-60.sch (EAGLE design)
At the start: 192 parts, among them IC3 TLC5947DAP, IC4 TLC5947DAP, Y1 16MHz

Commit message: Hardware debouncing and 5V VCC
Parts:
- added C10, C11, C12, C13, C14, C15, C16, C17, C18, C19, C20, C21, C22, C23, C24, C25, C26, C27, C28, C29, C30, C31, C32, C33, C34, C35, C36, C37, C38, C39, C40, C41, C42, C43, C44, C45, C46, C47, C48, C49, C50, C51, C52, C53, C54, C55, C56, C57, C58, C59, C60, C61, C62, C63, C64, C65, C66, C67, C68, C69, C70, C71, C72, C73, C74, C75, C76, C77, C78, C9: 1uF, Jordi:CAPACITOR0603
- added F1: 500mA, Jordi:FUSESMD-1812
- added IC1, IC10, IC11, IC12, IC13, IC14, IC15, IC16, IC17, IC18, IC19, IC2, IC20, IC21, IC22, IC23, IC24, IC25, IC26, IC27, IC28, IC29, IC30, IC31, IC32, IC33, IC34, IC35, IC36, IC37, IC38, IC39, IC40, IC41, IC42, IC43, IC44, IC45, IC46, IC47, IC48, IC49, IC5, IC50, IC51, IC52, IC53, IC54, IC55, IC56, IC57, IC58, IC59, IC6, IC60, IC61, IC62, IC63, IC64, IC65, IC66, IC67, IC68, IC69, IC7, IC70, IC71, IC72, IC8, IC9: 74LVC1G14DCK, 74xx-little-us:74LVC1G14DCK
- added JP1, JP2, JP3, JP4: USB-MICROBSMD, Jordi:USB-MICROBSMD
- added R100, R102, R104, R106, R108, R110, R112, R114, R116, R118, R120, R122, R124, R126, R128, R130, R132, R134, R136, R138, R140, R142, R144, R146, R148, R150, R152, R154, R156, R158, R160, R162, R164, R27, R28, R30, R32, R34, R36, R38, R40, R42, R44, R46, R48, R50, R52, R54, R56, R58, R60, R62, R64, R66, R68, R70, R72, R74, R76, R78, R80, R82, R84, R86, R88, R90, R92, R94, R96, R98: 4.7k?, Jordi:RESISTOR0603
- added R101, R103, R105, R107, R109, R111, R113, R115, R117, R119, R121, R123, R125, R127, R129, R131, R133, R135, R137, R139, R141, R143, R145, R147, R149, R151, R153, R155, R157, R159, R161, R163, R165, R26, R29, R31, R33, R35, R37, R39, R41, R43, R45, R47, R49, R51, R53, R55, R57, R59, R61, R63, R65, R67, R69, R71, R73, R75, R77, R79, R81, R83, R85, R87, R89, R91, R93, R95, R97, R99: 22k?, Jordi:RESISTOR0603
- J1: device Jordi:1X04M-0.1-PTH -> Jordi:2X03M-0.1-PTH-SHROUDED
- J2, S71: value (none) -> change
- R4, R5: value (none) -> 2.4k/3k
Connections:
- removed net +3V3: C6.2, C7.2, C8.2, IC3.VCC, IC4.VCC, J2.6, U$1.AVCC@24, U$1.AVCC@44, U$1.VCC@14, U$1.VCC@34, U$2.E3, U$2.VCC, U$3.VCC
- removed net C0: S1.SW1, S16.SW1, S31.SW1, S46.SW1, S61.SW1, U$2./Y7
- removed net N$100: D29.A, S29.SW2
- removed net N$101: D30.A, S30.SW2
- removed net N$102: D45.A, S45.SW2
- removed net N$103: D60.A, S60.SW2
- removed net N$13: D24.A, S24.SW2
- removed net N$14: D39.A, S39.SW2
- removed net N$15: D53.A, S53.SW2
- removed net N$16: D3.A, S3.SW2
- removed net N$21: D8.A, S8.SW2
- removed net N$30: D54.A, S54.SW2
- removed net N$31: D66.A, S66.SW2
- removed net N$32: D67.A, S67.SW2
- removed net N$37: D55.A, S55.SW2
- removed net N$38: D16.A, S16.SW2
- removed net N$39: D17.A, S17.SW2
- removed net N$40: D18.A, S18.SW2
- removed net N$41: D19.A, S19.SW2
- removed net N$42: D40.A, S40.SW2
- removed net N$43: D25.A, S25.SW2
- removed net N$45: D26.A, S26.SW2
- removed net N$48: D41.A, S41.SW2
- removed net N$49: D56.A, S56.SW2
- removed net N$52: D68.A, S68.SW2
- removed net N$53: D61.A, S61.SW2
- removed net N$54: D57.A, S57.SW2
- removed net N$56: D63.A, S63.SW2
- removed net N$57: D62.A, S62.SW2
- removed net N$58: D52.A, S52.SW2
- removed net N$59: D51.A, S51.SW2
- removed net N$60: D50.A, S50.SW2
- removed net N$62: D42.A, S42.SW2
- removed net N$64: D33.A, S33.SW2
- removed net N$65: D34.A, S34.SW2
- removed net N$66: D49.A, S49.SW2
- removed net N$67: D32.A, S32.SW2
- removed net N$68: D31.A, S31.SW2
- removed net N$71: D20.A, S20.SW2
- removed net N$72: D35.A, S35.SW2
- removed net N$73: D48.A, S48.SW2
- removed net N$76: D21.A, S21.SW2
- removed net N$77: D36.A, S36.SW2
- removed net N$79: D64.A, S64.SW2
- removed net N$80: D47.A, S47.SW2
- removed net N$81: D27.A, S27.SW2
- removed net N$84: D22.A, S22.SW2
- removed net N$85: D37.A, S37.SW2
- removed net N$86: D46.A, S46.SW2
- removed net N$88: D65.A, S65.SW2
- removed net N$89: D28.A, S28.SW2
- removed net N$91: D23.A, S23.SW2
- removed net N$92: D38.A, S38.SW2
- removed net N$93: D43.A, S43.SW2
- removed net N$96: D58.A, S58.SW2
- removed net N$97: D69.A, S69.SW2
- removed net N$98: D59.A, S59.SW2
- removed net N$99: D44.A, S44.SW2
- removed net SIN: IC3.SIN, U$1.PB2(MOSI)
- removed net VIN: D71.S, D72.S, D73.S, D74.S, D75.S, J1.4, J2.5, R10.2, R6.2, R7.2, R8.2, R9.2
- new net !C0: C24.1, C39.1, C54.1, C69.1, C9.1, S1.SW1, S16.SW1, S31.SW1, S46.SW1, S61.SW1, U$2./Y7
- new net !C1: C10.1, C25.1, C40.1, C55.1, S17.SW1, S2.SW1, S32.SW1, S47.SW1
- new net !C10: C19.1, C34.1, C49.1, C64.1, S11.SW1, S26.SW1, S41.SW1, S56.SW1
- new net !C11: C20.1, C35.1, C50.1, C65.1, S12.SW1, S27.SW1, S42.SW1, S57.SW1, S68.SW1
- new net !C12: C21.1, C36.1, C51.1, C66.1, C77.1, S13.SW1, S28.SW1, S43.SW1, S58.SW1, S69.SW1
- new net !C13: C22.1, C37.1, C52.1, C67.1, S14.SW1, S29.SW1, S44.SW1, S59.SW1
- new net !C14: C23.1, C38.1, C53.1, C68.1, S15.SW1, S30.SW1, S45.SW1, S60.SW1, S70.SW1
- new net !C2: C11.1, C26.1, C41.1, C56.1, S18.SW1, S3.SW1, S33.SW1, S48.SW1, S62.SW1
- new net !C3: C12.1, C27.1, C42.1, C57.1, C71.1, S19.SW1, S34.SW1, S4.SW1, S49.SW1, S63.SW1
- new net !C4: C13.1, C28.1, C43.1, C58.1, S20.SW1, S35.SW1, S5.SW1, S50.SW1
- new net !C5: C14.1, C29.1, C44.1, C59.1, S21.SW1, S36.SW1, S51.SW1, S6.SW1, S64.SW1
- new net !C6: C15.1, C30.1, C45.1, C60.1, C73.1, S22.SW1, S37.SW1, S52.SW1, S65.SW1, S7.SW1
- new net !C7: C16.1, C31.1, C46.1, C61.1, S23.SW1, S38.SW1, S53.SW1, S8.SW1
- new net !C8: C17.1, C32.1, C47.1, C62.1, S24.SW1, S39.SW1, S54.SW1, S66.SW1, S9.SW1
- new net !C9: C18.1, C33.1, C48.1, C63.1, C75.1, S10.SW1, S25.SW1, S40.SW1, S55.SW1, S67.SW1
- new net !COL: C9.2, IC1A.I, R26.1
- new net !COL1: C10.2, IC2A.I, R29.1
- new net !COL10: C19.2, IC13A.I, R47.1
- new net !COL11: C20.2, IC14A.I, R49.1
- new net !COL12: C21.2, IC15A.I, R51.1
- new net !COL13: C22.2, IC16A.I, R53.1
- new net !COL14: C23.2, IC17A.I, R55.1
- new net !COL15: C24.2, IC18A.I, R57.1
- new net !COL16: C25.2, IC19A.I, R59.1
- new net !COL17: C26.2, IC20A.I, R61.1
- new net !COL18: C27.2, IC21A.I, R63.1
- new net !COL19: C28.2, IC22A.I, R65.1
- new net !COL2: C11.2, IC5A.I, R31.1
- new net !COL20: C29.2, IC23A.I, R67.1
- new net !COL21: C30.2, IC24A.I, R69.1
- new net !COL22: C31.2, IC25A.I, R71.1
- new net !COL23: C32.2, IC26A.I, R73.1
- new net !COL24: C33.2, IC27A.I, R75.1
- new net !COL25: C34.2, IC28A.I, R77.1
- new net !COL26: C35.2, IC29A.I, R79.1
- new net !COL27: C36.2, IC30A.I, R81.1
- new net !COL28: C37.2, IC31A.I, R83.1
- new net !COL29: C38.2, IC32A.I, R85.1
- new net !COL3: C12.2, IC6A.I, R33.1
- new net !COL30: C39.2, IC33A.I, R87.1
- new net !COL31: C40.2, IC34A.I, R89.1
- new net !COL32: C41.2, IC35A.I, R91.1
- new net !COL33: C42.2, IC36A.I, R93.1
- new net !COL34: C43.2, IC37A.I, R95.1
- new net !COL35: C44.2, IC38A.I, R97.1
- new net !COL36: C45.2, IC39A.I, R99.1
- new net !COL37: C46.2, IC40A.I, R101.1
- new net !COL38: C47.2, IC41A.I, R103.1
- new net !COL39: C48.2, IC42A.I, R105.1
- new net !COL4: C13.2, IC7A.I, R35.1
- new net !COL40: C49.2, IC43A.I, R107.1
- new net !COL41: C50.2, IC44A.I, R109.1
- new net !COL42: C51.2, IC45A.I, R111.1
- new net !COL43: C52.2, IC46A.I, R113.1
- new net !COL44: C53.2, IC47A.I, R115.1
- new net !COL45: C54.2, IC48A.I, R117.1
- new net !COL46: C55.2, IC49A.I, R119.1
- new net !COL47: C56.2, IC50A.I, R121.1
- new net !COL48: C57.2, IC51A.I, R123.1
- new net !COL49: C58.2, IC52A.I, R125.1
- new net !COL5: C14.2, IC8A.I, R37.1
- new net !COL50: C59.2, IC53A.I, R127.1
- new net !COL51: C60.2, IC54A.I, R129.1
- new net !COL52: C61.2, IC55A.I, R131.1
- new net !COL53: C62.2, IC56A.I, R133.1
- new net !COL54: C63.2, IC57A.I, R135.1
- new net !COL55: C64.2, IC58A.I, R137.1
- new net !COL56: C65.2, IC59A.I, R139.1
- new net !COL57: C66.2, IC60A.I, R141.1
- new net !COL58: C67.2, IC61A.I, R143.1
- new net !COL59: C68.2, IC62A.I, R145.1
- new net !COL6: C15.2, IC9A.I, R39.1
- new net !COL60: C69.2, IC63A.I, R147.1
- new net !COL61: C70.2, IC64A.I, R149.1
- new net !COL62: C71.2, IC65A.I, R151.1
- new net !COL63: C72.2, IC66A.I, R153.1
- new net !COL64: C73.2, IC67A.I, R155.1
- new net !COL65: C74.2, IC68A.I, R157.1
- new net !COL66: C75.2, IC69A.I, R159.1
- new net !COL67: C76.2, IC70A.I, R161.1
- new net !COL68: C77.2, IC71A.I, R163.1
- new net !COL69: C78.2, IC72A.I, R165.1
- new net !COL7: C16.2, IC10A.I, R41.1
- new net !COL8: C17.2, IC11A.I, R43.1
- new net !COL9: C18.2, IC12A.I, R45.1
- new net +5V: C6.2, C7.2, C8.2, D71.S, D72.S, D73.S, D74.S, D75.S, F1.2, IC10P.VCC, IC11P.VCC, IC12P.VCC, IC13P.VCC, IC14P.VCC, IC15P.VCC, IC16P.VCC, IC17P.VCC, IC18P.VCC, IC19P.VCC, IC1P.VCC, IC20P.VCC, IC21P.VCC, IC22P.VCC, IC23P.VCC, IC24P.VCC, IC25P.VCC, IC26P.VCC, IC27P.VCC, IC28P.VCC, IC29P.VCC, IC2P.VCC, IC3.VCC, IC30P.VCC, IC31P.VCC, IC32P.VCC, IC33P.VCC, IC34P.VCC, IC35P.VCC, IC36P.VCC, IC37P.VCC, IC38P.VCC, IC39P.VCC, IC4.VCC, IC40P.VCC, IC41P.VCC, IC42P.VCC, IC43P.VCC, IC44P.VCC, IC45P.VCC, IC46P.VCC, IC47P.VCC, IC48P.VCC, IC49P.VCC, IC50P.VCC, IC51P.VCC, IC52P.VCC, IC53P.VCC, IC54P.VCC, IC55P.VCC, IC56P.VCC, IC57P.VCC, IC58P.VCC, IC59P.VCC, IC5P.VCC, IC60P.VCC, IC61P.VCC, IC62P.VCC, IC63P.VCC, IC64P.VCC, IC65P.VCC, IC66P.VCC, IC67P.VCC, IC68P.VCC, IC69P.VCC, IC6P.VCC, IC70P.VCC, IC71P.VCC, IC72P.VCC, IC7P.VCC, IC8P.VCC, IC9P.VCC, J1.2, J2.6, R10.2, R100.2, R102.2, R104.2, R106.2, R108.2, R110.2, R112.2, R114.2, R116.2, R118.2, R120.2, R122.2, R124.2, R126.2, R128.2, R130.2, R132.2, R134.2, R136.2, R138.2, R140.2, R142.2, R144.2, R146.2, R148.2, R150.2, R152.2, R154.2, R156.2, R158.2, R160.2, R162.2, R164.2, R27.2, R28.2, R30.2, R32.2, R34.2, R36.2, R38.2, R40.2, R42.2, R44.2, R46.2, R48.2, R50.2, R52.2, R54.2, R56.2, R58.2, R6.2, R60.2, R62.2, R64.2, R66.2, R68.2, R7.2, R70.2, R72.2, R74.2, R76.2, R78.2, R8.2, R80.2, R82.2, R84.2, R86.2, R88.2, R9.2, R90.2, R92.2, R94.2, R96.2, R98.2, U$1.AVCC@24, U$1.AVCC@44, U$1.VCC@14, U$1.VCC@34, U$2.E3, U$2.VCC, U$3.VCC
- new net MISO: J1.1, U$1.PB3(MISO)
- new net MOSI: IC3.SIN, J1.4, U$1.PB2(MOSI)
- new net N$109: IC16A.O
- new net N$110: IC17A.O
- new net N$112: IC18A.O
- new net N$113: IC19A.O
- new net N$114: IC20A.O
- new net N$115: IC21A.O
- new net N$116: IC22A.O
- new net N$117: IC23A.O
- new net N$118: IC24A.O
- new net N$119: IC25A.O
- new net N$120: IC26A.O
- new net N$121: IC27A.O
- new net N$122: IC28A.O
- new net N$123: IC29A.O
- new net N$124: IC30A.O
- new net N$125: IC31A.O
- new net N$126: IC32A.O
- new net N$130: IC33A.O
- new net N$131: IC34A.O
- new net N$132: IC35A.O
- new net N$133: IC36A.O
- new net N$134: IC37A.O
- new net N$135: IC38A.O
- new net N$136: IC39A.O
- new net N$137: IC40A.O
- new net N$138: IC41A.O
- new net N$139: IC42A.O
- new net N$140: IC43A.O
- new net N$141: IC44A.O
- new net N$142: IC45A.O
- new net N$143: IC46A.O
- new net N$144: IC47A.O
- new net N$148: IC48A.O
- new net N$149: IC49A.O
- new net N$150: IC50A.O
- new net N$151: IC51A.O
- new net N$152: IC52A.O
- new net N$153: IC53A.O
- new net N$154: IC54A.O
- new net N$155: IC55A.O
- new net N$156: IC56A.O
- new net N$157: IC57A.O
- new net N$158: IC58A.O
- new net N$159: IC59A.O
- new net N$160: IC60A.O
- new net N$161: IC61A.O
- new net N$162: IC62A.O
- new net N$166: IC63A.O
- new net N$167: IC64A.O
- new net N$168: IC65A.O
- new net N$169: IC66A.O
- new net N$170: IC67A.O
- new net N$171: IC68A.O
- new net N$172: IC69A.O
- new net N$173: IC70A.O
- new net N$174: IC71A.O
- new net N$175: IC72A.O
- new net SW1: D1.A, R26.2, R27.1, S1.SW2
- new net SW10: D10.A, R44.1, R45.2, S10.SW2
- new net SW11: D11.A, R46.1, R47.2, S11.SW2
- new net SW12: D12.A, R48.1, R49.2, S12.SW2
- new net SW13: D13.A, R50.1, R51.2, S13.SW2
- new net SW14: D14.A, R52.1, R53.2, S14.SW2
- new net SW15: D15.A, R54.1, R55.2, S15.SW2
- new net SW16: D16.A, R56.1, R57.2, S16.SW2
- new net SW17: D17.A, R58.1, R59.2, S17.SW2
- new net SW18: D18.A, R60.1, R61.2, S18.SW2
- new net SW19: D19.A, R62.1, R63.2, S19.SW2
- new net SW2: D2.A, R28.1, R29.2, S2.SW2
- new net SW20: D20.A, R64.1, R65.2, S20.SW2
- new net SW21: D21.A, R66.1, R67.2, S21.SW2
- new net SW22: D22.A, R68.1, R69.2, S22.SW2
- new net SW23: D23.A, R70.1, R71.2, S23.SW2
- new net SW24: D24.A, R72.1, R73.2, S24.SW2
- new net SW25: D25.A, R74.1, R75.2, S25.SW2
- new net SW26: D26.A, R76.1, R77.2, S26.SW2
- new net SW27: D27.A, R78.1, R79.2, S27.SW2
- new net SW28: D28.A, R80.1, R81.2, S28.SW2
- new net SW29: D29.A, R82.1, R83.2, S29.SW2
- new net SW3: D3.A, R30.1, R31.2, S3.SW2
- new net SW30: D30.A, R84.1, R85.2, S30.SW2
- new net SW31: D31.A, R86.1, R87.2, S31.SW2
- new net SW32: D32.A, R88.1, R89.2, S32.SW2
- new net SW33: D33.A, R90.1, R91.2, S33.SW2
- new net SW34: D34.A, R92.1, R93.2, S34.SW2
- new net SW35: D35.A, R94.1, R95.2, S35.SW2
- new net SW36: D36.A, R96.1, R97.2, S36.SW2
- new net SW37: D37.A, R98.1, R99.2, S37.SW2
- new net SW38: D38.A, R100.1, R101.2, S38.SW2
- new net SW39: D39.A, R102.1, R103.2, S39.SW2
- new net SW4: D4.A, R32.1, R33.2, S4.SW2
- new net SW40: D40.A, R104.1, R105.2, S40.SW2
- new net SW41: D41.A, R106.1, R107.2, S41.SW2
- new net SW42: D42.A, R108.1, R109.2, S42.SW2
- new net SW43: D43.A, R110.1, R111.2, S43.SW2
- new net SW44: D44.A, R112.1, R113.2, S44.SW2
- new net SW45: D45.A, R114.1, R115.2, S45.SW2
- new net SW46: D46.A, R116.1, R117.2, S46.SW2
- new net SW47: D47.A, R118.1, R119.2, S47.SW2
- new net SW48: D48.A, R120.1, R121.2, S48.SW2
- new net SW49: D49.A, R122.1, R123.2, S49.SW2
- new net SW5: D5.A, R34.1, R35.2, S5.SW2
- new net SW50: D50.A, R124.1, R125.2, S50.SW2
- new net SW51: D51.A, R126.1, R127.2, S51.SW2
- new net SW52: D52.A, R128.1, R129.2, S52.SW2
- new net SW53: D53.A, R130.1, R131.2, S53.SW2
- new net SW54: D54.A, R132.1, R133.2, S54.SW2
- new net SW55: D55.A, R134.1, R135.2, S55.SW2
- new net SW56: D56.A, R136.1, R137.2, S56.SW2
- new net SW57: D57.A, R138.1, R139.2, S57.SW2
- new net SW58: D58.A, R140.1, R141.2, S58.SW2
- new net SW59: D59.A, R142.1, R143.2, S59.SW2
- new net SW6: D6.A, R36.1, R37.2, S6.SW2
- new net SW60: D60.A, R144.1, R145.2, S60.SW2
- new net SW61: D61.A, R146.1, R147.2, S61.SW2
- new net SW62: D62.A, R148.1, R149.2, S62.SW2
- new net SW63: D63.A, R150.1, R151.2, S63.SW2
- new net SW64: D64.A, R152.1, R153.2, S64.SW2
- new net SW65: D65.A, R154.1, R155.2, S65.SW2
- new net SW66: D66.A, R156.1, R157.2, S66.SW2
- new net SW67: D67.A, R158.1, R159.2, S67.SW2
- new net SW68: D68.A, R160.1, R161.2, S68.SW2
- new net SW69: D69.A, R162.1, R163.2, S69.SW2
- new net SW7: D7.A, R38.1, R39.2, S7.SW2
- new net SW70: D70.A, R164.1, R165.2, S70.SW2
- new net SW8: D8.A, R40.1, R41.2, S8.SW2
- new net SW9: D9.A, R42.1, R43.2, S9.SW2
- net C1: no longer S17.SW1, S2.SW1, S32.SW1, S47.SW1
- net C10: no longer S11.SW1, S26.SW1, S41.SW1, S56.SW1
- net C11: no longer S12.SW1, S27.SW1, S42.SW1, S57.SW1, S68.SW1
- net C12: no longer S13.SW1, S28.SW1, S43.SW1, S58.SW1, S69.SW1
- net C13: no longer S14.SW1, S29.SW1, S44.SW1, S59.SW1
- net C14: no longer S15.SW1, S30.SW1, S45.SW1, S60.SW1, S70.SW1
- net C2: no longer S18.SW1, S3.SW1, S33.SW1, S48.SW1, S62.SW1
- net C3: no longer S19.SW1, S34.SW1, S4.SW1, S49.SW1, S63.SW1
- net C4: no longer S20.SW1, S35.SW1, S5.SW1, S50.SW1
- net C5: no longer S21.SW1, S36.SW1, S51.SW1, S6.SW1, S64.SW1
- net C6: no longer S22.SW1, S37.SW1, S52.SW1, S65.SW1, S7.SW1
- net C7: no longer S23.SW1, S38.SW1, S53.SW1, S8.SW1
- net C8: no longer S24.SW1, S39.SW1, S54.SW1, S66.SW1, S9.SW1
- net C9: no longer S10.SW1, S25.SW1, S40.SW1, S55.SW1, S67.SW1
- net D+: now also JP1.D+, JP2.D+, JP3.D+, JP4.D+, R2.1; no longer R2.2, U$1.D+
- net D-: now also JP1.D-, JP2.D-, JP3.D-, JP4.D-, R3.1; no longer R3.2, U$1.D-
- net GND: now also IC10P.GND, IC11P.GND, IC12P.GND, IC13P.GND, IC14P.GND, IC15P.GND, IC16P.GND, IC17P.GND, IC18P.GND, IC19P.GND, IC1P.GND, IC20P.GND, IC21P.GND, IC22P.GND, IC23P.GND, IC24P.GND, IC25P.GND, IC26P.GND, IC27P.GND, IC28P.GND, IC29P.GND, IC2P.GND, IC30P.GND, IC31P.GND, IC32P.GND, IC33P.GND, IC34P.GND, IC35P.GND, IC36P.GND, IC37P.GND, IC38P.GND, IC39P.GND, IC40P.GND, IC41P.GND, IC42P.GND, IC43P.GND, IC44P.GND, IC45P.GND, IC46P.GND, IC47P.GND, IC48P.GND, IC49P.GND, IC50P.GND, IC51P.GND, IC52P.GND, IC53P.GND, IC54P.GND, IC55P.GND, IC56P.GND, IC57P.GND, IC58P.GND, IC59P.GND, IC5P.GND, IC60P.GND, IC61P.GND, IC62P.GND, IC63P.GND, IC64P.GND, IC65P.GND, IC66P.GND, IC67P.GND, IC68P.GND, IC69P.GND, IC6P.GND, IC70P.GND, IC71P.GND, IC72P.GND, IC7P.GND, IC8P.GND, IC9P.GND, J1.6, JP1.GND, JP2.GND, JP3.GND, JP4.GND; no longer J1.1
- net LED-G11: now also C76.1
- net LED-G14: now also C78.1
- net LED-G2: now also C70.1
- net LED-G5: now also C72.1
- net LED-G8: now also C74.1
- net N$104: now also IC15A.O; no longer D70.A, S70.SW2
- net N$11: now also F1.1, JP1.VBUS, JP2.VBUS, JP3.VBUS, JP4.VBUS; no longer D2.A, S2.SW2
- net N$17: now also IC1A.O; no longer D4.A, S4.SW2
- net N$18: now also IC2A.O; no longer D5.A, S5.SW2
- net N$19: now also IC5A.O; no longer D6.A, S6.SW2
- net N$20: now also IC6A.O; no longer D7.A, S7.SW2
- net N$22: now also IC7A.O; no longer D9.A, S9.SW2
- net N$23: now also IC8A.O; no longer D10.A, S10.SW2
- net N$24: now also IC9A.O; no longer D11.A, S11.SW2
- net N$25: now also IC10A.O; no longer D12.A, S12.SW2
- net N$26: now also IC11A.O; no longer D13.A, S13.SW2
- net N$27: now also IC12A.O; no longer D14.A, S14.SW2
- net N$28: now also IC13A.O; no longer D15.A, S15.SW2
- net N$29: now also IC14A.O; no longer D1.A, S1.SW2
- net N$36: now also R2.2, U$1.D+; no longer J1.2, R3.1
- net N$44: now also R3.2, U$1.D-; no longer J1.3, R2.1
- net RST: now also J1.5
- net SCK: now also J1.3
- net XLAT: no longer U$1.PB3(MISO)
Other:
- note added: "change these (74hc595?)"
- note added: "check these"
- note added: "check values and packages"
- note added: "check xtal package"
- moved on the sheet: D1, D10, D11, D12, D13, D14, D15, D16, D17, D18, D19, D2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

Commit message: Back to 3V3 because LiPo
Parts:
- added C81: 470pF, Jordi:CAPACITOR0603
- added C82: 1uF, Jordi:CAPACITOR0603
- added D81: BAT20J, SparkFun-DiscreteSemi:DIODE-SCHOTTKY-BAT20J
- added IC73: VREG-5SOT23, Jordi:VREG-5SOT23
- added J3: (no value), Jordi:1X06M-0.1-PTH
- added Q1: MOSFET-PSUPERSOT, Jordi:MOSFET-PSUPERSOT
- added R168: 100K, Jordi:RESISTOR0603
- added USB: (no value), Jordi:1X04M-0.1-PTH
- R4, R5: value 2.4k/3k -> 4.7k/5.1k
Connections:
- removed net +5V: C6.2, C7.2, C8.2, D71.S, D72.S, D73.S, D74.S, D75.S, F1.2, IC10P.VCC, IC11P.VCC, IC12P.VCC, IC13P.VCC, IC14P.VCC, IC15P.VCC, IC16P.VCC, IC17P.VCC, IC18P.VCC, IC19P.VCC, IC1P.VCC, IC20P.VCC, IC21P.VCC, IC22P.VCC, IC23P.VCC, IC24P.VCC, IC25P.VCC, IC26P.VCC, IC27P.VCC, IC28P.VCC, IC29P.VCC, IC2P.VCC, IC3.VCC, IC30P.VCC, IC31P.VCC, IC32P.VCC, IC33P.VCC, IC34P.VCC, IC35P.VCC, IC36P.VCC, IC37P.VCC, IC38P.VCC, IC39P.VCC, IC4.VCC, IC40P.VCC, IC41P.VCC, IC42P.VCC, IC43P.VCC, IC44P.VCC, IC45P.VCC, IC46P.VCC, IC47P.VCC, IC48P.VCC, IC49P.VCC, IC50P.VCC, IC51P.VCC, IC52P.VCC, IC53P.VCC, IC54P.VCC, IC55P.VCC, IC56P.VCC, IC57P.VCC, IC58P.VCC, IC59P.VCC, IC5P.VCC, IC60P.VCC, IC61P.VCC, IC62P.VCC, IC63P.VCC, IC64P.VCC, IC65P.VCC, IC66P.VCC, IC67P.VCC, IC68P.VCC, IC69P.VCC, IC6P.VCC, IC70P.VCC, IC71P.VCC, IC72P.VCC, IC7P.VCC, IC8P.VCC, IC9P.VCC, J1.2, J2.6, R10.2, R100.2, R102.2, R104.2, R106.2, R108.2, R110.2, R112.2, R114.2, R116.2, R118.2, R120.2, R122.2, R124.2, R126.2, R128.2, R130.2, R132.2, R134.2, R136.2, R138.2, R140.2, R142.2, R144.2, R146.2, R148.2, R150.2, R152.2, R154.2, R156.2, R158.2, R160.2, R162.2, R164.2, R27.2, R28.2, R30.2, R32.2, R34.2, R36.2, R38.2, R40.2, R42.2, R44.2, R46.2, R48.2, R50.2, R52.2, R54.2, R56.2, R58.2, R6.2, R60.2, R62.2, R64.2, R66.2, R68.2, R7.2, R70.2, R72.2, R74.2, R76.2, R78.2, R8.2, R80.2, R82.2, R84.2, R86.2, R88.2, R9.2, R90.2, R92.2, R94.2, R96.2, R98.2, U$1.AVCC@24, U$1.AVCC@44, U$1.VCC@14, U$1.VCC@34, U$2.E3, U$2.VCC, U$3.VCC
- new net +3V3: C6.2, C7.2, C8.2, IC10P.VCC, IC11P.VCC, IC12P.VCC, IC13P.VCC, IC14P.VCC, IC15P.VCC, IC16P.VCC, IC17P.VCC, IC18P.VCC, IC19P.VCC, IC1P.VCC, IC20P.VCC, IC21P.VCC, IC22P.VCC, IC23P.VCC, IC24P.VCC, IC25P.VCC, IC26P.VCC, IC27P.VCC, IC28P.VCC, IC29P.VCC, IC2P.VCC, IC3.VCC, IC30P.VCC, IC31P.VCC, IC32P.VCC, IC33P.VCC, IC34P.VCC, IC35P.VCC, IC36P.VCC, IC37P.VCC, IC38P.VCC, IC39P.VCC, IC4.VCC, IC40P.VCC, IC41P.VCC, IC42P.VCC, IC43P.VCC, IC44P.VCC, IC45P.VCC, IC46P.VCC, IC47P.VCC, IC48P.VCC, IC49P.VCC, IC50P.VCC, IC51P.VCC, IC52P.VCC, IC53P.VCC, IC54P.VCC, IC55P.VCC, IC56P.VCC, IC57P.VCC, IC58P.VCC, IC59P.VCC, IC5P.VCC, IC60P.VCC, IC61P.VCC, IC62P.VCC, IC63P.VCC, IC64P.VCC, IC65P.VCC, IC66P.VCC, IC67P.VCC, IC68P.VCC, IC69P.VCC, IC6P.VCC, IC70P.VCC, IC71P.VCC, IC72P.VCC, IC73.OUT, IC7P.VCC, IC8P.VCC, IC9P.VCC, J1.2, J2.6, R100.2, R102.2, R104.2, R106.2, R108.2, R110.2, R112.2, R114.2, R116.2, R118.2, R120.2, R122.2, R124.2, R126.2, R128.2, R130.2, R132.2, R134.2, R136.2, R138.2, R140.2, R142.2, R144.2, R146.2, R148.2, R150.2, R152.2, R154.2, R156.2, R158.2, R160.2, R162.2, R164.2, R27.2, R28.2, R30.2, R32.2, R34.2, R36.2, R38.2, R40.2, R42.2, R44.2, R46.2, R48.2, R50.2, R52.2, R54.2, R56.2, R58.2, R60.2, R62.2, R64.2, R66.2, R68.2, R70.2, R72.2, R74.2, R76.2, R78.2, R80.2, R82.2, R84.2, R86.2, R88.2, R90.2, R92.2, R94.2, R96.2, R98.2, U$1.AVCC@24, U$1.AVCC@44, U$1.VCC@14, U$1.VCC@34, U$2.E3, U$2.VCC, U$3.VCC
- new net N$14: C81.1, IC73.BP
- new net SOUT: IC4.SOUT, J3.6
- new net VBAT: J2.2, Q1.D
- new net VCC: C82.2, D81.C, IC73.EN, IC73.IN, Q1.S
- new net VIN: D71.S, D72.S, D73.S, D74.S, D75.S, D81.A, F1.2, J2.5, Q1.G, R10.2, R168.2, R6.2, R7.2, R8.2, R9.2, USB.4
- net D+: now also USB.3
- net D-: now also USB.2
- net GND: now also C81.2, C82.1, IC73.GND, R168.1, USB.1
- net LED-A0: now also J3.1
- net LED-A1: now also J3.2
- net LED-A2: now also J3.3
- net LED-A3: now also J3.4
- net LED-A4: now also J3.5
Other:
- moved on the sheet: S71

Commit message: More work, maybe removing RGB LEDs after this
Connections:
- removed net C1: U$2./Y6
- removed net C10: U$3./Y5
- removed net C11: U$3./Y4
- removed net C12: U$3./Y3
- removed net C13: U$3./Y2
- removed net C14: U$3./Y1
- removed net C2: U$2./Y5
- removed net C3: U$2./Y4
- removed net C4: U$2./Y3
- removed net C5: U$2./Y2
- removed net C6: U$2./Y1
- removed net C7: U$2./Y0
- removed net C8: U$3./Y7
- removed net C9: U$3./Y6
- net !C1: now also U$2./Y6
- net !C10: now also U$3./Y5
- net !C11: now also U$3./Y4
- net !C12: now also U$3./Y3
- net !C13: now also U$3./Y2
- net !C14: now also U$3./Y1
- net !C2: now also U$2./Y5
- net !C3: now also U$2./Y4
- net !C4: now also U$2./Y3
- net !C5: now also U$2./Y2
- net !C6: now also U$2./Y1
- net !C7: now also U$2./Y0
- net !C8: now also U$3./Y7
- net !C9: now also U$3./Y6
Changed lines of the file:
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@@
 </segment>
 </net>
-<net name="C3" class="0">
-<segment>
-<wire x1="132.08" y1="147.32" x2="134.62" y2="147.32" width="0.1524" layer="91"/>
-<label x="134.62" y="147.32" size="1.778" layer="95"/>
-<pinref part="U$2" gate="G$1" pin="/Y4"/>
-</segment>
-</net>
 <net name="!C0" class="0">
 <segment>
@@
 </segment>
 </net>
-<net name="C2" class="0">
-<segment>
-<wire x1="132.08" y1="144.78" x2="134.62" y2="144.78" width="0.1524" layer="91"/>
-<label x="134.62" y="144.78" size="1.778" layer="95"/>
-<pinref part="U$2" gate="G$1" pin="/Y5"/>
-</segment>
-</net>
-<net name="C1" class="0">
-<segment>
-<wire x1="132.08" y1="142.24" x2="134.62" y2="142.24" width="0.1524" layer="91"/>
-<label x="134.62" y="142.24" size="1.778" layer="95"/>
-<pinref part="U$2" gate="G$1" pin="/Y6"/>
-</segment>
-</net>
 <net name="LED-G0" class="0">
 <segment>
@@
 </segment>
 </net>
-<net name="C4" class="0">
-<segment>
-<wire x1="132.08" y1="149.86" x2="134.62" y2="149.86" width="0.1524" layer="91"/>
-<label x="134.62" y="149.86" size="1.778" layer="95"/>
-<pinref part="U$2" gate="G$1" pin="/Y3"/>
-</segment>
-</net>
 <net name="LED-G1" class="0">
 <segment>
@@
 </segment>
 </net>
-<net name="C5" class="0">
-<segment>
-<wire x1="132.08" y1="152.4" x2="134.62" y2="152.4" width="0.1524" layer="91"/>
-<label x="134.62" y="152.4" size="1.778" layer="95"/>
-<pinref part="U$2" gate="G$1" pin="/Y2"/>
-</segment>
-</net>
 <net name="LED-G5" class="0">
 <segment>
@@
 </segment>
 </net>
-<net name="C6" class="0">
-<segment>
-<wire x1="132.08" y1="154.94" x2="134.62" y2="154.94" width="0.1524" layer="91"/>
-<label x="134.62" y="154.94" size="1.778" layer="95"/>
-<pinref part="U$2" gate="G$1" pin="/Y1"/>
-</segment>
-</net>
 <net name="LED-G6" class="0">
 <segment>
@@
 </segment>
 </net>
-<net name="C7" class="0">
-<segment>
-<wire x1="132.08" y1="157.48" x2="134.62" y2="157.48" width="0.1524" layer="91"/>
-<label x="134.62" y="157.48" size="1.778" layer="95"/>
-<pinref part="U$2" gate="G$1" pin="/Y0"/>
-</segment>
-</net>
 <net name="LED-G7" class="0">
 <segment>
@@
 </segment>
 </net>
-<net name="C8" class="0">
-<segment>
-<pinref part="U$3" gate="G$1" pin="/Y7"/>
-<wire x1="106.68" y1="175.26" x2="104.14" y2="175.26" width="0.1524" layer="91"/>
-<label x="104.14" y="175.26" size="1.778" layer="95" rot="R180"/>
-</segment>
-</net>
 <net name="LED-G8" class="0">
 <segment>
@@
 </segment>
 </net>
-<net name="C9" class="0">
-<segment>
-<wire x1="132.08" y1="172.72" x2="134.62" y2="172.72" width="0.1524" layer="91"/>
-<label x="134.62" y="172.72" size="1.778" layer="95"/>
-<pinref part="U$3" gate="G$1" pin="/Y6"/>
-</segment>
-</net>
 <net name="LED-G9" class="0">
 <segment>
@@
 </segment>
 </net>
-<net name="C10" class="0">
-<segment>
-<wire x1="132.08" y1="175.26" x2="134.62" y2="175.26" width="0.1524" layer="91"/>
-<label x="134.62" y="175.26" size="1.778" layer="95"/>
-<pinref part="U$3" gate="G$1" pin="/Y5"/>
-</segment>
-</net>
 <net name="LED-G10" class="0">
 <segment>
@@
 </segment>
 </net>
-<net name="C11" class="0">
-<segment>
-<wire x1="132.08" y1="177.8" x2="134.62" y2="177.8" width="0.1524" layer="91"/>
-<label x="134.62" y="177.8" size="1.778" layer="95"/>
-<pinref part="U$3" gate="G$1" pin="/Y4"/>
-</segment>
-</net>
 <net name="LED-G11" class="0">
 <segment>
@@
 </segment>
 </net>
-<net name="C12" class="0">
-<segment>
-<wire x1="132.08" y1="180.34" x2="134.62" y2="180.34" width="0.1524" layer="91"/>
-<label x="134.62" y="180.34" size="1.778" layer="95"/>
-<pinref part="U$3" gate="G$1" pin="/Y3"/>
-</segment>
-</net>
 <net name="LED-G12" class="0">
 <segment>
@@
 </segment>
 </net>
-<net name="C13" class="0">
-<segment>
-<wire x1="132.08" y1="182.88" x2="134.62" y2="182.88" width="0.1524" layer="91"/>
-<label x="134.62" y="182.88" size="1.778" layer="95"/>
-<pinref part="U$3" gate="G$1" pin="/Y2"/>
-</segment>
-</net>
 <net name="LED-G13" class="0">
 <segment>
@@
 </segment>
 </net>
-<net name="C14" class="0">
-<segment>
-<wire x1="132.08" y1="185.42" x2="134.62" y2="185.42" width="0.1524" layer="91"/>
-<label x="134.62" y="185.42" size="1.778" layer="95"/>
-<pinref part="U$3" gate="G$1" pin="/Y1"/>
-</segment>
-</net>
 <net name="LED-G14" class="0">
 <segment>
@@
 <junction x="43.18" y="-25.4"/>
 </segment>
+<segment>
+<wire x1="132.08" y1="142.24" x2="134.62" y2="142.24" width="0.1524" layer="91"/>
+<label x="134.62" y="142.24" size="1.778" layer="95"/>
+<pinref part="U$2" gate="G$1" pin="/Y6"/>
+</segment>
 </net>
 <net name="!C2" class="0">
@@
 <junction x="93.98" y="-25.4"/>
 </segment>
+<segment>
+<wire x1="132.08" y1="144.78" x2="134.62" y2="144.78" width="0.1524" layer="91"/>
+<label x="134.62" y="144.78" size="1.778" layer="95"/>
+<pinref part="U$2" gate="G$1" pin="/Y5"/>
+</segment>
 </net>
 <net name="!C3" class="0">
@@
 <junction x="144.78" y="-25.4"/>
 </segment>
+<segment>
+<wire x1="132.08" y1="147.32" x2="134.62" y2="147.32" width="0.1524" layer="91"/>
+<label x="134.62" y="147.32" size="1.778" layer="95"/>
+<pinref part="U$2" gate="G$1" pin="/Y4"/>
+</segment>
 </net>
 <net name="!C4" class="0">
@@
 <junction x="195.58" y="-25.4"/>
 </segment>
+<segment>
+<wire x1="132.08" y1="149.86" x2="134.62" y2="149.86" width="0.1524" layer="91"/>
+<label x="134.62" y="149.86" size="1.778" layer="95"/>
+<pinref part="U$2" gate="G$1" pin="/Y3"/>
+</segment>
 </net>
 <net name="!C5" class="0">
@@
 <junction x="246.38" y="-25.4"/>
 </segment>
+<segment>
+<wire x1="132.08" y1="152.4" x2="134.62" y2="152.4" width="0.1524" layer="91"/>
+<label x="134.62" y="152.4" size="1.778" layer="95"/>
+<pinref part="U$2" gate="G$1" pin="/Y2"/>
+</segment>
 </net>
 <net name="!C6" class="0">
@@
 <junction x="297.18" y="-25.4"/>
 </segment>
+<segment>
+<wire x1="132.08" y1="154.94" x2="134.62" y2="154.94" width="0.1524" layer="91"/>
+<label x="134.62" y="154.94" size="1.778" layer="95"/>
+<pinref part="U$2" gate="G$1" pin="/Y1"/>
+</segment>
 </net>
 <net name="!C7" class="0">
@@
 <junction x="347.98" y="-25.4"/>
 </segment>
+<segment>
+<wire x1="132.08" y1="157.48" x2="134.62" y2="157.48" width="0.1524" layer="91"/>
+<label x="134.62" y="157.48" size="1.778" layer="95"/>
+<pinref part="U$2" gate="G$1" pin="/Y0"/>
+</segment>
 </net>
 <net name="!C8" class="0">
@@
 <junction x="398.78" y="-25.4"/>
 </segment>
+<segment>
+<pinref part="U$3" gate="G$1" pin="/Y7"/>
+<wire x1="106.68" y1="175.26" x2="104.14" y2="175.26" width="0.1524" layer="91"/>
+<label x="104.14" y="175.26" size="1.778" layer="95" rot="R180"/>
+</segment>
 </net>
 <net name="!C9" class="0">
@@
 <junction x="449.58" y="-25.4"/>
 </segment>
+<segment>
+<wire x1="132.08" y1="172.72" x2="134.62" y2="172.72" width="0.1524" layer="91"/>
+<label x="134.62" y="172.72" size="1.778" layer="95"/>
+<pinref part="U$3" gate="G$1" pin="/Y6"/>
+</segment>
 </net>
 <net name="!C10" class="0">
@@
 <junction x="500.38" y="-25.4"/>
 </segment>
+<segment>
+<wire x1="132.08" y1="175.26" x2="134.62" y2="175.26" width="0.1524" layer="91"/>
+<label x="134.62" y="175.26" size="1.778" layer="95"/>
+<pinref part="U$3" gate="G$1" pin="/Y5"/>
+</segment>
 </net>
 <net name="!C11" class="0">
@@
 <junction x="551.18" y="-25.4"/>
 </segment>
+<segment>
+<wire x1="132.08" y1="177.8" x2="134.62" y2="177.8" width="0.1524" layer="91"/>
+<label x="134.62" y="177.8" size="1.778" layer="95"/>
+<pinref part="U$3" gate="G$1" pin="/Y4"/>
+</segment>
 </net>
 <net name="!C12" class="0">
@@
 <junction x="601.98" y="-25.4"/>
 </segment>
+<segment>
+<wire x1="132.08" y1="180.34" x2="134.62" y2="180.34" width="0.1524" layer="91"/>
+<label x="134.62" y="180.34" size="1.778" layer="95"/>
+<pinref part="U$3" gate="G$1" pin="/Y3"/>
+</segment>
 </net>
 <net name="!C13" class="0">
@@
 <junction x="652.78" y="-25.4"/>
 </segment>
+<segment>
+<wire x1="132.08" y1="182.88" x2="134.62" y2="182.88" width="0.1524" layer="91"/>
+<label x="134.62" y="182.88" size="1.778" layer="95"/>
+<pinref part="U$3" gate="G$1" pin="/Y2"/>
+</segment>
 </net>
 <net name="!C14" class="0">
@@
 <junction x="703.58" y="-25.4"/>
 </segment>
+<segment>
+<wire x1="132.08" y1="185.42" x2="134.62" y2="185.42" width="0.1524" layer="91"/>
+<label x="134.62" y="185.42" size="1.778" layer="95"/>
+<pinref part="U$3" gate="G$1" pin="/Y1"/>
+</segment>
 </net>

Commit message: Remove RGB LEDs, change reset switch
Parts:
- removed D74, D75: MOSFET-PSUPERSOT, Jordi:MOSFET-PSUPERSOT
- removed D79, D80: (no value), Jordi:BSS138SOT23
- removed IC4: TLC5947DAP, Jordi:TLC5947DAP
- removed R10, R19, R20, R9: 4.7k, Jordi:RESISTOR0603
- removed R14, R15, R24, R25: 100, Jordi:RESISTOR0603
- removed R5: 4.7k/5.1k, Jordi:RESISTOR0603
- added SJ1, SJ10, SJ11, SJ12, SJ13, SJ14, SJ15, SJ2, SJ3, SJ4, SJ5, SJ6, SJ7, SJ8, SJ9: JUMPER-PAD-3-2OF3_NC_BY_TRACE_SMALL, SparkFun-Passives:JUMPER-PAD-3-2OF3_NC_BY_TRACE_SMALL
- S71: value change -> RESET; device Jordi:SWITCH-TACTILESMD -> Jordi:SWITCH-TACTILESMD-RA
Connections:
- net !C0 renamed C0
- net !C1 renamed C1
- net !C10 renamed C10
- net !C12 renamed C12
- net !C13 renamed C13
- net !C3 renamed C3
- net !C4 renamed C4
- net !C6 renamed C6
- net !C7 renamed C7
- net !C9 renamed C9
- removed net !C11: C20.1, C35.1, C50.1, C65.1, S12.SW1, S27.SW1, S42.SW1, S57.SW1, S68.SW1, U$3./Y4
- removed net !C14: C23.1, C38.1, C53.1, C68.1, S15.SW1, S30.SW1, S45.SW1, S60.SW1, S70.SW1, U$3./Y1
- removed net !C2: C11.1, C26.1, C41.1, C56.1, S18.SW1, S3.SW1, S33.SW1, S48.SW1, S62.SW1, U$2./Y5
- removed net !C5: C14.1, C29.1, C44.1, C59.1, S21.SW1, S36.SW1, S51.SW1, S6.SW1, S64.SW1, U$2./Y2
- removed net !C8: C17.1, C32.1, C47.1, C62.1, S24.SW1, S39.SW1, S54.SW1, S66.SW1, S9.SW1, U$3./Y7
- removed net LED-B0: IC3.OUT2, S1.D2, S16.D2, S31.D2, S46.D2, S61.D2
- removed net LED-B1: IC3.OUT5, S17.D2, S2.D2, S32.D2, S47.D2
- removed net LED-B10: IC4.OUT11, S11.D2, S26.D2, S41.D2, S56.D2
- removed net LED-B11: IC4.OUT14, S12.D2, S27.D2, S42.D2, S57.D2, S68.D2
- removed net LED-B12: IC4.OUT17, S13.D2, S28.D2, S43.D2, S58.D2, S69.D2
- removed net LED-B13: IC4.OUT20, S14.D2, S29.D2, S44.D2, S59.D2
- removed net LED-B14: IC4.OUT23, S15.D2, S30.D2, S45.D2, S60.D2, S70.D2
- removed net LED-B2: IC3.OUT8, S18.D2, S3.D2, S33.D2, S48.D2, S62.D2
- removed net LED-B3: IC3.OUT11, S19.D2, S34.D2, S4.D2, S49.D2, S63.D2
- removed net LED-B4: IC3.OUT14, S20.D2, S35.D2, S5.D2, S50.D2
- removed net LED-B5: IC3.OUT17, S21.D2, S36.D2, S51.D2, S6.D2, S64.D2
- removed net LED-B6: IC3.OUT20, S22.D2, S37.D2, S52.D2, S65.D2, S7.D2
- removed net LED-B7: IC3.OUT23, S23.D2, S38.D2, S53.D2, S8.D2
- removed net LED-B8: IC4.OUT5, S24.D2, S39.D2, S54.D2, S66.D2, S9.D2
- removed net LED-B9: IC4.OUT8, S10.D2, S25.D2, S40.D2, S55.D2, S67.D2
- removed net LED-G0: IC3.OUT0, S1.D1, S16.D1, S31.D1, S46.D1, S61.D1
- removed net LED-G1: IC3.OUT3, S17.D1, S2.D1, S32.D1, S47.D1
- removed net LED-G10: IC4.OUT9, S11.D1, S26.D1, S41.D1, S56.D1
- removed net LED-G11: C76.1, IC4.OUT12, S12.D1, S27.D1, S42.D1, S57.D1, S68.D1
- removed net LED-G12: IC4.OUT15, S13.D1, S28.D1, S43.D1, S58.D1, S69.D1
- removed net LED-G13: IC4.OUT18, S14.D1, S29.D1, S44.D1, S59.D1
- removed net LED-G14: C78.1, IC4.OUT21, S15.D1, S30.D1, S45.D1, S60.D1, S70.D1
- removed net LED-G2: C70.1, IC3.OUT6, S18.D1, S3.D1, S33.D1, S48.D1, S62.D1
- removed net LED-G3: IC3.OUT9, S19.D1, S34.D1, S4.D1, S49.D1, S63.D1
- removed net LED-G4: IC3.OUT12, S20.D1, S35.D1, S5.D1, S50.D1
- removed net LED-G5: C72.1, IC3.OUT15, S21.D1, S36.D1, S51.D1, S6.D1, S64.D1
- removed net LED-G6: IC3.OUT18, S22.D1, S37.D1, S52.D1, S65.D1, S7.D1
- removed net LED-G7: IC3.OUT21, S23.D1, S38.D1, S53.D1, S8.D1
- removed net LED-G8: C74.1, IC4.OUT3, S24.D1, S39.D1, S54.D1, S66.D1, S9.D1
- removed net LED-G9: IC4.OUT6, S10.D1, S25.D1, S40.D1, S55.D1, S67.D1
- removed net LED-R0: IC3.OUT1, S1.LED2, S16.LED2, S31.LED2, S46.LED2, S61.LED2
- removed net LED-R1: IC3.OUT4, S17.LED2, S2.LED2, S32.LED2, S47.LED2
- removed net LED-R10: IC4.OUT10, S11.LED2, S26.LED2, S41.LED2, S56.LED2
- removed net LED-R11: IC4.OUT13, S12.LED2, S27.LED2, S42.LED2, S57.LED2, S68.LED2
- removed net LED-R12: IC4.OUT16, S13.LED2, S28.LED2, S43.LED2, S58.LED2, S69.LED2
- removed net LED-R13: IC4.OUT19, S14.LED2, S29.LED2, S44.LED2, S59.LED2
- removed net LED-R14: IC4.OUT22, S15.LED2, S30.LED2, S45.LED2, S60.LED2, S70.LED2
- removed net LED-R2: IC3.OUT7, S18.LED2, S3.LED2, S33.LED2, S48.LED2, S62.LED2
- removed net LED-R3: IC3.OUT10, S19.LED2, S34.LED2, S4.LED2, S49.LED2, S63.LED2
- removed net LED-R4: IC3.OUT13, S20.LED2, S35.LED2, S5.LED2, S50.LED2
- removed net LED-R5: IC3.OUT16, S21.LED2, S36.LED2, S51.LED2, S6.LED2, S64.LED2
- removed net LED-R6: IC3.OUT19, S22.LED2, S37.LED2, S52.LED2, S65.LED2, S7.LED2
- removed net LED-R7: IC3.OUT22, S23.LED2, S38.LED2, S53.LED2, S8.LED2
- removed net LED-R8: IC4.OUT4, S24.LED2, S39.LED2, S54.LED2, S66.LED2, S9.LED2
- removed net LED-R9: IC4.OUT7, S10.LED2, S25.LED2, S40.LED2, S55.LED2, S67.LED2
- removed net N$104: IC15A.O
- removed net N$107: D79.B, R19.2, R24.2
- removed net N$108: D80.B, R20.2, R25.2
- removed net N$109: IC16A.O
- removed net N$110: IC17A.O
- removed net N$69: D75.G, R10.1, R15.2
- removed net N$70: D74.G, R14.2, R9.1
- removed net N$87: D79.C, R14.1
- removed net N$95: D80.C, R15.1
- new net C11: C20.1, C35.1, C50.1, C65.1, C76.1, S12.SW1, S27.SW1, S42.SW1, S57.SW1, S68.SW1, U$3./Y4
- new net C14: C23.1, C38.1, C53.1, C68.1, C78.1, S15.SW1, S30.SW1, S45.SW1, S60.SW1, S70.SW1, U$3./Y1
- new net C2: C11.1, C26.1, C41.1, C56.1, C70.1, S18.SW1, S3.SW1, S33.SW1, S48.SW1, S62.SW1, U$2./Y5
- new net C5: C14.1, C29.1, C44.1, C59.1, C72.1, S21.SW1, S36.SW1, S51.SW1, S6.SW1, S64.SW1, U$2./Y2
- new net C8: C17.1, C32.1, C47.1, C62.1, C74.1, S24.SW1, S39.SW1, S54.SW1, S66.SW1, S9.SW1, U$3./Y7
- new net LED0: IC3.OUT0
- new net LED1: IC3.OUT1
- new net LED10: IC3.OUT10
- new net LED11: IC3.OUT11
- new net LED12: IC3.OUT12
- new net LED13: IC3.OUT13
- new net LED14: IC3.OUT14
- new net LED15: IC3.OUT15
- new net LED16: IC3.OUT16
- new net LED17: IC3.OUT17
- new net LED18: IC3.OUT18
- new net LED19: IC3.OUT19
- new net LED2: IC3.OUT2
- new net LED20: IC3.OUT20
- new net LED21: IC3.OUT21
- new net LED22: IC3.OUT22
- new net LED23: IC3.OUT23
- new net LED3: IC3.OUT3
- new net LED4: IC3.OUT4
- new net LED5: IC3.OUT5
- new net LED6: IC3.OUT6
- new net LED7: IC3.OUT7
- new net LED8: IC3.OUT8
- new net LED9: IC3.OUT9
- new net N$13: S16.LED1, S17.LED1, S18.LED1, S19.LED1, S20.LED1
- new net N$15: S31.LED1, S32.LED1, S33.LED1, S34.LED1, S35.LED1
- new net N$16: S46.LED1, S47.LED1, S48.LED1, S49.LED1, S50.LED1
- new net N$21: S61.LED1, S62.LED1, S63.LED1
- new net N$30: S68.LED1, S69.LED1, S70.LED1
- new net N$31: S56.LED1, S57.LED1, S58.LED1, S59.LED1, S60.LED1
- new net N$32: S41.LED1, S42.LED1, S43.LED1, S44.LED1, S45.LED1
- new net N$37: S26.LED1, S27.LED1, S28.LED1, S29.LED1, S30.LED1
- new net N$38: S11.LED1, S12.LED1, S13.LED1, S14.LED1, S15.LED1
- new net N$39: IC1A.O, SJ1.3
- new net N$40: D2.C, SJ2.1
- new net N$41: D73.D
- new net N$42: D72.D
- new net N$43: D71.D
- new net N$45: D76.E, D77.E, D78.E, R16.1, R17.1, R18.1
- new net N$48: D4.C, SJ4.1
- new net N$49: D5.C, SJ5.1
- new net N$52: D6.C, SJ6.1
- new net N$53: D7.C, SJ7.1
- new net N$54: IC5A.O, SJ3.3
- new net N$56: IC6A.O, SJ4.3
- new net N$57: IC7A.O, SJ5.3
- new net N$58: D8.C, SJ8.1
- new net N$59: D9.C, SJ9.1
- new net N$60: D10.C, SJ10.1
- new net N$62: D11.C, SJ11.1
- new net N$64: D12.C, SJ12.1
- new net N$65: D13.C, SJ13.1
- new net N$66: D14.C, SJ14.1
- new net N$67: D15.C, SJ15.1
- net +3V3: no longer IC4.VCC
- net BLANK: no longer IC4.BLANK
- net GND: no longer D76.E, D77.E, D78.E, D79.E, D80.E, IC4.GND, IC4.PAD, R16.1, R17.1, R18.1, R19.1, R20.1, R5.2, S71.2
- net LED-A3: no longer R24.1
- net LED-A4: no longer R25.1
- net N$12: now also S1.LED1, S2.LED1, S3.LED1, S4.LED1, S5.LED1; no longer IC3.SOUT, IC4.SIN
- net N$17: now also D1.C, SJ1.1; no longer IC1A.O
- net N$18: now also IC8A.O, SJ6.3; no longer IC2A.O
- net N$19: now also IC9A.O, SJ7.3; no longer IC5A.O
- net N$20: now also IC10A.O, SJ8.3; no longer IC6A.O
- net N$22: now also IC2A.O, SJ2.3; no longer IC7A.O
- net N$23: now also IC11A.O, SJ9.3; no longer IC8A.O
- net N$24: now also IC12A.O, SJ10.3; no longer IC9A.O
- net N$25: now also IC13A.O, SJ11.3; no longer IC10A.O
- net N$26: now also IC14A.O, SJ12.3; no longer IC11A.O
- net N$27: now also IC15A.O, SJ13.3; no longer IC12A.O
- net N$28: now also IC16A.O, SJ14.3; no longer IC13A.O
- net N$29: now also IC17A.O, SJ15.3; no longer IC14A.O
- net N$47: now also D3.C, SJ3.1; no longer IC4.IREF, R5.1
- net N$51: no longer D71.D, S1.LED1, S11.LED1, S12.LED1, S13.LED1, S14.LED1, S15.LED1, S2.LED1, S3.LED1, S4.LED1, S5.LED1
- net N$55: no longer D72.D, S16.LED1, S17.LED1, S18.LED1, S19.LED1, S20.LED1, S26.LED1, S27.LED1, S28.LED1, S29.LED1, S30.LED1
- net N$61: no longer D73.D, S31.LED1, S32.LED1, S33.LED1, S34.LED1, S35.LED1, S41.LED1, S42.LED1, S43.LED1, S44.LED1, S45.LED1
- net N$63: no longer D74.D, S46.LED1, S47.LED1, S48.LED1, S49.LED1, S50.LED1, S56.LED1, S57.LED1, S58.LED1, S59.LED1, S60.LED1
- net N$78: no longer D75.D, S61.LED1, S62.LED1, S63.LED1, S68.LED1, S69.LED1, S70.LED1
- net R0: now also SJ1.2, SJ10.2, SJ11.2, SJ12.2, SJ13.2, SJ14.2, SJ15.2, SJ2.2, SJ3.2, SJ4.2, SJ5.2, SJ6.2, SJ7.2, SJ8.2, SJ9.2, U$1.PF1(ADC1); no longer D1.C, D10.C, D11.C, D12.C, D13.C, D14.C, D15.C, D2.C, D3.C, D4.C, D5.C, D6.C, D7.C, D8.C, D9.C
- net R1: now also U$1.PF4(ADC4)
- net R2: now also U$1.PF5(ADC5)
- net R3: now also U$1.PF6(ADC6)
- net R4: now also U$1.PF7(ADC7)
- net RST: no longer S71.4
- net SCK: no longer IC4.SCLK
- net SOUT: now also IC3.SOUT; no longer IC4.SOUT
- net VIN: no longer D74.S, D75.S, R10.2, R9.2
- net XLAT: no longer IC4.XLAT
Other:
- moved on the sheet: C10, C11, C12, C13, C14, C15, C16, C17, C18, C19, C20, C21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
