File: hardware/ION-60/Eagle/ION-60/ION-60.sch (EAGLE design)
At the start: 486 parts, among them IC1 74LVC1G14DCK, IC10 74LVC1G14DCK, IC11 74LVC1G14DCK, IC12 74LVC1G14DCK, IC13 74LVC1G14DCK, IC14 74LVC1G14DCK, IC15 74LVC1G14DCK, IC16 74LVC1G14DCK, IC17 74LVC1G14DCK, IC18 74LVC1G14DCK, IC19 74LVC1G14DCK, IC2 74LVC1G14DCK, IC20 74LVC1G14DCK, IC21 74LVC1G14DCK, IC22 74LVC1G14DCK, IC23 74LVC1G14DCK, IC24 74LVC1G14DCK, IC25 74LVC1G14DCK, IC26 74LVC1G14DCK, IC27 74LVC1G14DCK, IC28 74LVC1G14DCK, IC29 74LVC1G14DCK, IC3 TLC5947DAP, IC30 74LVC1G14DCK, IC31 74LVC1G14DCK, IC32 74LVC1G14DCK, IC33 74LVC1G14DCK, IC34 74LVC1G14DCK, IC35 74LVC1G14DCK, IC36 74LVC1G14DCK, IC37 74LVC1G14DCK, IC38 74LVC1G14DCK, IC39 74LVC1G14DCK, IC40 74LVC1G14DCK, IC41 74LVC1G14DCK, IC42 74LVC1G14DCK, IC43 74LVC1G14DCK, IC44 74LVC1G14DCK, IC45 74LVC1G14DCK, IC46 74LVC1G14DCK, IC47 74LVC1G14DCK, IC48 74LVC1G14DCK, IC49 74LVC1G14DCK, IC5 74LVC1G14DCK, IC50 74LVC1G14DCK, IC51 74LVC1G14DCK, IC52 74LVC1G14DCK, IC53 74LVC1G14DCK, IC54 74LVC1G14DCK, IC55 74LVC1G14DCK, IC56 74LVC1G14DCK, IC57 74LVC1G14DCK, IC58 74LVC1G14DCK, IC59 74LVC1G14DCK, IC6 74LVC1G14DCK, IC60 74LVC1G14DCK, IC61 74LVC1G14DCK, IC62 74LVC1G14DCK, IC63 74LVC1G14DCK, IC64 74LVC1G14DCK, IC65 74LVC1G14DCK, IC66 74LVC1G14DCK, IC67 74LVC1G14DCK, IC68 74LVC1G14DCK, IC69 74LVC1G14DCK, IC7 74LVC1G14DCK, IC70 74LVC1G14DCK, IC71 74LVC1G14DCK, IC72 74LVC1G14DCK, IC73 VREG-5SOT23, IC8 74LVC1G14DCK, IC9 74LVC1G14DCK, J2 change, Q1 MOSFET-PSUPERSOT, Y1 16MHz

Commit message: Lots more work
Parts:
- removed J1: (no value), Jordi:2X03M-0.1-PTH-SHROUDED
- removed J2: change, Jordi:1X06M-0.05-PTH
- removed J3: (no value), Jordi:1X06M-0.1-PTH
- removed JP1, JP2, JP3, JP4: USB-MICROBSMD, Jordi:USB-MICROBSMD
- removed U$2, U$3: 74LVC138AD, SparkFun-DigitalIC:74LVC138AD
- added C79, C80, C83, C84: 1uF, Jordi:CAPACITOR0603
- added COL-EXP, LED-EXP: (no value), Jordi:1X06M-0.05-PTH
- added D74, D75, D79, D80: (no value), SparkFun-DiscreteSemi:DIODESOD123
- added EXP: check, Jordi:1X06M-0.05-PTH
- added IC4, IC74, IC75, IC76: 74LVC1G14DCK, 74xx-little-us:74LVC1G14DCK
- added IC77, IC78: 74LS595D, SparkFun-DigitalIC:74LS595D
- added ICSP: (no value), Jordi:2X03M-0.1-PTH-SHROUDED
- added R10, R15, R20, R5: 4.7k?, Jordi:RESISTOR0603
- added R14, R19, R24, R9: 22k?, Jordi:RESISTOR0603
- added R166, R167, R169, R170, R25: 10K, Jordi:RESISTOR0603
- added ROW-EXP: (no value), Jordi:1X06M-0.1-PTH
- added RST: (no value), Jordi:SWITCH-TACTILESMD-RA
- added S72, S73, S74, S75, S76, S77, S78, S79, S80, S81, S82: (no value), Jordi:CHERRY-MX-LED1X1
- added SJ16, SJ17, SJ18, SJ19, SJ20, SJ21, SJ22, SJ23, SJ24, SJ25, SJ26, SJ27, SJ28, SJ29, SJ30, SJ31, SJ32, SJ33, SJ34, SJ35, SJ36, SJ37, SJ38, SJ39, SJ40, SJ41, SJ42, SJ43, SJ44, SJ45, SJ46, SJ47, SJ48, SJ49, SJ50, SJ51, SJ52, SJ53, SJ54, SJ55, SJ56, SJ57, SJ58, SJ59, SJ60, SJ61, SJ62, SJ63, SJ64, SJ65, SJ66, SJ67, SJ68, SJ69, SJ70, SJ71, SJ72, SJ73, SJ74: JUMPER-PAD-3-2OF3_NC_BY_TRACE_SMALL, SparkFun-Passives:JUMPER-PAD-3-2OF3_NC_BY_TRACE_SMALL
- added USB1, USB2: USB-MICROBSMD, Jordi:USB-MICROBSMD
- S71: value RESET -> (none); device Jordi:SWITCH-TACTILESMD-RA -> Jordi:CHERRY-MX-LED1X1
Connections:
- net SW31 renamed N$12
- net SW32 renamed N$13
- net SW33 renamed N$15
- net SW34 renamed N$16
- net SW35 renamed N$30
- net SW36 renamed N$31
- net SW37 renamed N$32
- net SW38 renamed N$37
- net SW39 renamed N$38
- net SW40 renamed N$41
- net SW41 renamed N$42
- net SW42 renamed N$43
- net SW43 renamed N$51
- net SW44 renamed N$55
- net SW45 renamed N$61
- removed net !E1: U$1.PE6, U$2./E1, U$3./E1
- removed net A0: U$1.PB4(ADC11), U$2.A0, U$3.A0
- removed net A1: U$1.PB5(ADC12), U$2.A1, U$3.A1
- removed net A2: U$1.PB6(ADC13), U$2.A2, U$3.A2
- removed net A3: U$1.PB7, U$2./E2, U$3.E3
- removed net BLANK: IC3.BLANK, U$1.PB0(SS)
- removed net LED-A0: J3.1, R21.1
- removed net LED-A1: J3.2, R22.1
- removed net LED-A2: J3.3, R23.1
- removed net LED-A3: J3.4
- removed net LED-A4: J3.5
- removed net N$12 (its old number): S1.LED1, S2.LED1, S3.LED1, S4.LED1, S5.LED1
- removed net N$13 (its old number): S16.LED1, S17.LED1, S18.LED1, S19.LED1, S20.LED1
- removed net N$15 (its old number): S31.LED1, S32.LED1, S33.LED1, S34.LED1, S35.LED1
- removed net N$16 (its old number): S46.LED1, S47.LED1, S48.LED1, S49.LED1, S50.LED1
- removed net N$30 (its old number): S68.LED1, S69.LED1, S70.LED1
- removed net N$31 (its old number): S56.LED1, S57.LED1, S58.LED1, S59.LED1, S60.LED1
- removed net N$32 (its old number): S41.LED1, S42.LED1, S43.LED1, S44.LED1, S45.LED1
- removed net N$37 (its old number): S26.LED1, S27.LED1, S28.LED1, S29.LED1, S30.LED1
- removed net N$38 (its old number): S11.LED1, S12.LED1, S13.LED1, S14.LED1, S15.LED1
- removed net N$41 (its old number): D73.D
- removed net N$42 (its old number): D72.D
- removed net N$43 (its old number): D71.D
- removed net N$51 (its old number): S10.LED1, S6.LED1, S7.LED1, S8.LED1, S9.LED1
- removed net N$55 (its old number): S21.LED1, S22.LED1, S23.LED1, S24.LED1, S25.LED1
- removed net N$61 (its old number): S36.LED1, S37.LED1, S38.LED1, S39.LED1, S40.LED1
- removed net SOUT: IC3.SOUT, J3.6
- removed net XLAT: IC3.XLAT
- new net !COL70: C79.2, IC4A.I, R9.1
- new net !COL71: C80.2, IC74A.I, R14.1
- new net !COL72: C83.2, IC75A.I, R19.1
- new net !COL73: C84.2, IC76A.I, R24.1
- new net C-!OE: COL-EXP.3, IC77.G, IC78.G, U$1.PD7(ADC10)
- new net C-CLK: COL-EXP.5, IC77.SCK, IC78.SCK, U$1.PD5
- new net C-LAT: COL-EXP.4, IC77.RCK, IC78.RCK, U$1.PD6(ADC9)
- new net C-SIN: IC77.SER, U$1.PD4(ADC8)
- new net C-SOUT: COL-EXP.6, IC78.QH*
- new net C15: IC78.QH, ROW-EXP.6
- new net G0: D71.D, S1.LED1, S16.LED1, S17.LED1, S18.LED1, S19.LED1, S2.LED1, S20.LED1, S21.LED1, S3.LED1, S31.LED1, S32.LED1, S33.LED1, S34.LED1, S35.LED1, S36.LED1, S4.LED1, S46.LED1, S47.LED1, S48.LED1, S49.LED1, S5.LED1, S50.LED1, S51.LED1, S6.LED1
- new net G1: D72.D, S22.LED1, S23.LED1, S24.LED1, S37.LED1, S38.LED1, S39.LED1, S52.LED1, S53.LED1, S54.LED1, S61.LED1, S62.LED1, S63.LED1, S64.LED1, S67.LED1, S68.LED1, S69.LED1, S7.LED1, S70.LED1, S71.LED1, S72.LED1, S73.LED1, S74.LED1, S75.LED1, S76.LED1, S77.LED1, S78.LED1, S79.LED1, S8.LED1, S80.LED1, S81.LED1, S82.LED1, S9.LED1
- new net G2: D73.D, S10.LED1, S11.LED1, S12.LED1, S13.LED1, S14.LED1, S15.LED1, S25.LED1, S26.LED1, S27.LED1, S28.LED1, S29.LED1, S30.LED1, S40.LED1, S41.LED1, S42.LED1, S43.LED1, S44.LED1, S45.LED1, S55.LED1, S56.LED1, S57.LED1, S58.LED1, S59.LED1, S60.LED1
- new net LED-BLANK: IC3.BLANK, LED-EXP.3, U$1.PB0(SS)
- new net LED-G0: R21.1, U$1.PB5(ADC12)
- new net LED-G1: R22.1, U$1.PB6(ADC13)
- new net LED-G2: R23.1, U$1.PB7
- new net LED-SOUT: IC3.SOUT, LED-EXP.6
- new net LED-XLAT: IC3.XLAT, LED-EXP.4, U$1.PB4(ADC11)
- new net N$100: IC21A.O, SJ19.1
- new net N$101: D20.C, SJ20.3
- new net N$102: IC22A.O, SJ20.1
- new net N$103: D32.C, SJ32.3
- new net N$104: D31.C, SJ31.3
- new net N$107: D61.A, R146.1, R147.2, S61.SW1, S71.SW2
- new net N$108: IC68A.O, SJ66.1
- new net N$109: D65.C, SJ65.3
- new net N$110: IC67A.O, SJ65.1
- new net N$111: D64.C, SJ64.3
- new net N$127: IC56A.O, SJ54.3
- new net N$128: IC57A.O, SJ55.3
- new net N$129: IC58A.O, SJ56.3
- new net N$145: IC59A.O, SJ57.3
- new net N$146: IC60A.O, SJ58.3
- new net N$147: IC61A.O, SJ59.3
- new net N$163: D80.C, SJ74.3
- new net N$164: IC76A.O, SJ74.1
- new net N$165: D80.A, R20.1, R24.2, S70.SW2, S82.SW1
- new net N$176: IC49A.O, SJ47.1
- new net N$177: D48.C, SJ48.3
- new net N$178: IC50A.O, SJ48.1
- new net N$179: D49.C, SJ49.3
- new net N$180: IC48A.O, SJ46.1
- new net N$181: IC51A.O, SJ49.1
- new net N$182: D50.C, SJ50.3
- new net N$183: IC52A.O, SJ50.1
- new net N$184: D36.C, SJ36.1
- new net N$185: D37.C, SJ37.1
- new net N$186: D38.C, SJ38.1
- new net N$187: D39.C, SJ39.1
- new net N$188: D40.C, SJ40.1
- new net N$189: D41.C, SJ41.1
- new net N$190: D42.C, SJ42.1
- new net N$191: D43.C, SJ43.1
- new net N$192: D44.C, SJ44.1
- new net N$193: D45.C, SJ45.1
- new net N$194: IC77.QH*, IC78.SER
- new net N$68: IC18A.O, SJ16.1
- new net N$69: D17.C, SJ17.3
- new net N$70: IC19A.O, SJ17.1
- new net N$71: D18.C, SJ18.3
- new net N$72: IC20A.O, SJ18.1
- new net N$73: IC23A.O, SJ21.3
- new net N$76: IC24A.O, SJ22.3
- new net N$77: IC25A.O, SJ23.3
- new net N$79: IC26A.O, SJ24.3
- new net N$80: IC27A.O, SJ25.3
- new net N$81: IC28A.O, SJ26.3
- new net N$84: IC29A.O, SJ27.3
- new net N$85: IC30A.O, SJ28.3
- new net N$86: IC31A.O, SJ29.3
- new net N$87: IC32A.O, SJ30.3
- new net N$88: D30.C, SJ30.1
- new net N$89: D29.C, SJ29.1
- new net N$91: D28.C, SJ28.1
- new net N$92: D27.C, SJ27.1
- new net N$93: D26.C, SJ26.1
- new net N$95: D25.C, SJ25.1
- new net N$96: D24.C, SJ24.1
- new net N$97: D23.C, SJ23.1
- new net N$98: D22.C, SJ22.1
- new net N$99: D21.C, SJ21.1
- new net SW71: D75.A, R10.1, R14.2, S69.SW1, S80.SW2
- new net SW72: D79.A, R15.1, R19.2, S81.SW2
- net +3V3: now also COL-EXP.2, EXP.6, IC4P.VCC, IC74P.VCC, IC75P.VCC, IC76P.VCC, IC77.SCL, IC77.VCC, IC78.SCL, IC78.VCC, ICSP.2, LED-EXP.2, R10.2, R15.2, R20.2, R5.2; no longer J1.2, J2.6, U$2.E3, U$2.VCC, U$3.VCC
- net C0: now also IC77.QA, S61.SW2, S71.SW1; no longer S61.SW1, U$2./Y7
- net C1: now also C70.1, IC77.QB, S72.SW1; no longer U$2./Y6
- net C10: now also C78.1, IC78.QC, S78.SW1; no longer U$3./Y5
- net C11: now also C79.1, IC78.QD, S79.SW2; no longer C76.1, U$3./Y4
- net C12: now also C80.1, IC78.QE, S69.SW2, S80.SW1; no longer C77.1, S69.SW1, U$3./Y3
- net C13: now also C83.1, IC78.QF, S81.SW1; no longer U$3./Y2
- net C14: now also C84.1, IC78.QG, S82.SW2; no longer C78.1, U$3./Y1
- net C2: now also C71.1, IC77.QC, S73.SW2; no longer C70.1, U$2./Y5
- net C3: now also C72.1, IC77.QD, S63.SW2, S74.SW1; no longer C71.1, S63.SW1, U$2./Y4
- net C4: now also C73.1, IC77.QE, S75.SW1; no longer U$2./Y3
- net C5: now also C74.1, IC77.QF, S76.SW2; no longer C72.1, U$2./Y2
- net C6: now also C75.1, IC77.QG; no longer C73.1, U$2./Y1
- net C7: now also IC77.QH; no longer U$2./Y0
- net C8: now also C76.1, IC78.QA; no longer C74.1, U$3./Y7
- net C9: now also C77.1, IC78.QB, S67.SW2, S77.SW1; no longer C75.1, S67.SW1, U$3./Y6
- net D+: now also USB1.D+, USB2.D+; no longer JP1.D+, JP2.D+, JP3.D+, JP4.D+
- net D-: now also USB1.D-, USB2.D-; no longer JP1.D-, JP2.D-, JP3.D-, JP4.D-
- net GND: now also COL-EXP.1, EXP.1, IC4P.GND, IC74P.GND, IC75P.GND, IC76P.GND, IC77.GND, IC78.GND, ICSP.6, LED-EXP.1, R166.1, R167.1, R169.1, R170.1, R25.1, RST.1, USB1.GND, USB2.GND; no longer J1.6, J2.1, JP1.GND, JP2.GND, JP3.GND, JP4.GND, S71.1, U$2.GND, U$3./E2, U$3.GND
- net LED0: now also S46.LED2, S60.LED2, S72.LED2, S75.LED2
- net LED1: now also S31.LED2, S45.LED2, S61.LED2, S71.LED2
- net LED10: now also S18.LED2, S28.LED2, S70.LED2, S82.LED2
- net LED11: now also S13.LED2, S3.LED2, S78.LED2, S81.LED2
- net LED12: now also S49.LED2, S52.LED2, S57.LED2
- net LED13: now also S34.LED2, S37.LED2, S42.LED2
- net LED14: now also S19.LED2, S22.LED2, S27.LED2
- net LED15: now also S12.LED2, S4.LED2, S7.LED2
- net LED16: now also S50.LED2, S53.LED2, S56.LED2
- net LED17: now also S35.LED2, S38.LED2, S41.LED2
- net LED18: now also S20.LED2, S23.LED2, S26.LED2
- net LED19: now also S11.LED2, S5.LED2, S8.LED2
- net LED2: now also S16.LED2, S30.LED2, S62.LED2, S73.LED2
- net LED20: now also S51.LED2, S54.LED2, S55.LED2
- net LED21: now also S36.LED2, S39.LED2, S40.LED2
- net LED22: now also S21.LED2, S24.LED2, S25.LED2
- net LED23: now also S10.LED2, S6.LED2, S9.LED2
- net LED3: now also S1.LED2, S15.LED2, S63.LED2, S74.LED2
- net LED4: now also S47.LED2, S59.LED2, S64.LED2, S76.LED2
- net LED5: now also S32.LED2, S44.LED2, S65.LED2
- net LED6: now also S17.LED2, S29.LED2, S66.LED2
- net LED7: now also S14.LED2, S2.LED2, S67.LED2, S77.LED2
- net LED8: now also S48.LED2, S58.LED2, S68.LED2, S79.LED2
- net LED9: now also S33.LED2, S43.LED2, S69.LED2, S80.LED2
- net MISO: now also ICSP.1; no longer J1.1
- net MOSI: now also ICSP.4; no longer J1.4
- net N$11: now also USB1.VBUS, USB2.VBUS; no longer JP1.VBUS, JP2.VBUS, JP3.VBUS, JP4.VBUS
- net N$112: now also IC66A.O, SJ64.1; no longer IC18A.O
- net N$113: now also D63.C, SJ63.3; no longer IC19A.O
- net N$114: now also IC65A.O, SJ63.1; no longer IC20A.O
- net N$115: now also D62.C, SJ62.3; no longer IC21A.O
- net N$116: now also IC64A.O, SJ62.1; no longer IC22A.O
- net N$117: now also D61.C, SJ61.3; no longer IC23A.O
- net N$118: now also IC63A.O, SJ61.1; no longer IC24A.O
- net N$119: now also IC33A.O, SJ31.1; no longer IC25A.O
- net N$120: now also IC34A.O, SJ32.1; no longer IC26A.O
- net N$121: now also D33.C, SJ33.3; no longer IC27A.O
- net N$122: now also IC35A.O, SJ33.1; no longer IC28A.O
- net N$123: now also D34.C, SJ34.3; no longer IC29A.O
- net N$124: now also IC53A.O, SJ51.3; no longer IC30A.O
- net N$125: now also IC54A.O, SJ52.3; no longer IC31A.O
- net N$126: now also IC55A.O, SJ53.3; no longer IC32A.O
- net N$130: now also IC36A.O, SJ34.1; no longer IC33A.O
- net N$131: now also D35.C, SJ35.3; no longer IC34A.O
- net N$132: now also IC37A.O, SJ35.1; no longer IC35A.O
- net N$133: now also IC38A.O, SJ36.3; no longer IC36A.O
- net N$134: now also IC39A.O, SJ37.3; no longer IC37A.O
- net N$135: now also IC40A.O, SJ38.3; no longer IC38A.O
- net N$136: now also IC41A.O, SJ39.3; no longer IC39A.O
- net N$137: now also IC42A.O, SJ40.3; no longer IC40A.O
- net N$138: now also IC43A.O, SJ41.3; no longer IC41A.O
- net N$139: now also IC44A.O, SJ42.3; no longer IC42A.O
- net N$140: now also IC45A.O, SJ43.3; no longer IC43A.O
- net N$141: now also IC46A.O, SJ44.3; no longer IC44A.O
- net N$142: now also IC47A.O, SJ45.3; no longer IC45A.O
- net N$143: now also D46.C, SJ46.3; no longer IC46A.O
- net N$144: now also D47.C, SJ47.3; no longer IC47A.O
- net N$148: now also IC62A.O, SJ60.3; no longer IC48A.O
- net N$149: now also D69.C, SJ69.3; no longer IC49A.O
- net N$150: now also IC71A.O, SJ69.1; no longer IC50A.O
- net N$151: now also D70.C, SJ70.3; no longer IC51A.O
- net N$152: now also IC72A.O, SJ70.1; no longer IC52A.O
- net N$153: now also D67.C, SJ67.3; no longer IC53A.O
- net N$154: now also IC69A.O, SJ67.1; no longer IC54A.O
- net N$155: now also D68.C, SJ68.3; no longer IC55A.O
- net N$156: now also IC70A.O, SJ68.1; no longer IC56A.O
- net N$157: now also D74.C, SJ71.3; no longer IC57A.O
- net N$158: now also IC4A.O, SJ71.1; no longer IC58A.O
- net N$159: now also D75.C, SJ72.3; no longer IC59A.O
- net N$160: now also IC74A.O, SJ72.1; no longer IC60A.O
- net N$161: now also D79.C, SJ73.3; no longer IC61A.O
- net N$162: now also IC75A.O, SJ73.1; no longer IC62A.O
- net N$166: now also D60.C, SJ60.1; no longer IC63A.O
- net N$167: now also D59.C, SJ59.1; no longer IC64A.O
- net N$168: now also D58.C, SJ58.1; no longer IC65A.O
- net N$169: now also D57.C, SJ57.1; no longer IC66A.O
- net N$17: now also SJ1.3; no longer SJ1.1
- net N$170: now also D56.C, SJ56.1; no longer IC67A.O
- net N$171: now also D55.C, SJ55.1; no longer IC68A.O
- net N$172: now also D54.C, SJ54.1; no longer IC69A.O
- net N$173: now also D53.C, SJ53.1; no longer IC70A.O
- net N$174: now also D52.C, SJ52.1; no longer IC71A.O
- net N$175: now also D51.C, SJ51.1; no longer IC72A.O
- net N$21: now also D66.C, SJ66.3; no longer S61.LED1, S62.LED1, S63.LED1
- net N$22: now also D2.C; no longer IC2A.O
- net N$39: now also SJ1.1; no longer SJ1.3
- net N$40: now also IC2A.O; no longer D2.C
- net N$47: now also SJ3.3; no longer SJ3.1
- net N$48: now also IC5A.O, SJ3.1; no longer D4.C, SJ4.1
- net N$49: now also D4.C, SJ4.3; no longer D5.C, SJ5.1
- net N$54: now also IC6A.O, SJ4.1; no longer IC5A.O, SJ3.3
- net N$56: now also D5.C, SJ5.3; no longer IC6A.O, SJ4.3
- net N$57: now also SJ5.1; no longer SJ5.3
- net N$63: now also D16.C, SJ16.3; no longer S51.LED1, S52.LED1, S53.LED1, S54.LED1, S55.LED1
- net N$78: now also D19.C, SJ19.3; no longer S64.LED1, S65.LED1, S66.LED1, S67.LED1
- net R0: now also R25.2, ROW-EXP.1, U$1.PF0(ADC0); no longer U$1.PF1(ADC1)
- net R1: now also R166.2, ROW-EXP.2, SJ16.2, SJ17.2, SJ18.2, SJ19.2, SJ20.2, SJ21.2, SJ22.2, SJ23.2, SJ24.2, SJ25.2, SJ26.2, SJ27.2, SJ28.2, SJ29.2, SJ30.2; no longer D16.C, D17.C, D18.C, D19.C, D20.C, D21.C, D22.C, D23.C, D24.C, D25.C, D26.C, D27.C, D28.C, D29.C, D30.C
- net R2: now also R167.2, ROW-EXP.3, SJ31.2, SJ32.2, SJ33.2, SJ34.2, SJ35.2, SJ36.2, SJ37.2, SJ38.2, SJ39.2, SJ40.2, SJ41.2, SJ42.2, SJ43.2, SJ44.2, SJ45.2; no longer D31.C, D32.C, D33.C, D34.C, D35.C, D36.C, D37.C, D38.C, D39.C, D40.C, D41.C, D42.C, D43.C, D44.C, D45.C
- net R3: now also R169.2, ROW-EXP.4, SJ46.2, SJ47.2, SJ48.2, SJ49.2, SJ50.2, SJ51.2, SJ52.2, SJ53.2, SJ54.2, SJ55.2, SJ56.2, SJ57.2, SJ58.2, SJ59.2, SJ60.2; no longer D46.C, D47.C, D48.C, D49.C, D50.C, D51.C, D52.C, D53.C, D54.C, D55.C, D56.C, D57.C, D58.C, D59.C, D60.C
- net R4: now also R170.2, ROW-EXP.5, SJ61.2, SJ62.2, SJ63.2, SJ64.2, SJ65.2, SJ66.2, SJ69.2, SJ70.2, SJ71.2, SJ72.2, SJ73.2, SJ74.2; no longer D61.C, D62.C, D63.C, D64.C, D65.C, D66.C, D67.C, D68.C, D69.C, D70.C
- net RST: now also ICSP.5, RST.3; no longer J1.5, S71.3
- net RX: now also EXP.4; no longer J2.4
- net SCK: now also ICSP.3, LED-EXP.5; no longer J1.3
- net SW61: now also D74.A, R5.1, R9.2, S68.SW2, S79.SW1; no longer D61.A, R146.1, R147.2, S61.SW2
- net SW62: now also S72.SW2; no longer S62.SW2
- net SW63: now also S62.SW2, S73.SW1; no longer S63.SW2
- net SW64: now also S63.SW1, S74.SW2; no longer S64.SW2
- net SW65: now also S75.SW2; no longer S65.SW2
- net SW66: now also S64.SW2, S76.SW1; no longer S66.SW2
- net SW67: now also S65.SW2; no longer S67.SW2
- net SW68: now also S66.SW2; no longer S68.SW2
- net SW69: now also S67.SW1, S77.SW2; no longer S69.SW2
- net SW70: now also S78.SW2; no longer S70.SW2
- net TX: now also EXP.3; no longer J2.3
- net VBAT: now also EXP.2; no longer J2.2
- net VIN: now also EXP.5; no longer J2.5
Other:
- note removed: "change these (74hc595?)"
